File: hardware/alpha/dacattac-alpha.kicad_sch (KiCad schematic)
At the start: 0 parts

Commit message: WIP
Other:
- added sheet video-misc (video-misc.kicad_sch)
Changed lines of the file:
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@@
     (comment 1 "${LICENSE}")
   )
-  (sheet (at 121.285 78.74) (size 54.61 29.845) (fields_autoplaced)
+  (sheet (at 154.94 55.88) (size 54.61 29.845) (fields_autoplaced)
     (stroke (width 0.1524) (type solid))
     (fill (color 0 0 0 0.0000))
-    (property "Sheetname" "audio" (at 121.285 78.0284 0)
+    (property "Sheetname" "audio" (at 154.94 55.1684 0)
       (effects (font (size 1.27 1.27)) (justify left bottom))
     )
-    (property "Sheetfile" "audio.kicad_sch" (at 121.285 109.1696 0)
+    (property "Sheetfile" "audio.kicad_sch" (at 154.94 86.3096 0)
       (effects (font (size 1.27 1.27)) (justify left top))
     )
@@
     )
   )
-  (sheet (at 64.135 78.74) (size 54.61 29.845) (fields_autoplaced)
+  (sheet (at 97.79 55.88) (size 54.61 29.845) (fields_autoplaced)
     (stroke (width 0.1524) (type solid))
     (fill (color 0 0 0 0.0000))
-    (property "Sheetname" "video" (at 64.135 78.0284 0)
+    (property "Sheetname" "video" (at 97.79 55.1684 0)
       (effects (font (size 1.27 1.27)) (justify left bottom))
     )
-    (property "Sheetfile" "video.kicad_sch" (at 64.135 109.1696 0)
+    (property "Sheetfile" "video.kicad_sch" (at 97.79 86.3096 0)
+      (effects (font (size 1.27 1.27)) (justify left top))
+    )
+    (instances
+      (project "dacattac-alpha"
+        (path "/487245ca-0c1f-4f9d-bc99-20c8f558090f" (page "1"))
+      )
+    )
+  )
+  (sheet (at 154.94 100.33) (size 54.61 29.845) (fields_autoplaced)
+    (stroke (width 0.1524) (type solid))
+    (fill (color 0 0 0 0.0000))
+    (property "Sheetname" "power" (at 154.94 99.6184 0)
+      (effects (font (size 1.27 1.27)) (justify left bottom))
+    )
+    (property "Sheetfile" "power.kicad_sch" (at 154.94 130.7596 0)
+      (effects (font (size 1.27 1.27)) (justify left top))
+    )
+    (instances
+      (project "dacattac-alpha"
+        (path "/487245ca-0c1f-4f9d-bc99-20c8f558090f" (page "4"))
+      )
+    )
+  )
+  (sheet (at 97.79 100.33) (size 54.61 29.845) (fields_autoplaced)
+    (stroke (width 0.1524) (type solid))
+    (fill (color 0 0 0 0.0000))
+    (property "Sheetname" "video-misc" (at 97.79 99.6184 0)
+      (effects (font (size 1.27 1.27)) (justify left bottom))
+    )
+    (property "Sheetfile" "video-misc.kicad_sch" (at 97.79 130.7596 0)
       (effects (font (size 1.27 1.27)) (justify left top))
     )
@@
     )
   )
-  (sheet (at 178.435 78.74) (size 54.61 29.845) (fields_autoplaced)
-    (stroke (width 0.1524) (type solid))
-    (fill (color 0 0 0 0.0000))
-    (property "Sheetname" "power" (at 178.435 78.0284 0)
-      (effects (font (size 1.27 1.27)) (justify left bottom))
-    )
-    (property "Sheetfile" "power.kicad_sch" (at 178.435 109.1696 0)
-      (effects (font (size 1.27 1.27)) (justify left top))
-    )
-    (instances
-      (project "dacattac-alpha"
-        (path "/487245ca-0c1f-4f9d-bc99-20c8f558090f" (page "4"))
-      )
-    )
-  )
   (sheet_instances
-    (path "/" (page "1"))
+    (path "/" (page "5"))
   )
 )
