File: hardware/alpha/video.kicad_sch (KiCad schematic)
At the start: 103 parts, among them J1 BANK2_AUX, J2 OUT1, J3 OUT2, U1 L78L05_SO8, U3 L79L05_SO8, U4 AD768, U5 MAX4104, U6 AD8620, U7 MAX4104, U8 MCP47FEB22A0-E/ST

Commit message: Updated
Parts:
- added R31: 0, symbol Device:R
Connections:
- net GND: now also R31.1
- net GNDA: now also R31.2
Changed lines of the file:
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@@
   (junction (at 182.88 60.96) (diameter 0) (color 0 0 0 0)
   )
+  (junction (at 33.02 182.88) (diameter 0) (color 0 0 0 0)
+  )
   (junction (at 223.52 70.485) (diameter 0) (color 0 0 0 0)
   )
@@
     (stroke (width 0) (type default))
   )
+  (wire (pts (xy 33.02 182.88) (xy 36.195 182.88))
+    (stroke (width 0) (type default))
+  )
   (wire (pts (xy 210.82 75.565) (xy 213.36 75.565))
     (stroke (width 0) (type default))
@@
     (stroke (width 0) (type default))
   )
+  (wire (pts (xy 43.815 182.88) (xy 45.72 182.88))
+    (stroke (width 0) (type default))
+  )
   (wire (pts (xy 183.515 139.7) (xy 183.515 132.715))
     (stroke (width 0) (type default))
@@
     (stroke (width 0) (type default))
   )
-  (wire (pts (xy 33.02 166.37) (xy 33.02 180.975))
+  (wire (pts (xy 33.02 166.37) (xy 33.02 182.88))
     (stroke (width 0) (type default))
   )
@@
     (stroke (width 0) (type default))
   )
+  (wire (pts (xy 33.02 182.88) (xy 33.02 186.055))
+    (stroke (width 0) (type default))
+  )
   (wire (pts (xy 147.955 142.24) (xy 156.21 142.24))
     (stroke (width 0) (type default))
@@
     (stroke (width 0) (type default))
   )
+  (wire (pts (xy 45.72 182.88) (xy 45.72 186.055))
+    (stroke (width 0) (type default))
+  )
   (wire (pts (xy 242.57 107.315) (xy 236.22 107.315))
     (stroke (width 0) (type default))
@@
     )
   )
-  (symbol (lib_id "power:GND") (at 33.02 180.975 0) (unit 1)
+  (symbol (lib_id "power:GND") (at 33.02 186.055 0) (unit 1)
     (in_bom yes) (on_board yes) (dnp no) (fields_autoplaced)
-    (property "Reference" "#PWR03" (at 33.02 187.325 0)
+    (property "Reference" "#PWR03" (at 33.02 192.405 0)
       (effects (font (size 1.27 1.27)) hide)
     )
-    (property "Value" "GND" (at 33.02 185.42 0)
+    (property "Value" "GND" (at 33.02 190.5 0)
       (effects (font (size 1.27 1.27)))
     )
-    (property "Footprint" "" (at 33.02 180.975 0)
+    (property "Footprint" "" (at 33.02 186.055 0)
       (effects (font (size 1.27 1.27)) hide)
     )
-    (property "Datasheet" "" (at 33.02 180.975 0)
+    (property "Datasheet" "" (at 33.02 186.055 0)
       (effects (font (size 1.27 1.27)) hide)
     )
@@
     )
   )
+  (symbol (lib_id "Device:R") (at 40.005 182.88 90) (unit 1)
+    (in_bom yes) (on_board yes) (dnp no)
+    (property "Reference" "R31" (at 40.005 180.34 90)
+      (effects (font (size 1.27 1.27)))
+    )
+    (property "Value" "0" (at 40.005 182.88 90)
+      (effects (font (size 1.27 1.27)))
+    )
+    (property "Footprint" "" (at 40.005 184.658 90)
+      (effects (font (size 1.27 1.27)) hide)
+    )
+    (property "Datasheet" "~" (at 40.005 182.88 0)
+      (effects (font (size 1.27 1.27)) hide)
+    )
+    (pin "1")
+    (pin "2")
+    (instances
+      (project "dacattac-alpha"
+        (path "/487245ca-0c1f-4f9d-bc99-20c8f558090f/b4bbface-dd1a-4873-ab51-f35caad404be"
+          (reference "R31") (unit 1)
+        )
+      )
+    )
+  )
   (symbol (lib_id "AD768:AD768") (at 50.165 95.885 0) (unit 1)
     (in_bom yes) (on_board yes) (dnp no)
@@
         )
       )
+    )
+  )
+  (symbol (lib_id "power:GNDA") (at 45.72 186.055 0) (unit 1)
+    (in_bom yes) (on_board yes) (dnp no) (fields_autoplaced)
+    (property "Reference" "#PWR054" (at 45.72 192.405 0)
+      (effects (font (size 1.27 1.27)) hide)
+    )
+    (property "Value" "GNDA" (at 45.72 191.135 0)
+      (effects (font (size 1.27 1.27)))
+    )
+    (property "Footprint" "" (at 45.72 186.055 0)
+      (effects (font (size 1.27 1.27)) hide)
+    )
+    (property "Datasheet" "" (at 45.72 186.055 0)
+      (effects (font (size 1.27 1.27)) hide)
+    )
+    (pin "1")
+    (instances
+      (project "dacattac-alpha"
+        (path "/487245ca-0c1f-4f9d-bc99-20c8f558090f/b4bbface-dd1a-4873-ab51-f35caad404be"
+          (reference "#PWR054") (unit 1)
+        )
+      )

Commit message: Updated
Parts:
- added C69: NF, symbol Device:C
- added C70: 180p, symbol Device:C
- added R43, R44: 2k2, symbol Device:R
- C1, C2, C3, C4: value 0.1uF -> 0.1u
- C18, C20, C29, C30, C31: value 100pF -> 100p
- C19: value 82pF -> 82p
- C34: value 56pF -> 56p
- C38: value 270pF -> 270p
- C39: value 180p -> 560p
- C40: value NF -> 100p
- C41: value 18pF -> 18p
- C42: value 220pF -> 220p
- C45: value 100nF -> 100n
- C5, C6: value 33uF -> 33u
- C7, C8: value 0.1 -> 0.1u
- J2: value OUT1 -> VIDEO OUT1
- J3: value OUT2 -> VIDEO OUT2
- L1, L2, L5, L6: value 5.6uH -> 5.6u
- R19: value 1K8 -> 1k8
- R2: value 3K9 -> 3k9
- R20: value 4K7 -> 4k7
- R22: value 2K2 -> 2k2
- R25, R5: value 3K3 -> 3k3
- R3: value 10K -> 10k
- R8: value 475 -> 470
- U6: value AD8620 -> TLE2082
- renumbered J1 to P30
Connections:
- net +5V: now also R43.1, R44.1
- net GNDA: now also C69.2, C70.2
- net at C41.2, C42.2, L13.4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: now also C69.1, C70.1
- net HACKRF_VCC renamed +3.3V_HACKRF
- net SCL renamed DA_SCL
- net DA_SCL: now also R43.2
- net SDA renamed DA_SDA
- net DA_SDA: now also R44.2
Other:
- note removed: "TO CHECK: ORIENTATION OF ALL OP-AMPS! SOME HAVE BEEN FLIPPED / PINS CHANGED!! GROUNDS"
- moved on the sheet: C1, C11, C12, C13, C14, C15, C16, C17, C18, C19, C2, C20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

Commit message: WIP
Parts:
- removed C1 (x2), C2 (x2), C3, C4, C7, C8: 0.1u, symbol Device:C
- removed C5, C6: 33u, symbol Device:C
- removed L1: 5.6uH, symbol Device:L
- removed L1, L2 (x2): 5.6u, symbol Device:L
- removed R31: 0, symbol Device:R
- removed R43, R44: 2k2, symbol Device:R
- removed U1: L78L05_SO8, Package_SO:SOIC-8_3.9x4.9mm_P1.27mm, symbol Regulator_Linear:L78L05_SO8
- removed U3: L79L05_SO8, Package_SO:SOIC-8_3.9x4.9mm_P1.27mm, symbol Regulator_Linear:L79L05_SO8
- removed unit 3 of U6
- removed U8: MCP47FEB22A0-E/ST, Package_SO:SOIC-8_3.9x4.9mm_P1.27mm, symbol mcp47febxx:MCP47FEBXX
- C11, C12, C13, C14, C15, C16, C17, C21, C22, C23, C43, C44: value 0.1 -> 100n; footprint (none) -> Capacitor_SMD:C_0603_1608Metric
- C18, C19, C20, C24, C25, C26, C27, C28, C29, C30, C31, C32, C33, C34, C35, C36, C37, C38, C39, C40, C41, C42, C45, C46, C47, C48, C50, C69, C70: footprint (none) -> Capacitor_SMD:C_0603_1608Metric
- C49: footprint (none) -> BFC2808xxxxx:BFC2808xxxxx
- JP1: footprint (none) -> Connector_PinHeader_2.54mm:PinHeader_1x03_P2.54mm_Vertical
- L5, L6: footprint (none) -> Inductor_SMD:L_1210_3225Metric
- R1, R10, R11, R12, R13, R14, R15, R16, R17, R18, R19, R2, R20, R22, R23, R24, R25, R26, R27, R28, R3, R4, R5, R6, R7, R8, R9: footprint (none) -> Resistor_SMD:R_0603_1608Metric
- R21: value 1K -> 1k; footprint (none) -> Resistor_SMD:R_0603_1608Metric
- U4: footprint (none) -> Package_SO:SOIC-28W_7.5x18.7mm_P1.27mm
Other:
- note added: "C49: BFC280811229"
- moved on the sheet: C11, C12, C13, C14, C15, C16, C17, C18, C19, C20, C21, C22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

Commit message: WIP
Parts:
- removed P30: BANK2_AUX, symbol Connector_Generic:Conn_02x10_Odd_Even
Connections:
- net CLK renamed DAC_CLK

Commit message: WIP
Parts:
- J2, J3: footprint (none) -> MOLEX_73101:731010120
- L10, L11, L12, L13, L14, L7, L8, L9: footprint (none) -> NEOSID_7MM:NEOSID_7MM
Changed lines of the file:
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@@
       (effects (font (size 1.27 1.27)) (justify right))
     )
-    (property "Footprint" "" (at 257.81 140.97 0)
+    (property "Footprint" "NEOSID_7MM:NEOSID_7MM" (at 257.81 140.97 0)
       (effects (font (size 1.27 1.27)) hide)
     )
@@
       (effects (font (size 1.27 1.27)) (justify right))
     )
-    (property "Footprint" "" (at 161.925 102.87 0)
+    (property "Footprint" "NEOSID_7MM:NEOSID_7MM" (at 161.925 102.87 0)
       (effects (font (size 1.27 1.27)) hide)
     )
@@
       (effects (font (size 1.27 1.27)))
     )
-    (property "Footprint" "" (at 187.325 78.105 0)
+    (property "Footprint" "NEOSID_7MM:NEOSID_7MM" (at 187.325 78.105 0)
       (effects (font (size 1.27 1.27)) hide)
     )
@@
       (effects (font (size 1.27 1.27)) (justify left))
     )
-    (property "Footprint" "" (at 278.13 84.455 0)
+    (property "Footprint" "MOLEX_73101:731010120" (at 278.13 84.455 0)
       (effects (font (size 1.27 1.27)) hide)
     )
@@
       (effects (font (size 1.27 1.27)))
     )
-    (property "Footprint" "" (at 202.565 78.105 0)
+    (property "Footprint" "NEOSID_7MM:NEOSID_7MM" (at 202.565 78.105 0)
       (effects (font (size 1.27 1.27)) hide)
     )
@@
       (effects (font (size 1.27 1.27)))
     )
-    (property "Footprint" "" (at 217.805 78.105 0)
+    (property "Footprint" "NEOSID_7MM:NEOSID_7MM" (at 217.805 78.105 0)
       (effects (font (size 1.27 1.27)) hide)
     )
@@
       (effects (font (size 1.27 1.27)) (justify left))
     )
-    (property "Footprint" "" (at 278.13 107.315 0)
+    (property "Footprint" "MOLEX_73101:731010120" (at 278.13 107.315 0)
       (effects (font (size 1.27 1.27)) hide)
     )
@@
       (effects (font (size 1.27 1.27)) (justify right))
     )
-    (property "Footprint" "" (at 146.685 102.87 0)
+    (property "Footprint" "NEOSID_7MM:NEOSID_7MM" (at 146.685 102.87 0)
       (effects (font (size 1.27 1.27)) hide)
     )
@@
       (effects (font (size 1.27 1.27)))
     )
-    (property "Footprint" "" (at 156.845 86.995 0)
+    (property "Footprint" "NEOSID_7MM:NEOSID_7MM" (at 156.845 86.995 0)
       (effects (font (size 1.27 1.27)) hide)
     )
@@
       (effects (font (size 1.27 1.27)))
     )
-    (property "Footprint" "" (at 172.085 86.995 0)
-      (effects (font (size 1.27 1.27)) hide)
-    )
+    (property "Footprint" "NEOSID_7MM:NEOSID_7MM" (at 172.085 86.995 0)
+      (effects (font (size 1.27 1.27)) hide)
+    )

Commit message: WIP
Connections:
- net GNDA: now also L10.6, L11.6, L12.6, L13.6, L14.6, L7.6, L8.6, L9.6; no longer L10.1, L11.1, L12.1, L13.1, L14.1, L7.1, L8.1, L9.1
Changed lines of the file:
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@@
   (junction (at 263.525 107.315) (diameter 0) (color 0 0 0 0)
   )
+  (junction (at 248.92 133.985) (diameter 0) (color 0 0 0 0)
+  )
   (junction (at 170.815 128.905) (diameter 0) (color 0 0 0 0)
   )
@@
   (junction (at 210.185 66.04) (diameter 0) (color 0 0 0 0)
   )
-  (junction (at 248.92 133.985) (diameter 0) (color 0 0 0 0)
-  )
   (junction (at 225.425 72.39) (diameter 0) (color 0 0 0 0)
   )
@@
     (stroke (width 0) (type default))
   )
-  (wire (pts (xy 248.92 133.985) (xy 248.92 135.89))
-    (stroke (width 0) (type default))
-  )
   (wire (pts (xy 164.465 66.04) (xy 164.465 72.39))
     (stroke (width 0) (type default))
@@
     (stroke (width 0) (type default))
   )
+  (wire (pts (xy 248.92 133.985) (xy 248.92 135.89))
+    (stroke (width 0) (type default))
+  )
   (wire (pts (xy 20.955 92.075) (xy 29.21 92.075))
     (stroke (width 0) (type default))
@@
     (effects (font (size 1.27 1.27)) (justify left bottom))
   )
-  (global_label "DAC_AD[0..15]" (shape input) (at 31.75 73.66 0) (fields_autoplaced)
+  (global_label "AD[0..15]" (shape input) (at 31.75 73.66 0) (fields_autoplaced)
     (effects (font (size 1.27 1.27)) (justify left))
-    (property "Intersheetrefs" "${INTERSHEET_REFS}" (at 48.2215 73.66 0)
+    (property "Intersheetrefs" "${INTERSHEET_REFS}" (at 43.6253 73.66 0)
       (effects (font (size 1.27 1.27)) (justify left) hide)
     )
@@
     (pin "1")
     (pin "4")
-    (pin "1")
-    (pin "1")
+    (pin "6")
+    (pin "6")
     (instances
       (project "dacattac-alpha"
@@
       (effects (font (size 1.27 1.27)) hide)
     )
+    (pin "6")
     (pin "1")
-    (pin "1")
-    (pin "1")
+    (pin "6")
     (pin "4")
     (instances
@@
     (pin "1")
     (pin "4")
-    (pin "1")
-    (pin "1")
+    (pin "6")
+    (pin "6")
     (instances
       (project "dacattac-alpha"
@@
     )
     (pin "4")
+    (pin "6")
     (pin "1")
-    (pin "1")
-    (pin "1")
+    (pin "6")
     (instances
       (project "dacattac-alpha"
@@
     )
     (pin "4")
+    (pin "6")
     (pin "1")
-    (pin "1")
-    (pin "1")
+    (pin "6")
     (instances
       (project "dacattac-alpha"
@@
       (effects (font (size 1.27 1.27)) hide)
     )
-    (pin "1")
-    (pin "1")
+    (pin "6")
+    (pin "6")
     (pin "1")
     (pin "4")
@@
       (effects (font (size 1.27 1.27)) hide)
     )
-    (pin "1")
+    (pin "6")
     (pin "4")
     (pin "5")
     (pin "1")
-    (pin "1")
+    (pin "6")
     (pin "2")
     (instances
@@
     (pin "1")
     (pin "2")
-    (pin "1")
-    (pin "1")
+    (pin "6")
+    (pin "6")
     (pin "4")
     (instances

Commit message: WIP
Connections:
- net at C18.2, C19.2, C20.2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: now also L7.1, L8.5; no longer L7.5, L8.1
- net at C29.2, C30.2, C31.2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: now also L8.1; no longer L8.5
- net at C18.1, C19.1, C20.1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: now also L7.5; no longer L7.1

Commit message: WIP
Other:
- moved on the sheet: R6, R7
Changed lines of the file:
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@@
   (junction (at 104.14 132.08) (diameter 0) (color 0 0 0 0)
   )
-  (junction (at 103.505 103.505) (diameter 0) (color 0 0 0 0)
+  (junction (at 104.14 103.505) (diameter 0) (color 0 0 0 0)
   )
   (junction (at 215.9 111.76) (diameter 0) (color 0 0 0 0)
@@
     (stroke (width 0) (type default))
   )
-  (wire (pts (xy 103.505 103.505) (xy 105.41 103.505))
+  (wire (pts (xy 104.14 103.505) (xy 105.41 103.505))
     (stroke (width 0) (type default))
   )
@@
     (stroke (width 0) (type default))
   )
-  (wire (pts (xy 103.505 106.68) (xy 103.505 103.505))
+  (wire (pts (xy 104.14 106.68) (xy 104.14 103.505))
     (stroke (width 0) (type default))
   )
@@
     (stroke (width 0) (type default))
   )
-  (wire (pts (xy 101.6 103.505) (xy 103.505 103.505))
+  (wire (pts (xy 102.87 103.505) (xy 104.14 103.505))
     (stroke (width 0) (type default))
   )
@@
     (stroke (width 0) (type default))
   )
-  (wire (pts (xy 101.6 106.68) (xy 103.505 106.68))
+  (wire (pts (xy 102.87 106.68) (xy 104.14 106.68))
     (stroke (width 0) (type default))
   )
@@
     (stroke (width 0) (type default))
   )
-  (wire (pts (xy 84.455 103.505) (xy 93.98 103.505))
-    (stroke (width 0) (type default))
-  )
   (wire (pts (xy 69.85 125.095) (xy 76.2 125.095))
     (stroke (width 0) (type default))
@@
     (stroke (width 0) (type default))
   )
-  (wire (pts (xy 93.98 106.68) (xy 92.075 106.68))
+  (wire (pts (xy 95.25 106.68) (xy 93.345 106.68))
     (stroke (width 0) (type default))
   )
@@
     (stroke (width 0) (type default))
   )
-  (wire (pts (xy 92.075 106.68) (xy 92.075 108.585))
+  (wire (pts (xy 93.345 106.68) (xy 93.345 108.585))
     (stroke (width 0) (type default))
   )
@@
     (stroke (width 0) (type default))
   )
+  (wire (pts (xy 93.98 103.505) (xy 95.25 103.505))
+    (stroke (width 0) (type default))
+  )
   (wire (pts (xy 194.945 95.885) (xy 194.945 99.06))
     (stroke (width 0) (type default))
@@
     (effects (font (size 1.27 1.27)) (justify left bottom))
   )
-  (label "OFFSET_ADJ" (at 193.04 41.275 0) (fields_autoplaced)
-    (effects (font (size 1.27 1.27)) (justify left bottom))
-  )
   (label "AD0" (at 22.86 86.995 0) (fields_autoplaced)
     (effects (font (size 1.27 1.27)) (justify left bottom))
@@
     (effects (font (size 1.27 1.27)) (justify left bottom))
   )
-  (label "GAIN_ADJ" (at 85.09 103.505 0) (fields_autoplaced)
-    (effects (font (size 1.27 1.27)) (justify left bottom))
-  )
   (label "AD5" (at 22.86 99.695 0) (fields_autoplaced)
     (effects (font (size 1.27 1.27)) (justify left bottom))
@@
     (effects (font (size 1.27 1.27)) (justify left bottom))
   )
+  (global_label "GAIN_ADJ" (shape input) (at 93.98 103.505 180) (fields_autoplaced)
+    (effects (font (size 1.27 1.27)) (justify right))
+    (property "Intersheetrefs" "${INTERSHEET_REFS}" (at 82.4071 103.505 0)
+      (effects (font (size 1.27 1.27)) (justify right) hide)
+    )
+  )
   (global_label "AD[0..15]" (shape input) (at 31.75 73.66 0) (fields_autoplaced)
     (effects (font (size 1.27 1.27)) (justify left))
@@
     )
   )
-  (symbol (lib_id "Device:R") (at 97.79 103.505 90) (unit 1)
+  (global_label "OFFSET_ADJ" (shape input) (at 191.135 41.275 180) (fields_autoplaced)
+    (effects (font (size 1.27 1.27)) (justify right))
+    (property "Intersheetrefs" "${INTERSHEET_REFS}" (at 177.0222 41.275 0)
+      (effects (font (size 1.27 1.27)) (justify right) hide)
+    )
+  )
+  (symbol (lib_id "Device:R") (at 99.06 103.505 90) (unit 1)
     (in_bom yes) (on_board yes) (dnp no)
-    (property "Reference" "R7" (at 102.235 102.235 90)
+    (property "Reference" "R7" (at 103.505 102.235 90)
       (effects (font (size 1.27 1.27)))
     )
-    (property "Value" "330" (at 97.79 103.505 90)
+    (property "Value" "330" (at 99.06 103.505 90)
       (effects (font (size 1.27 1.27)))
     )
-    (property "Footprint" "Resistor_SMD:R_0603_1608Metric" (at 97.79 105.283 90)
+    (property "Footprint" "Resistor_SMD:R_0603_1608Metric" (at 99.06 105.283 90)
       (effects (font (size 1.27 1.27)) hide)
     )
-    (property "Datasheet" "~" (at 97.79 103.505 0)
+    (property "Datasheet" "~" (at 99.06 103.505 0)
       (effects (font (size 1.27 1.27)) hide)
     )
@@
     )
   )
-  (symbol (lib_id "Device:R") (at 97.79 106.68 90) (unit 1)
+  (symbol (lib_id "Device:R") (at 99.06 106.68 90) (unit 1)
     (in_bom yes) (on_board yes) (dnp no)
-    (property "Reference" "R6" (at 97.79 109.22 90)
+    (property "Reference" "R6" (at 99.06 109.22 90)
       (effects (font (size 1.27 1.27)))
     )
-    (property "Value" "R" (at 97.79 106.68 90)
+    (property "Value" "R" (at 99.06 106.68 90)
       (effects (font (size 1.27 1.27)))
     )
-    (property "Footprint" "Resistor_SMD:R_0603_1608Metric" (at 97.79 108.458 90)
+    (property "Footprint" "Resistor_SMD:R_0603_1608Metric" (at 99.06 108.458 90)
       (effects (font (size 1.27 1.27)) hide)
     )
-    (property "Datasheet" "~" (at 97.79 106.68 0)
+    (property "Datasheet" "~" (at 99.06 106.68 0)
       (effects (font (size 1.27 1.27)) hide)
     )
@@
     )
   )
-  (symbol (lib_id "power:GNDA") (at 92.075 108.585 0) (unit 1)
+  (symbol (lib_id "power:GNDA") (at 93.345 108.585 0) (unit 1)
     (in_bom yes) (on_board yes) (dnp no)
-    (property "Reference" "#PWR021" (at 92.075 114.935 0)
+    (property "Reference" "#PWR021" (at 93.345 114.935 0)
       (effects (font (size 1.27 1.27)) hide)
     )
-    (property "Value" "GNDA" (at 92.075 112.395 0)
+    (property "Value" "GNDA" (at 93.345 112.395 0)
       (effects (font (size 1.27 1.27)))
     )
-    (property "Footprint" "" (at 92.075 108.585 0)
+    (property "Footprint" "" (at 93.345 108.585 0)
       (effects (font (size 1.27 1.27)) hide)
     )
-    (property "Datasheet" "" (at 92.075 108.585 0)
+    (property "Datasheet" "" (at 93.345 108.585 0)
       (effects (font (size 1.27 1.27)) hide)
     )
