File: hardware/alpha/video.kicad_sch (KiCad schematic)
At the start: 87 parts, among them J2 VIDEO OUT1, J3 VIDEO OUT2, U4 AD768, U5 MAX4104, U6 TLE2082, U7 MAX4104

Commit message: WIP
Parts:
- removed C11: 100n, Capacitor_SMD:C_0603_1608Metric, symbol Device:C
Changed lines of the file:
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@@
   (junction (at 149.225 72.39) (diameter 0) (color 0 0 0 0)
   )
-  (junction (at 92.71 71.755) (diameter 0) (color 0 0 0 0)
-  )
   (junction (at 164.465 86.995) (diameter 0) (color 0 0 0 0)
   )
@@
   (junction (at 210.185 72.39) (diameter 0) (color 0 0 0 0)
   )
-  (junction (at 78.74 59.69) (diameter 0) (color 0 0 0 0)
-  )
   (junction (at 155.575 113.665) (diameter 0) (color 0 0 0 0)
   )
@@
     (stroke (width 0) (type default))
   )
-  (wire (pts (xy 92.71 71.755) (xy 92.71 69.215))
-    (stroke (width 0) (type default))
-  )
   (wire (pts (xy 160.655 66.04) (xy 164.465 66.04))
     (stroke (width 0) (type default))
@@
     (stroke (width 0) (type default))
   )
-  (wire (pts (xy 78.74 59.69) (xy 78.74 61.595))
+  (wire (pts (xy 78.74 57.785) (xy 78.74 61.595))
     (stroke (width 0) (type default))
   )
@@
     (stroke (width 0) (type default))
   )
-  (wire (pts (xy 78.74 59.69) (xy 92.71 59.69))
-    (stroke (width 0) (type default))
-  )
   (wire (pts (xy 210.185 86.995) (xy 210.185 95.885))
     (stroke (width 0) (type default))
@@
     (stroke (width 0) (type default))
   )
-  (wire (pts (xy 78.74 57.785) (xy 78.74 59.69))
-    (stroke (width 0) (type default))
-  )
   (wire (pts (xy 81.915 94.615) (xy 81.915 133.985))
     (stroke (width 0) (type default))
@@
   )
   (wire (pts (xy 102.235 76.835) (xy 97.79 76.835))
-    (stroke (width 0) (type default))
-  )
-  (wire (pts (xy 92.71 59.69) (xy 92.71 61.595))
     (stroke (width 0) (type default))
   )
@@
         )
       )
-    )
-  )
-  (symbol (lib_id "Device:C") (at 92.71 65.405 0) (unit 1)
-    (in_bom yes) (on_board yes) (dnp no)
-    (property "Reference" "C11" (at 96.52 64.135 0)
-      (effects (font (size 1.27 1.27)) (justify left))
-    )
-    (property "Value" "100n" (at 96.52 66.675 0)
-      (effects (font (size 1.27 1.27)) (justify left))
-    )
-    (property "Footprint" "Capacitor_SMD:C_0603_1608Metric" (at 93.6752 69.215 0)
-      (effects (font (size 1.27 1.27)) hide)
-    )
-    (property "Datasheet" "~" (at 92.71 65.405 0)
-      (effects (font (size 1.27 1.27)) hide)
-    )
-    (pin "2")
-    (pin "1")
-    (instances
-      (project "dacattac-alpha"
-        (path "/487245ca-0c1f-4f9d-bc99-20c8f558090f/b4bbface-dd1a-4873-ab51-f35caad404be"
-          (reference "C11") (unit 1)
-        )
-        (path "/487245ca-0c1f-4f9d-bc99-20c8f558090f/e1e307fe-d49b-45b6-b177-774a7a482979"
-          (reference "C79") (unit 1)
-        )
-      )

Commit message: WIP
Parts:
- removed J3: VIDEO OUT2, MOLEX_73101:731010120, symbol Connector:Conn_Coaxial
- removed R18: 75, Resistor_SMD:R_0603_1608Metric, symbol Device:R
Connections:
- net VIDEO: now reaches R17.1, R24.2, R27.1, U7.1
Other:
- moved on the sheet: J2
Changed lines of the file:
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@@
     (stroke (width 0) (type default))
   )
-  (wire (pts (xy 272.415 84.455) (xy 273.05 84.455))
+  (wire (pts (xy 272.415 84.455) (xy 273.685 84.455))
     (stroke (width 0) (type default))
   )
@@
     (stroke (width 0) (type default))
   )
-  (wire (pts (xy 278.13 89.535) (xy 278.13 90.805))
+  (wire (pts (xy 278.765 89.535) (xy 278.765 90.805))
     (stroke (width 0) (type default))
   )
@@
     (stroke (width 0) (type default))
   )
-  (wire (pts (xy 278.13 112.395) (xy 278.13 113.665))
-    (stroke (width 0) (type default))
-  )
   (wire (pts (xy 19.05 130.175) (xy 19.05 142.875))
     (stroke (width 0) (type default))
@@
     (stroke (width 0) (type default))
   )
-  (wire (pts (xy 264.795 107.315) (xy 263.525 107.315))
+  (wire (pts (xy 263.525 107.315) (xy 267.97 107.315))
     (stroke (width 0) (type default))
   )
@@
     (stroke (width 0) (type default))
   )
-  (wire (pts (xy 272.415 107.315) (xy 273.05 107.315))
-    (stroke (width 0) (type default))
-  )
   (wire (pts (xy 200.66 111.76) (xy 194.945 111.76))
     (stroke (width 0) (type default))
@@
     )
   )
+  (global_label "VIDEO" (shape input) (at 267.97 107.315 0) (fields_autoplaced)
+    (effects (font (size 1.27 1.27)) (justify left))
+    (property "Intersheetrefs" "${INTERSHEET_REFS}" (at 276.3981 107.315 0)
+      (effects (font (size 1.27 1.27)) (justify left) hide)
+    )
+  )
   (global_label "DAC_CLK" (shape input) (at 24.765 142.875 0) (fields_autoplaced)
     (effects (font (size 1.27 1.27)) (justify left))
@@
     )
   )
-  (symbol (lib_id "Device:R") (at 268.605 107.315 90) (unit 1)
-    (in_bom yes) (on_board yes) (dnp no)
-    (property "Reference" "R18" (at 268.605 109.855 90)
-      (effects (font (size 1.27 1.27)))
-    )
-    (property "Value" "75" (at 268.605 107.315 90)
-      (effects (font (size 1.27 1.27)))
-    )
-    (property "Footprint" "Resistor_SMD:R_0603_1608Metric" (at 268.605 109.093 90)
-      (effects (font (size 1.27 1.27)) hide)
-    )
-    (property "Datasheet" "~" (at 268.605 107.315 0)
-      (effects (font (size 1.27 1.27)) hide)
-    )
-    (pin "2")
-    (pin "1")
-    (instances
-      (project "dacattac-alpha"
-        (path "/487245ca-0c1f-4f9d-bc99-20c8f558090f/b4bbface-dd1a-4873-ab51-f35caad404be"
-          (reference "R18") (unit 1)
-        )
-        (path "/487245ca-0c1f-4f9d-bc99-20c8f558090f/e1e307fe-d49b-45b6-b177-774a7a482979"
-          (reference "R76") (unit 1)
-        )
-      )
-    )
-  )
   (symbol (lib_id "Device:R") (at 78.74 109.22 0) (unit 1)
     (in_bom yes) (on_board yes) (dnp no)
@@
     )
   )
-  (symbol (lib_id "Connector:Conn_Coaxial") (at 278.13 84.455 0) (unit 1)
+  (symbol (lib_id "Connector:Conn_Coaxial") (at 278.765 84.455 0) (unit 1)
     (in_bom yes) (on_board yes) (dnp no)
-    (property "Reference" "J2" (at 276.225 78.105 0)
+    (property "Reference" "J2" (at 276.86 78.105 0)
       (effects (font (size 1.27 1.27)) (justify left))
     )
-    (property "Value" "VIDEO OUT1" (at 269.875 80.645 0)
+    (property "Value" "VIDEO OUT1" (at 270.51 80.645 0)
       (effects (font (size 1.27 1.27)) (justify left))
     )
-    (property "Footprint" "MOLEX_73101:731010120" (at 278.13 84.455 0)
+    (property "Footprint" "MOLEX_73101:731010120" (at 278.765 84.455 0)
       (effects (font (size 1.27 1.27)) hide)
     )
-    (property "Datasheet" " ~" (at 278.13 84.455 0)
+    (property "Datasheet" " ~" (at 278.765 84.455 0)
       (effects (font (size 1.27 1.27)) hide)
     )
@@
     )
   )
-  (symbol (lib_id "power:GNDA") (at 278.13 90.805 0) (unit 1)
+  (symbol (lib_id "power:GNDA") (at 278.765 90.805 0) (unit 1)
     (in_bom yes) (on_board yes) (dnp no)
-    (property "Reference" "#PWR041" (at 278.13 97.155 0)
+    (property "Reference" "#PWR041" (at 278.765 97.155 0)
       (effects (font (size 1.27 1.27)) hide)
     )
-    (property "Value" "GNDA" (at 278.13 94.615 0)
+    (property "Value" "GNDA" (at 278.765 94.615 0)
       (effects (font (size 1.27 1.27)))
     )
-    (property "Footprint" "" (at 278.13 90.805 0)
+    (property "Footprint" "" (at 278.765 90.805 0)
       (effects (font (size 1.27 1.27)) hide)
     )
-    (property "Datasheet" "" (at 278.13 90.805 0)
+    (property "Datasheet" "" (at 278.765 90.805 0)
       (effects (font (size 1.27 1.27)) hide)
     )
@@
     )
   )
-  (symbol (lib_id "Connector:Conn_Coaxial") (at 278.13 107.315 0) (unit 1)
-    (in_bom yes) (on_board yes) (dnp no)
-    (property "Reference" "J3" (at 275.59 100.965 0)
-      (effects (font (size 1.27 1.27)) (justify left))
-    )
-    (property "Value" "VIDEO OUT2" (at 269.875 103.505 0)
-      (effects (font (size 1.27 1.27)) (justify left))
-    )
-    (property "Footprint" "MOLEX_73101:731010120" (at 278.13 107.315 0)
-      (effects (font (size 1.27 1.27)) hide)
-    )
-    (property "Datasheet" " ~" (at 278.13 107.315 0)
-      (effects (font (size 1.27 1.27)) hide)
-    )
-    (pin "2")
-    (pin "1")
-    (instances
-      (project "dacattac-alpha"
-        (path "/487245ca-0c1f-4f9d-bc99-20c8f558090f/b4bbface-dd1a-4873-ab51-f35caad404be"
-          (reference "J3") (unit 1)
-        )
-        (path "/487245ca-0c1f-4f9d-bc99-20c8f558090f/e1e307fe-d49b-45b6-b177-774a7a482979"
-          (reference "J7") (unit 1)
-        )
-      )
-    )
-  )
   (symbol (lib_id "Device:R") (at 118.11 138.43 0) (unit 1)
     (in_bom yes) (on_board yes) (dnp no)
@@
     (in_bom yes) (on_board yes) (dnp no)
     (property "Reference" "R27" (at 265.43 125.095 0)
-      (effects (font (size 1.27 1.27)) (justify left))
+      (effects (font (size 1.27 1.27)) (justify left) hide)
     )
     (property "Value" "330" (at 263.525 127 90)
@@
         )
       )
-    )
-  )
-  (symbol (lib_id "power:GNDA") (at 278.13 113.665 0) (unit 1)
-    (in_bom yes) (on_board yes) (dnp no)
-    (property "Reference" "#PWR042" (at 278.13 120.015 0)
-      (effects (font (size 1.27 1.27)) hide)
-    )
-    (property "Value" "GNDA" (at 278.13 117.475 0)
-      (effects (font (size 1.27 1.27)))
-    )
-    (property "Footprint" "" (at 278.13 113.665 0)
-      (effects (font (size 1.27 1.27)) hide)
-    )
-    (property "Datasheet" "" (at 278.13 113.665 0)
-      (effects (font (size 1.27 1.27)) hide)
-    )
-    (pin "1")
-    (instances
-      (project "dacattac-alpha"
-        (path "/487245ca-0c1f-4f9d-bc99-20c8f558090f/b4bbface-dd1a-4873-ab51-f35caad404be"
-          (reference "#PWR042") (unit 1)
-        )
-        (path "/487245ca-0c1f-4f9d-bc99-20c8f558090f/e1e307fe-d49b-45b6-b177-774a7a482979"
-          (reference "#PWR0137") (unit 1)
-        )
-      )

Commit message: WIP
Parts:
- J2: value VIDEO OUT1 -> VIDEO OUT
Changed lines of the file:
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@@
       (effects (font (size 1.27 1.27)) (justify left))
     )
-    (property "Value" "VIDEO OUT1" (at 270.51 80.645 0)
+    (property "Value" "VIDEO OUT" (at 270.51 80.645 0)
       (effects (font (size 1.27 1.27)) (justify left))
     )

Commit message: WIP
Connections:
- net GNDA renamed GNDV

Commit message: WIP
Connections:
- net GNDV is gone; now on net GND: C16.2, C17.2, C21.2, C22.2, C23.2, C24.2, C25.2, C26.2, C27.2, C28.2, C32.2, C33.2, C35.2, C36.2, C39.2, C40.2, C43.2, C44.2, C45.2, C47.2, C48.2, C50.2, C69.2, C70.2, J2.2 (Ext), JP1.3 (B), L10.6, L11.6, L12.6, L13.6, L14.4, L14.6, L7.6, L8.6, L9.6, R1.2, R12.2, R15.2, R16.2, R22.2, R28.2, R3.2, R6.1, U4.28 (LADCOM), U4.5 (REFCOM), U5.3 (+)

Commit message: Added / updated BOm
Parts:
- L5, L6: value 5.6u -> 5u6
- R6: value R -> NF
Other:
- note removed: "C49: BFC280811229"
Changed lines of the file:
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@@
     (stroke (width 0) (type default))
-  )
-  (text "C49: BFC280811229" (at 212.725 158.75 0)
-    (effects (font (size 1.27 1.27)) (justify left bottom))
   )
   (text "LP FILTER" (at 198.12 60.96 0)
@@
       (effects (font (size 1.27 1.27)) (justify left))
     )
-    (property "Value" "5.6u" (at 80.01 66.675 0)
+    (property "Value" "5u6" (at 80.01 66.675 0)
       (effects (font (size 1.27 1.27)) (justify left))
     )
@@
       (effects (font (size 1.27 1.27)) (justify left))
     )
-    (property "Value" "5.6u" (at 86.995 140.335 90)
+    (property "Value" "5u6" (at 86.995 140.335 90)
       (effects (font (size 1.27 1.27)) (justify left))
     )
@@
       (effects (font (size 1.27 1.27)))
     )
-    (property "Value" "R" (at 99.06 106.68 90)
-      (effects (font (size 1.27 1.27)))
-    )
+    (property "Value" "NF" (at 99.06 106.68 90)
+      (effects (font (size 1.27 1.27)))
+    )
