File: hardware/alpha/video.kicad_sch (KiCad schematic)
At the start: 84 parts, among them J2 VIDEO OUT, U4 AD768, U5 MAX4104, U6 TLE2082, U7 MAX4104

Commit message: WIP
Connections:
- net VIDEO: no longer R27.1
- net at R19.2, R20.1, R24.1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: now also R27.1
Other:
- moved on the sheet: R24
Changed lines of the file:
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@@
   (junction (at 225.425 72.39) (diameter 0) (color 0 0 0 0)
   )
+  (junction (at 253.365 107.315) (diameter 0) (color 0 0 0 0)
+  )
   (junction (at 144.145 79.375) (diameter 0) (color 0 0 0 0)
   )
@@
     (stroke (width 0) (type default))
   )
-  (wire (pts (xy 252.73 107.315) (xy 248.92 107.315))
+  (wire (pts (xy 254.635 107.315) (xy 253.365 107.315))
     (stroke (width 0) (type default))
   )
@@
     (stroke (width 0) (type default))
   )
-  (wire (pts (xy 260.35 107.315) (xy 263.525 107.315))
+  (wire (pts (xy 262.255 107.315) (xy 263.525 107.315))
     (stroke (width 0) (type default))
   )
@@
     (stroke (width 0) (type default))
   )
+  (wire (pts (xy 253.365 107.315) (xy 248.92 107.315))
+    (stroke (width 0) (type default))
+  )
   (wire (pts (xy 93.98 132.08) (xy 93.98 134.62))
     (stroke (width 0) (type default))
@@
     (stroke (width 0) (type default))
   )
-  (wire (pts (xy 263.525 107.315) (xy 263.525 121.285))
-    (stroke (width 0) (type default))
-  )
   (wire (pts (xy 248.92 146.05) (xy 248.92 148.59))
     (stroke (width 0) (type default))
@@
     (stroke (width 0) (type default))
   )
+  (wire (pts (xy 263.525 120.015) (xy 253.365 120.015))
+    (stroke (width 0) (type default))
+  )
   (wire (pts (xy 252.73 138.43) (xy 254.635 138.43))
     (stroke (width 0) (type default))
@@
     (stroke (width 0) (type default))
   )
+  (wire (pts (xy 263.525 121.285) (xy 263.525 120.015))
+    (stroke (width 0) (type default))
+  )
   (wire (pts (xy 170.815 128.905) (xy 176.53 128.905))
     (stroke (width 0) (type default))
@@
     (stroke (width 0) (type default))
   )
+  (wire (pts (xy 253.365 120.015) (xy 253.365 107.315))
+    (stroke (width 0) (type default))
+  )
   (wire (pts (xy 175.895 59.69) (xy 179.705 59.69))
     (stroke (width 0) (type default))
@@
     )
   )
-  (symbol (lib_id "Device:R") (at 256.54 107.315 90) (unit 1)
+  (symbol (lib_id "Device:R") (at 258.445 107.315 90) (unit 1)
     (in_bom yes) (on_board yes) (dnp no)
-    (property "Reference" "R24" (at 256.54 104.775 90)
+    (property "Reference" "R24" (at 258.445 104.775 90)
       (effects (font (size 1.27 1.27)))
     )
-    (property "Value" "270" (at 256.54 107.315 90)
+    (property "Value" "270" (at 258.445 107.315 90)
       (effects (font (size 1.27 1.27)))
     )
-    (property "Footprint" "Resistor_SMD:R_0603_1608Metric" (at 256.54 109.093 90)
+    (property "Footprint" "Resistor_SMD:R_0603_1608Metric" (at 258.445 109.093 90)
       (effects (font (size 1.27 1.27)) hide)
     )
-    (property "Datasheet" "~" (at 256.54 107.315 0)
+    (property "Datasheet" "~" (at 258.445 107.315 0)
       (effects (font (size 1.27 1.27)) hide)
     )

Commit message: WIP
Changed lines of the file:
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@@
 	)
 	(symbol
-		(lib_name "KJL_ADJ:KJL_ADJ_SGL")
 		(lib_id "KJL_ADJ:KJL_ADJ_SGL")
 		(at 187.325 86.995 90)
@@
 		(on_board yes)
 		(dnp no)
-		(fields_autoplaced yes)
 		(property "Reference" "#PWR08"
 			(at 78.74 61.595 0)
@@
 		)
 		(property "Value" "+5V"
-			(at 78.74 52.705 0)
+			(at 78.74 53.34 0)
 			(effects
 				(font

Commit message: WIP
Parts:
- renumbered C13 to C1, C24 to C10, C25 to C11, C20 to C12, C19 to C13, C18 to C14, C26 to C15, C27 to C16, C29 to C17, C30 to C18, C31 to C19, C12 to C2, C28 to C20, C32 to C21, C33 to C22, C34 to C23, C35 to C24, C36 to C25, C37 to C26, C38 to C27, C39 to C28, C40 to C29, C14 to C3, C41 to C30, C42 to C31, C45 to C32, C70 to C33, C69 to C34, C48 to C35, C46 to C36, C49 to C37, C43 to C38, C44 to C39, C16 to C4, C47 to C40, C50 to C41, C15 to C5, C17 to C6, C21 to C7, C23 to C8, C22 to C9, J2 to J1, L5 to L1, L14 to L10, L6 to L2, L9 to L3, L7 to L4, L10 to L5, L8 to L6, L11 to L7, L12 to L8, L13 to L9, R8 to R1, R4 to R10, R5 to R11, R11 to R12, R14 to R13, R13 to R14, R23 to R15, R22 to R16, R21 to R17, R15 to R18, R20 to R19, R9 to R2, R16 to R20, R19 to R21, R25 to R22, R26 to R23, R27 to R25, R28 to R26, R17 to R27, R1 to R3, R7 to R4, R6 to R5, R12 to R6, R10 to R7, R2 to R8, R3 to R9, U4 to U1, U5 to U2, U6 to U3, U7 to U4
