File: hardware/alpha/video.kicad_sch (KiCad schematic)
At the start: 84 parts, among them J1 VIDEO OUT, U1 AD768, U2 MAX4104, U3 TLE2082, U4 MAX4104

Commit message: WIP
Connections:
- net ADAC+: now reaches C1.2, C2.2, L1.2, U1.25 (VCC)
- net ADAC-: now reaches C3.2, C4.1, C5.1, C6.1, L2.1, U1.26 (VEE)
Changed lines of the file:
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@@
+		)
+	)
+	(label "ADAC+"
+		(at 73.66 80.01 90)
+		(fields_autoplaced yes)
+		(effects
+			(font
+				(size 1.27 1.27)
+			)
+			(justify left bottom)
 		)
 	)
@@
 		(fields_autoplaced yes)
 		(effects
+			(font
+				(size 1.27 1.27)
+			)
+			(justify left bottom)
+		)
+	)
+	(label "ADAC-"
+		(at 73.025 122.555 0)
+		(fields_autoplaced yes)
+		(effects
