File: hardware/alpha/dacattac-alpha.kicad_pcb (KiCad board)
At the start: 4 copper layers, 120 x 75 mm, 13 parts, among them J4 MOUNTING_HOLE, J5 MOUNTING_HOLE, J6 MOUNTING_HOLE, J7 MOUNTING_HOLE, J8 MOUNTING_HOLE, J9 MOUNTING_HOLE, P20 GPIO, P22 I2S, P28 SD, P30 BANK2_AUX, P9 BASEBAND

Commit message: WIP
Parts:
- removed J5: MOUNTING_HOLE, hackrf:GSG-HOLE126MIL-COPPER
- removed P9: BASEBAND, hackrf:GSG-HEADER-2x8
- added C1: 100n, Capacitor_SMD:C_0603_1608Metric, F.Cu at (-16.6, 24.7)
- added C11: 100n, Capacitor_SMD:C_0603_1608Metric, F.Cu at (-77.3, 38.6)
- added C12: 100n, Capacitor_SMD:C_0603_1608Metric, F.Cu at (-77.3, 41.1)
- added C13: 100n, Capacitor_SMD:C_0603_1608Metric, F.Cu at (-77.3, 43.6)
- added C14: 100n, Capacitor_SMD:C_0603_1608Metric, F.Cu at (-77.3, 46.1)
- added C15: 100n, Capacitor_SMD:C_0603_1608Metric, F.Cu at (-77.3, 48.6)
- added C16: 100n, Capacitor_SMD:C_0603_1608Metric, F.Cu at (-77.3, 51.1)
- added C17: 100n, Capacitor_SMD:C_0603_1608Metric, F.Cu at (-77.3, 53.6)
- added C18: 100p, Capacitor_SMD:C_0603_1608Metric, F.Cu at (-77.3, 56.1)
- added C19: 82p, Capacitor_SMD:C_0603_1608Metric, F.Cu at (-77.3, 58.7)
- added C2: 100n, Capacitor_SMD:C_0603_1608Metric, F.Cu at (-16.6, 27.2)
- added C20: 100p, Capacitor_SMD:C_0603_1608Metric, F.Cu at (-77.3, 61.2)
- added C21: 100n, Capacitor_SMD:C_0603_1608Metric, F.Cu at (-77.3, 63.7)
- added C22: 100n, Capacitor_SMD:C_0603_1608Metric, F.Cu at (-77.3, 66.2)
- added C23: 100n, Capacitor_SMD:C_0603_1608Metric, F.Cu at (-73.2, 38.6)
- added C24: 1n, Capacitor_SMD:C_0603_1608Metric, F.Cu at (-73.2, 41.1)
- added C25: 560p, Capacitor_SMD:C_0603_1608Metric, F.Cu at (-73.2, 43.6)
- added C26: 680p, Capacitor_SMD:C_0603_1608Metric, F.Cu at (-73.2, 46.1)
- added C27: 2n2, Capacitor_SMD:C_0603_1608Metric, F.Cu at (-73.2, 48.6)
- added C28: 1n, Capacitor_SMD:C_0603_1608Metric, F.Cu at (-73.2, 51.1)
- added C29: 100p, Capacitor_SMD:C_0603_1608Metric, F.Cu at (-73.2, 53.6)
- added C3: 100n, Capacitor_SMD:C_0603_1608Metric, F.Cu at (-16.6, 29.7)
- added C30: 100p, Capacitor_SMD:C_0603_1608Metric, F.Cu at (-73.2, 56.1)
- added C31: 100p, Capacitor_SMD:C_0603_1608Metric, F.Cu at (-73.2, 58.7)
- added C32: 220p, Capacitor_SMD:C_0603_1608Metric, F.Cu at (-73.2, 61.2)
- added C33: 82p, Capacitor_SMD:C_0603_1608Metric, F.Cu at (-73.2, 63.7)
- added C34: 56p, Capacitor_SMD:C_0603_1608Metric, F.Cu at (-73.2, 66.2)
- added C35: 390p, Capacitor_SMD:C_0603_1608Metric, F.Cu at (-69.2, 38.6)
- added C36: 220p, Capacitor_SMD:C_0603_1608Metric, F.Cu at (-69.2, 41.1)
- added C37: NF, Capacitor_SMD:C_0603_1608Metric, F.Cu at (-69.2, 43.6)
- added C38: 270p, Capacitor_SMD:C_0603_1608Metric, F.Cu at (-69.2, 46.1)
- added C39: 560p, Capacitor_SMD:C_0603_1608Metric, F.Cu at (-69.2, 48.6)
- added C4: 100n, Capacitor_SMD:C_0603_1608Metric, F.Cu at (-16.6, 32.2)
- added C40: 100p, Capacitor_SMD:C_0603_1608Metric, F.Cu at (-69.2, 51.1)
- added C41: 18p, Capacitor_SMD:C_0603_1608Metric, F.Cu at (-69.2, 53.6)
- added C42: 220p, Capacitor_SMD:C_0603_1608Metric, F.Cu at (-69.2, 56.1)
- added C43: 100n, Capacitor_SMD:C_0603_1608Metric, F.Cu at (-69.2, 58.7)
- added C44: 100n, Capacitor_SMD:C_0603_1608Metric, F.Cu at (-69.2, 61.2)
- added C45: 100n, Capacitor_SMD:C_0603_1608Metric, F.Cu at (-69.2, 63.7)
- added C46: 47p, Capacitor_SMD:C_0603_1608Metric, F.Cu at (-69.2, 66.2)
- added C47: 390p, Capacitor_SMD:C_0603_1608Metric, F.Cu at (-65.2, 38.6)
- added C48: 4p7, Capacitor_SMD:C_0603_1608Metric, F.Cu at (-65.2, 41.1)
- added C49: 2p-18p, BFC2808xxxxx:BFC2808xxxxx, F.Cu at (-38.5, 41.1)
- added C5: 100n, Capacitor_SMD:C_0603_1608Metric, F.Cu at (-16.6, 34.7)
- added C50: 560p, Capacitor_SMD:C_0603_1608Metric, F.Cu at (-65.2, 43.6)
- added C51: 2n2, Capacitor_SMD:C_0603_1608Metric, F.Cu at (-30.6, 55.8)
- added C52: 2n2, Capacitor_SMD:C_0603_1608Metric, F.Cu at (-30.6, 58.3)
- added C53: 2u2, Capacitor_SMD:C_0603_1608Metric, F.Cu at (-30.6, 60.8)
- added C54: 100n, Capacitor_SMD:C_0603_1608Metric, F.Cu at (-30.6, 63.3)
- added C55: 10uF, Capacitor_SMD:C_0603_1608Metric, F.Cu at (-30.6, 65.8)
- added C56: 2u2, Capacitor_SMD:C_0603_1608Metric, F.Cu at (-30.6, 68.3)
- added C57: 100n, Capacitor_SMD:C_0603_1608Metric, F.Cu at (-30.6, 70.8)
- added C58: 100n, Capacitor_SMD:C_0603_1608Metric, F.Cu at (-26.6, 55.8)
- added C59: 100n, Capacitor_SMD:C_0603_1608Metric, F.Cu at (-26.6, 58.3)
- added C6: 100n, Capacitor_SMD:C_0603_1608Metric, F.Cu at (-16.6, 37.2)
- added C60: 2u2, Capacitor_SMD:C_0603_1608Metric, F.Cu at (-26.6, 60.8)
- added C61: 2u2, Capacitor_SMD:C_0603_1608Metric, F.Cu at (-26.6, 63.3)
- added C62: 10n, Capacitor_SMD:C_0603_1608Metric, F.Cu at (-77.3, 70.7)
- added C63: 10u, Capacitor_SMD:C_0603_1608Metric, F.Cu at (-77.3, 73.2)
- added C64: 4.7u, Capacitor_SMD:C_0603_1608Metric, F.Cu at (-77.3, 75.7)
- added C65: 4n7, Capacitor_SMD:C_0603_1608Metric, F.Cu at (-77.3, 78.2)
- added C66: 220n, Capacitor_SMD:C_0603_1608Metric, F.Cu at (-77.3, 80.7)
- added C67: C, Capacitor_SMD:C_0603_1608Metric, F.Cu at (-73.2, 70.7)
- added C68: 10u, Capacitor_SMD:C_0603_1608Metric, F.Cu at (-73.2, 73.2)
- added C69: NF, Capacitor_SMD:C_0603_1608Metric, F.Cu at (-65.2, 46.1)
- added C70: 180p, Capacitor_SMD:C_0603_1608Metric, F.Cu at (-65.2, 48.6)
- added C71: 100n, Capacitor_SMD:C_0603_1608Metric, F.Cu at (-12.6, 24.7)
- added C72: 100n, Capacitor_SMD:C_0603_1608Metric, F.Cu at (-12.6, 27.2)
- added C73: 100n, Capacitor_SMD:C_0603_1608Metric, F.Cu at (-12.6, 29.7)
- added C74: 100n, Capacitor_SMD:C_0603_1608Metric, F.Cu at (-12.6, 32.2)
- added C77: 100n, Capacitor_SMD:C_0603_1608Metric, F.Cu at (-12.6, 34.7)
- added C78: 100n, Capacitor_SMD:C_0603_1608Metric, F.Cu at (-12.6, 37.2)
- added C84: 33u, Capacitor_SMD:C_1210_3225Metric, F.Cu at (-5.32, 40.6)
- added C85: 33u, Capacitor_SMD:C_1210_3225Metric, F.Cu at (-5.32, 44.9)
- added C87: 100n, Capacitor_SMD:C_0603_1608Metric, F.Cu at (-8.57, 24.7)
- added C88: 100n, Capacitor_SMD:C_0603_1608Metric, F.Cu at (-8.57, 27.2)
- added D1: MBR0540T1, Diode_SMD:D_SOD-123, F.Cu at (-64.3, 86.0)
- added D2: MBR0540T1, Diode_SMD:D_SOD-123, F.Cu at (-64.3, 89.3)
- added J1: EXT +/- 8V, Connector_Molex:Molex_KK-254_AE-6410-03A_1x03_P2.54mm_Vertical, F.Cu at (-77.0, 85.9)
- added JP1: TEST, Connector_PinHeader_2.54mm:PinHeader_1x03_P2.54mm_Vertical, F.Cu at (-44.4, 59.9)
- added JP2: FILTER MODE, Jumper:SolderJumper-3_P1.3mm_Open_Pad1.0x1.5mm, F.Cu at (-12.9, 56.3)
- added JP3: DE EMPHASIS, Jumper:SolderJumper-3_P1.3mm_Open_Pad1.0x1.5mm, F.Cu at (-12.9, 60.1)
- added L10: 09760, NEOSID_7MM:NEOSID_7MM, F.Cu at (-49.2, 21.6)
- added L11: 09750, NEOSID_7MM:NEOSID_7MM, F.Cu at (-40.6, 21.6)
- added L12: 09750, NEOSID_7MM:NEOSID_7MM, F.Cu at (-75.0, 32.1)
- added L13: 09750, NEOSID_7MM:NEOSID_7MM, F.Cu at (-66.4, 32.1)
- added L14: 09500, NEOSID_7MM:NEOSID_7MM, F.Cu at (-57.8, 32.1)
- added L15: 10u, Inductor_SMD:L_1210_3225Metric, F.Cu at (-64.4, 78.0)
- added L16: 4u7, Inductor_SMD:L_1210_3225Metric, F.Cu at (-64.4, 82.2)
- added L17: 5.6u, Inductor_SMD:L_1210_3225Metric, F.Cu at (-21.4, 25.5)
- added L18: 5.6u, Inductor_SMD:L_1210_3225Metric, F.Cu at (-21.4, 29.7)
- added L21: 5.6u, Inductor_SMD:L_1210_3225Metric, F.Cu at (-21.4, 33.9)
- added L22: 5.6u, Inductor_SMD:L_1210_3225Metric, F.Cu at (-21.4, 38.1)
- added L5: 5.6u, Inductor_SMD:L_1210_3225Metric, F.Cu at (-39.5, 47.0)
- added L6: 5.6u, Inductor_SMD:L_1210_3225Metric, F.Cu at (-39.5, 51.2)
- added L7: 09510, NEOSID_7MM:NEOSID_7MM, F.Cu at (-75.0, 21.6)
- added L8: 09770, NEOSID_7MM:NEOSID_7MM, F.Cu at (-66.4, 21.6)
- added L9: 09760, NEOSID_7MM:NEOSID_7MM, F.Cu at (-57.8, 21.6)
- added Q1: 2N7002, Package_TO_SOT_SMD:SOT-23, F.Cu at (-18.2, 56.8)
- added Q2: 2N7002, Package_TO_SOT_SMD:SOT-23, F.Cu at (-18.2, 61.2)
- added Q3: IRF7324, Package_SO:SOIC-8_3.9x4.9mm_P1.27mm, F.Cu at (-63.0, 72.7)
- added R1: 33, Resistor_SMD:R_0603_1608Metric, F.Cu at (-65.2, 51.1)
- added R10: 75, Resistor_SMD:R_0603_1608Metric, F.Cu at (-61.2, 43.6)
- added R11: 330, Resistor_SMD:R_0603_1608Metric, F.Cu at (-61.2, 46.1)
- added R12: 68, Resistor_SMD:R_0603_1608Metric, F.Cu at (-61.2, 48.6)
- added R13: 100, Resistor_SMD:R_0603_1608Metric, F.Cu at (-61.2, 51.1)
- added R14: 100, Resistor_SMD:R_0603_1608Metric, F.Cu at (-61.2, 53.6)
- added R15: 100, Resistor_SMD:R_0603_1608Metric, F.Cu at (-61.2, 56.1)
- added R16: 100, Resistor_SMD:R_0603_1608Metric, F.Cu at (-61.2, 58.7)
- added R17: 75, Resistor_SMD:R_0603_1608Metric, F.Cu at (-61.2, 61.2)
- added R18: 75, Resistor_SMD:R_0603_1608Metric, F.Cu at (-61.2, 63.7)
- added R19: 1k8, Resistor_SMD:R_0603_1608Metric, F.Cu at (-61.2, 66.2)
- added R2: 3k9, Resistor_SMD:R_0603_1608Metric, F.Cu at (-65.2, 53.6)
- added R20: 4k7, Resistor_SMD:R_0603_1608Metric, F.Cu at (-57.2, 38.6)
- added R21: 1k, Resistor_SMD:R_0603_1608Metric, F.Cu at (-57.2, 41.1)
- added R22: 2k2, Resistor_SMD:R_0603_1608Metric, F.Cu at (-57.2, 43.6)
- added R23: 10, Resistor_SMD:R_0603_1608Metric, F.Cu at (-57.2, 46.1)
- added R24: 270, Resistor_SMD:R_0603_1608Metric, F.Cu at (-57.2, 48.6)
- added R25: 3k3, Resistor_SMD:R_0603_1608Metric, F.Cu at (-57.2, 51.1)
- added R26: 180, Resistor_SMD:R_0603_1608Metric, F.Cu at (-57.2, 53.6)
- added R27: 330, Resistor_SMD:R_0603_1608Metric, F.Cu at (-57.2, 56.1)
- added R28: 100, Resistor_SMD:R_0603_1608Metric, F.Cu at (-57.2, 58.7)
- added R29: 470, Resistor_SMD:R_0603_1608Metric, F.Cu at (-26.6, 65.8)
- added R3: 10k, Resistor_SMD:R_0603_1608Metric, F.Cu at (-65.2, 56.1)
- added R30: 470, Resistor_SMD:R_0603_1608Metric, F.Cu at (-26.6, 68.3)
- added R32: 10k, Resistor_SMD:R_0603_1608Metric, F.Cu at (-26.6, 70.8)
- added R33: 18k, Resistor_SMD:R_0603_1608Metric, F.Cu at (-22.6, 55.8)
- added R34: 0, Resistor_SMD:R_0603_1608Metric, F.Cu at (-22.6, 58.3)
- added R35: 0, Resistor_SMD:R_0603_1608Metric, F.Cu at (-22.6, 60.8)
- added R36: NF, Resistor_SMD:R_0603_1608Metric, F.Cu at (-22.6, 63.3)
- added R37: 0, Resistor_SMD:R_0603_1608Metric, F.Cu at (-22.6, 65.8)
- added R38: R, Resistor_SMD:R_0603_1608Metric, F.Cu at (-73.2, 75.7)
- added R39: R, Resistor_SMD:R_0603_1608Metric, F.Cu at (-73.2, 78.2)
- added R4: 100, Resistor_SMD:R_0603_1608Metric, F.Cu at (-65.2, 58.7)
- added R40: 4k99, Resistor_SMD:R_0603_1608Metric, F.Cu at (-73.2, 80.7)
- added R41: R, Resistor_SMD:R_0603_1608Metric, F.Cu at (-69.2, 70.7)
- added R42: R, Resistor_SMD:R_0603_1608Metric, F.Cu at (-69.2, 73.2)
- added R45: R, Resistor_SMD:R_0603_1608Metric, F.Cu at (-69.2, 75.7)
- added R46: 0, Resistor_SMD:R_1210_3225Metric, F.Cu at (-21.4, 42.4)
- added R5: 3k3, Resistor_SMD:R_0603_1608Metric, F.Cu at (-65.2, 61.2)
- added R6: R, Resistor_SMD:R_0603_1608Metric, F.Cu at (-65.2, 63.7)
- added R61: 2k2, Resistor_SMD:R_0603_1608Metric, F.Cu at (-8.57, 29.7)
- added R62: 2k2, Resistor_SMD:R_0603_1608Metric, F.Cu at (-8.57, 32.2)
- added R7: 330, Resistor_SMD:R_0603_1608Metric, F.Cu at (-65.2, 66.2)
- added R8: 470, Resistor_SMD:R_0603_1608Metric, F.Cu at (-61.2, 38.6)
- added R9: 33, Resistor_SMD:R_0603_1608Metric, F.Cu at (-61.2, 41.1)
- added U1: 74LVCH16T245, Package_TO_SOT_SMD:SOT-23-6, F.Cu at (-5.57, 49.2)
- added U10: MCP1700x-120xxMB, Package_TO_SOT_SMD:SOT-89-3, F.Cu at (-17.2, 74.5)
- added U13: L78L05_SO8, Package_SO:SOIC-8_3.9x4.9mm_P1.27mm, F.Cu at (-28.4, 26.6)
- added U14: L79L05_SO8, Package_SO:SOIC-8_3.9x4.9mm_P1.27mm, F.Cu at (-28.4, 33.1)
- added U16: TLE2082, Package_SO:SOIC-8_3.9x4.9mm_P1.27mm, F.Cu at (-28.4, 39.5)
- added U17: MCP47FEB22A0-E/ST, Package_SO:SOIC-8_3.9x4.9mm_P1.27mm, F.Cu at (-28.4, 46.0)
- added U3: 74LVC1T45, Package_SO:TSSOP-48_6.1x12.5mm_P0.5mm, F.Cu at (168.8, 77.0)
- added U4: AD768, Package_SO:SOIC-28W_7.5x18.7mm_P1.27mm, F.Cu at (-48.2, 46.8)
- added U5: MAX4104, Package_TO_SOT_SMD:SOT-23-5, F.Cu at (-39.5, 59.8)
- added U6: TLE2082, Package_SO:SOIC-8_3.9x4.9mm_P1.27mm, F.Cu at (-51.0, 60.8)
- added U7: MAX4104, Package_TO_SOT_SMD:SOT-23-5, F.Cu at (-39.5, 64.2)
- added U9: PCM5102, Package_SO:TSSOP-20_4.4x6.5mm_P0.65mm, F.Cu at (-16.2, 67.5)
- P20: value GPIO -> P20
- P22: value I2S -> P22
Connections:
- net /mcu/usb/power/B2AUX1 renamed /video-misc/LAD15
- net /mcu/usb/power/B2AUX10 renamed /video-misc/LAD6
- net /mcu/usb/power/B2AUX11 renamed /video-misc/LAD5
- net /mcu/usb/power/B2AUX12 renamed /video-misc/LAD4
- net /mcu/usb/power/B2AUX13 renamed /video-misc/LAD3
- net /mcu/usb/power/B2AUX14 renamed /video-misc/LAD2
- net /mcu/usb/power/B2AUX15 renamed /video-misc/LAD1
- net /mcu/usb/power/B2AUX16 renamed /video-misc/LAD0
- net /mcu/usb/power/B2AUX2 renamed /video-misc/LAD14
- net /mcu/usb/power/B2AUX3 renamed /video-misc/LAD13
- net /mcu/usb/power/B2AUX4 renamed /video-misc/LAD12
- net /mcu/usb/power/B2AUX5 renamed /video-misc/LAD11
- net /mcu/usb/power/B2AUX6 renamed /video-misc/LAD10
- net /mcu/usb/power/B2AUX7 renamed /video-misc/LAD9
- net /mcu/usb/power/B2AUX8 renamed /video-misc/LAD8
- net /mcu/usb/power/B2AUX9 renamed /video-misc/LAD7
- P20 pad 1: /mcu/usb/power/VBAT -> unconnected-(P20-Pin_1-Pad1)
- P20 pad 10: /mcu/usb/power/GPIO3_13 -> unconnected-(P20-Pin_10-Pad10)
- P20 pad 11: /mcu/usb/power/GPIO3_14 -> unconnected-(P20-Pin_11-Pad11)
- P20 pad 12: /mcu/usb/power/GPIO3_15 -> unconnected-(P20-Pin_12-Pad12)
- P20 pad 13: GND -> unconnected-(P20-Pin_13-Pad13)
- P20 pad 14: /mcu/usb/power/ADC0_6 -> unconnected-(P20-Pin_14-Pad14)
- P20 pad 15: GND -> unconnected-(P20-Pin_15-Pad15)
- P20 pad 16: /mcu/usb/power/ADC0_2 -> unconnected-(P20-Pin_16-Pad16)
- P20 pad 17: /mcu/usb/power/VBUSCTRL -> /power/VBUSCTRL
- P20 pad 18: /mcu/usb/power/ADC0_5 -> unconnected-(P20-Pin_18-Pad18)
- P20 pad 19: GND -> unconnected-(P20-Pin_19-Pad19)
- P20 pad 2: /mcu/usb/power/RTC_ALARM -> unconnected-(P20-Pin_2-Pad2)
- P20 pad 20: /mcu/usb/power/ADC0_0 -> unconnected-(P20-Pin_20-Pad20)
- P20 pad 21: /mcu/usb/power/VBUS -> /power/VBUS
- P20 pad 22: /mcu/usb/power/VIN -> unconnected-(P20-Pin_22-Pad22)
- P20 pad 3: VCC -> unconnected-(P20-Pin_3-Pad3)
- P20 pad 4: /mcu/usb/power/WAKEUP -> unconnected-(P20-Pin_4-Pad4)
- P20 pad 5: /mcu/usb/power/GPIO3_8 -> unconnected-(P20-Pin_5-Pad5)
- P20 pad 6: /mcu/usb/power/GPIO3_9 -> unconnected-(P20-Pin_6-Pad6)
- P20 pad 7: /mcu/usb/power/GPIO3_10 -> unconnected-(P20-Pin_7-Pad7)
- P20 pad 8: /mcu/usb/power/GPIO3_11 -> unconnected-(P20-Pin_8-Pad8)
- P20 pad 9: /mcu/usb/power/GPIO3_12 -> unconnected-(P20-Pin_9-Pad9)
- P22 pad 1: CLKOUT -> unconnected-(P22-Pin_1-Pad1)
- P22 pad 11: VCC -> +3.3VP
- P22 pad 12: /mcu/usb/power/I2S0_RX_SCK -> unconnected-(P22-Pin_12-Pad12)
- P22 pad 13: /mcu/usb/power/I2S0_RX_SDA -> /audio/I2S_SDA
- P22 pad 14: /mcu/usb/power/I2S0_RX_MCLK -> unconnected-(P22-Pin_14-Pad14)
- P22 pad 15: /mcu/usb/power/I2S0_RX_WS -> /audio/I2S_WS
- P22 pad 16: /mcu/usb/power/I2S0_TX_SCK -> /audio/I2S_SCK
- P22 pad 17: /mcu/usb/power/I2S0_TX_MCLK -> unconnected-(P22-Pin_17-Pad17)
- P22 pad 19: /mcu/usb/power/U0_RXD -> unconnected-(P22-Pin_19-Pad19)
- P22 pad 2: CLKIN -> unconnected-(P22-Pin_2-Pad2)
- P22 pad 20: /mcu/usb/power/U0_TXD -> unconnected-(P22-Pin_20-Pad20)
- P22 pad 21: /mcu/usb/power/P2_9 -> unconnected-(P22-Pin_21-Pad21)
- P22 pad 22: /mcu/usb/power/P2_13 -> unconnected-(P22-Pin_22-Pad22)
- P22 pad 23: /mcu/usb/power/P2_8 -> unconnected-(P22-Pin_23-Pad23)
- P22 pad 24: SDA -> /audio/SDA
- P22 pad 25: CLK6 -> unconnected-(P22-Pin_25-Pad25)
- P22 pad 26: SCL -> /audio/SCL
- P22 pad 3: /mcu/usb/power/RESET -> unconnected-(P22-Pin_3-Pad3)
- P22 pad 5: /mcu/usb/power/I2C1_SCL -> unconnected-(P22-Pin_5-Pad5)
- P22 pad 6: /mcu/usb/power/I2C1_SDA -> unconnected-(P22-Pin_6-Pad6)
- P22 pad 7: /mcu/usb/power/SPIFI_CIPO -> unconnected-(P22-Pin_7-Pad7)
- P22 pad 8: /mcu/usb/power/SPIFI_SCK -> unconnected-(P22-Pin_8-Pad8)
- P22 pad 9: /mcu/usb/power/SPIFI_COPI -> unconnected-(P22-Pin_9-Pad9)
- P30 pad 1: VCC -> +3.3VP
- P30 pad 19: /mcu/usb/power/GCK0 -> /video-misc/LCLK

Commit message: WIP
Parts:
- added J10: HOLE, hackrf:GSG-HOLE126MIL-COPPER, F.Cu at (83.7, 67.7)
- added J11: HOLE, hackrf:GSG-HOLE126MIL-COPPER, F.Cu at (83.7, 134.7)
- added J2: VIDEO OUT1, MOLEX_73101:731010120, F.Cu at (79.7, 96.3)
- added J3: VIDEO OUT2, MOLEX_73101:731010120, F.Cu at (79.7, 78.3)
- added J5: 5V I2C, Connector_Molex:Molex_KK-254_AE-6410-04A_1x04_P2.54mm_Vertical, F.Cu at (-38.8, 93.6)
- added J5: 5V I2C, Connector_Molex:Molex_KK-254_AE-6410-04A_1x04_P2.54mm_Vertical, F.Cu at (105.2, 129.6)
- added U11: TPS63700DRCT, TPS63700DRCT:VREG_V62_16624-01YE, F.Cu at (-17.4, 108.0)
- added U2: TPS61170DRVR, TPS61170DRVR:SON65P200X200X80-7N, F.Cu at (-17.8, 112.2)
- J12: renamed from J8; value MOUNTING_HOLE -> HOLE
- J13: renamed from J9; value MOUNTING_HOLE -> HOLE
- J14: renamed from J7; value MOUNTING_HOLE -> HOLE
- J15: renamed from J6; value MOUNTING_HOLE -> HOLE
- J4: value MOUNTING_HOLE -> AUDIO_OUT; footprint hackrf:GSG-HOLE126MIL-COPPER -> PJRAN2X1U01X:PJRAN2X1U01X
- U1: footprint Package_TO_SOT_SMD:SOT-23-6 -> Package_SO:TSSOP-48_6.1x12.5mm_P0.5mm
- U17: footprint Package_SO:SOIC-8_3.9x4.9mm_P1.27mm -> Package_SO:TSSOP-8_3x3mm_P0.65mm
- U3: footprint Package_SO:TSSOP-48_6.1x12.5mm_P0.5mm -> Package_TO_SOT_SMD:SOT-23-6
- moved C21 208.3 mm to (130.7, 75.2), turned to 90 degrees
- moved C2 202.8 mm to (174.9, 93.8)
- moved U4 199.7 mm to (148.4, 81.6)
- moved C1 198.7 mm to (174.9, 77.8)
- moved R3 198.1 mm to (132.2, 72.2)
- moved C4 195.0 mm to (168.4, 93.8), turned to 180 degrees
- moved R2 194.9 mm to (128.7, 72.8)
- moved R6 194.0 mm to (128.7, 68.8), turned to 180 degrees
- moved R7 194.0 mm to (128.7, 70.8), turned to 180 degrees
- moved R5 193.5 mm to (127.7, 75.2), turned to -90 degrees
- moved C3 191.2 mm to (168.4, 77.8)
- moved R4 191.2 mm to (125.2, 75.2), turned to 90 degrees
- moved C45 190.8 mm to (121.2, 75.0), turned to -90 degrees
- moved C41 188.1 mm to (116.2, 85.2), turned to 90 degrees
- moved C42 187.0 mm to (116.2, 80.2), turned to -90 degrees
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Connections:
- net DAC_AD0 renamed AD0
- net DAC_AD1 renamed AD1
- net DAC_AD2 renamed AD2
- net DAC_AD3 renamed AD3
- J4 pad 1: GND -> Net-(J4-IN1)
- L10 pad 1: GNDA -> Net-(L10-Pad1)
- L10 pad 6: (no net) -> GNDA
- L11 pad 1: GNDA -> Net-(C29-Pad2)
- L11 pad 6: (no net) -> GNDA
- L12 pad 1: GNDA -> Net-(C34-Pad2)
- L12 pad 6: (no net) -> GNDA
- L13 pad 1: GNDA -> Net-(C37-Pad2)
- L13 pad 6: (no net) -> GNDA
- L14 pad 1: GNDA -> Net-(C46-Pad2)
- L14 pad 6: (no net) -> GNDA
- L7 pad 1: GNDA -> Net-(JP1-C)
- L7 pad 6: (no net) -> GNDA
- L8 pad 1: GNDA -> Net-(C18-Pad2)
- L8 pad 6: (no net) -> GNDA
- L9 pad 1: GNDA -> Net-(L7-Pad2)
- L9 pad 6: (no net) -> GNDA
- P30 pad 10: /video-misc/LAD7 -> /video-misc/LAD9
- P30 pad 11: /video-misc/LAD8 -> /video-misc/LAD6
- P30 pad 12: /video-misc/LAD9 -> /video-misc/LAD7
- P30 pad 13: /video-misc/LAD10 -> /video-misc/LAD4
- P30 pad 14: /video-misc/LAD11 -> /video-misc/LAD5
- P30 pad 15: /video-misc/LAD12 -> /video-misc/LAD2
- P30 pad 16: /video-misc/LAD13 -> /video-misc/LAD3
- P30 pad 17: /video-misc/LAD14 -> /video-misc/LAD0
- P30 pad 18: /video-misc/LAD15 -> /video-misc/LAD1
- P30 pad 3: /video-misc/LAD0 -> /video-misc/LAD14
- P30 pad 4: /video-misc/LAD1 -> /video-misc/LAD15
- P30 pad 5: /video-misc/LAD2 -> /video-misc/LAD12
- P30 pad 6: /video-misc/LAD3 -> /video-misc/LAD13
- P30 pad 7: /video-misc/LAD4 -> /video-misc/LAD10
- P30 pad 8: /video-misc/LAD5 -> /video-misc/LAD11
- P30 pad 9: /video-misc/LAD6 -> /video-misc/LAD8
- U4 pad 11: DAC_AD4 -> AD4
- U4 pad 12: DAC_AD5 -> AD5
- U4 pad 13: DAC_AD6 -> AD6
- U4 pad 14: DAC_AD7 -> AD7
- U4 pad 17: DAC_AD8 -> AD8
- U4 pad 18: DAC_AD9 -> AD9
- U4 pad 19: DAC_AD10 -> AD10
- U4 pad 20: DAC_AD11 -> AD11
- U4 pad 21: DAC_AD12 -> AD12
- U4 pad 22: DAC_AD13 -> AD13
- U4 pad 23: DAC_AD14 -> AD14
- U4 pad 24: DAC_AD15 -> AD15
Routing:
- net Net-(U7-+): track 0.00 -> 1.58 mm
Other:
- board text removed: "P16 CLKIN"
- board text removed: "P2 CLKOUT"
- board text removed: "P80 SHIELD"

Commit message: WIP
Parts:
- moved C26 211.6 mm to (131.9, 98.1)
- moved C27 211.5 mm to (131.9, 99.9)
- moved C28 211.3 mm to (131.9, 101.7)
- moved C24 210.4 mm to (131.9, 88.0)
- moved C25 210.3 mm to (131.9, 89.7)
- moved C23 207.1 mm to (129.9, 78.8)
- moved L7 204.8 mm to (117.7, 91.0), turned to 180 degrees
- moved C22 200.6 mm to (122.5, 84.6), turned to 180 degrees
- moved L8 200.5 mm to (117.7, 101.1), turned to 180 degrees
- moved L9 196.5 mm to (126.0, 91.0), turned to 180 degrees
- moved C18 193.0 mm to (112.6, 91.0), turned to -90 degrees
- moved L10 192.4 mm to (126.0, 101.1), turned to 180 degrees
- moved R10 192.2 mm to (127.1, 82.1), turned to 180 degrees
- moved R12 191.6 mm to (127.1, 83.9), turned to 180 degrees
- moved C19 190.8 mm to (110.8, 91.0), turned to -90 degrees
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Connections:
- L7 pad 1: Net-(JP1-C) -> Net-(C18-Pad2)
- L7 pad 5: Net-(C18-Pad2) -> Net-(JP1-C)
- L8 pad 1: Net-(C18-Pad2) -> Net-(C29-Pad2)
- L8 pad 5: Net-(C29-Pad2) -> Net-(C18-Pad2)

Commit message: WIP
Parts:
- removed the J5 at (-38.8, 93.6)
- removed U16: TLE2082, Package_SO:SOIC-8_3.9x4.9mm_P1.27mm
- C63, C68: footprint Capacitor_SMD:C_0603_1608Metric -> Capacitor_SMD:C_1210_3225Metric
- P28: value SD -> P28
- Q3: value IRF7324 -> IRLML2244; footprint Package_SO:SOIC-8_3.9x4.9mm_P1.27mm -> Package_TO_SOT_SMD:SOT-23
- R32: value 10k -> R
- R33: value 18k -> R
- moved C62 263.4 mm to (183.9, 104.7), turned to 180 degrees
- moved C67 262.2 mm to (184.3, 120.0), turned to 90 degrees
- moved C64 258.9 mm to (180.7, 97.9), turned to 180 degrees
- moved R40 258.8 mm to (184.2, 107.3), turned to 180 degrees
- moved R45 256.7 mm to (184.2, 116.4), turned to 90 degrees
- moved C66 255.6 mm to (176.4, 112.6), turned to 180 degrees
- moved R41 255.5 mm to (182.0, 117.4), turned to 90 degrees
- moved C65 255.1 mm to (175.1, 115.6), turned to -90 degrees
- moved C68 252.8 mm to (174.9, 121.5)
- moved R42 252.2 mm to (179.7, 113.6), turned to 180 degrees
- moved C63 251.6 mm to (172.8, 101.4), turned to 90 degrees
- moved R38 251.2 mm to (176.8, 99.6)
- moved R39 251.0 mm to (176.6, 102.2), turned to 180 degrees
- moved L15 250.4 mm to (185.0, 100.8), turned to -90 degrees
- moved L16 250.0 mm to (183.7, 112.6)
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Connections:
- C1 pad 1: +3.3VP -> +3.3V_HACKRF
- C2 pad 1: +3.3VP -> +3.3V_HACKRF
- C5 pad 1: +3.3VP -> +3.3V_HACKRF
- P22 pad 11: +3.3VP -> +3.3V_HACKRF
- P28 pad 1: VCC -> +3.3V_HACKRF
- P28 pad 10: /mcu/usb/power/SD_POW -> unconnected-(P28-Pin_10-Pad10)
- P28 pad 11: /mcu/usb/power/SD_CLK -> unconnected-(P28-Pin_11-Pad11)
- P28 pad 13: GCK2 -> unconnected-(P28-Pin_13-Pad13)
- P28 pad 14: GCK1 -> unconnected-(P28-Pin_14-Pad14)
- P28 pad 15: /mcu/usb/power/B1AUX14 -> unconnected-(P28-Pin_15-Pad15)
- P28 pad 16: /mcu/usb/power/B1AUX13 -> unconnected-(P28-Pin_16-Pad16)
- P28 pad 17: /mcu/usb/power/CPLD_TCK -> unconnected-(P28-Pin_17-Pad17)
- P28 pad 18: /mcu/usb/power/BANK2F3M2 -> unconnected-(P28-Pin_18-Pad18)
- P28 pad 19: /mcu/usb/power/CPLD_TDI -> unconnected-(P28-Pin_19-Pad19)
- P28 pad 20: /mcu/usb/power/BANK2F3M6 -> unconnected-(P28-Pin_20-Pad20)
- P28 pad 21: /mcu/usb/power/BANK2F3M12 -> unconnected-(P28-Pin_21-Pad21)
- P28 pad 22: /mcu/usb/power/BANK2F3M4 -> unconnected-(P28-Pin_22-Pad22)
- P28 pad 3: /mcu/usb/power/SD_CD -> unconnected-(P28-Pin_3-Pad3)
- P28 pad 4: /mcu/usb/power/SD_DAT3 -> unconnected-(P28-Pin_4-Pad4)
- P28 pad 5: /mcu/usb/power/SD_DAT2 -> unconnected-(P28-Pin_5-Pad5)
- P28 pad 6: /mcu/usb/power/SD_DAT1 -> unconnected-(P28-Pin_6-Pad6)
- P28 pad 7: /mcu/usb/power/SD_DAT0 -> unconnected-(P28-Pin_7-Pad7)
- P28 pad 8: /mcu/usb/power/SD_VOLT0 -> unconnected-(P28-Pin_8-Pad8)
- P28 pad 9: /mcu/usb/power/SD_CMD -> unconnected-(P28-Pin_9-Pad9)
- P30 pad 1: +3.3VP -> +3.3V_HACKRF
- Q1 pad 1: +3.3VP -> +3.3V_HACKRF
- Q2 pad 1: +3.3VP -> +3.3V_HACKRF
- Q3 pad 1: /power/VBUS -> /power/VBUSCTRL
- Q3 pad 2: /power/VBUSCTRL -> /power/VBUS
- Q3 pad 3: (no net) -> VIN
- U1 pad 1: +3.3VP -> +3.3V_HACKRF
- U1 pad 31: +3.3VP -> +3.3V_HACKRF
- U1 pad 42: +3.3VP -> +3.3V_HACKRF
- U3 pad 1: +3.3VP -> +3.3V_HACKRF
- U6 pad 4: (no net) -> -5VA
- U6 pad 8: (no net) -> +5VA
Routing:
- net GND: track 0.00 -> 47.8 mm, vias 0 -> 12
- net AD7: track 0.00 -> 39.1 mm
- net AD6: track 0.00 -> 38.6 mm
- net AD5: track 0.00 -> 37.1 mm, vias 0 -> 2
- net AD4: track 0.00 -> 36.7 mm, vias 0 -> 2
- net AD3: track 0.00 -> 34.7 mm, vias 0 -> 2
- net AD2: track 0.00 -> 34.2 mm, vias 0 -> 2
- net AD15: track 0.00 -> 33.0 mm
- net AD1: track 0.00 -> 32.7 mm, vias 0 -> 2
- net AD0: track 0.00 -> 32.2 mm, vias 0 -> 2
- net AD14: track 0.00 -> 31.9 mm
- net AD13: track 0.00 -> 30.5 mm
- net AD12: track 0.00 -> 29.3 mm
- net AD11: track 0.00 -> 28.2 mm
- net AD10: track 0.00 -> 27.7 mm
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
Commit message: WIP
Parts:
- moved C1 1.27 mm to (162.1, 85.9)
Routing:
- net GND: track 47.8 -> 56.7 mm, vias 12 -> 14
- net DAC_CLK: track 22.1 -> 25.3 mm
- net +5V: track 12.2 -> 11.4 mm
- net +3.3V_HACKRF: track 16.9 -> 17.6 mm
- net AD4: track 36.7 -> 36.1 mm

Commit message: WIP
Parts:
- moved L6 24.0 mm to (149.5, 94.2), turned to -90 degrees
- moved C12 18.2 mm to (150.6, 78.8), turned to 180 degrees
- moved C3 17.4 mm to (162.0, 85.8), turned to 180 degrees
- moved C13 16.3 mm to (150.6, 77.2), turned to 180 degrees
- moved C1 16.0 mm to (174.2, 75.4), turned to 90 degrees
- moved R4 9.08 mm to (133.9, 77.8), turned to 180 degrees
- moved L5 8.88 mm to (154.9, 92.3)
- moved R3 8.20 mm to (124.0, 72.7), turned to -90 degrees
- moved R17 7.95 mm to (96.0, 94.3)
- moved R6 6.85 mm to (126.6, 75.2), turned to 0 degrees
- moved R1 6.49 mm to (133.9, 73.7), turned to 180 degrees
- moved C4 6.30 mm to (173.0, 90.2)
- moved C21 5.53 mm to (125.8, 72.7), turned to -90 degrees
- moved C17 4.45 mm to (149.8, 71.4)
- moved C23 4.33 mm to (125.5, 78.7)
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Connections:
- R23 pad 1: /video/OFFSET_ADJ -> OFFSET_ADJ
- R7 pad 1: /video/GAIN_ADJ -> GAIN_ADJ
- U17 pad 3: /video-misc/OFFSET_ADJ -> OFFSET_ADJ
- U17 pad 4: /video-misc/GAIN_ADJ -> GAIN_ADJ
Routing:
- net GND: track 56.7 -> 90.9 mm, vias 14 -> 15
- net Net-(U4-VEE): track 0.00 -> 31.2 mm, vias 0 -> 2
- net Net-(U4-IOUTB): track 0.00 -> 27.2 mm
- net +3.3V_HACKRF: track 17.6 -> 44.4 mm, vias 2 -> 4
- net Net-(R17-Pad1): track 0.00 -> 26.2 mm
- net Net-(U7-+): track 1.31 -> 26.2 mm
- net GNDA: track 0.00 -> 24.4 mm, vias 0 -> 6
- net Net-(U4-VCC): track 0.00 -> 21.3 mm, vias 0 -> 2
- net +5V: track 11.4 -> 31.3 mm, vias 2 -> 4
- net Net-(U4-REF_OUT): track 0.00 -> 18.7 mm, vias 0 -> 2
- net Net-(U4-NR): track 0.00 -> 16.8 mm, vias 0 -> 2
- net Net-(R4-Pad2): track 0.00 -> 16.3 mm, vias 0 -> 4
- net Net-(U7--): track 0.00 -> 15.0 mm
- net Net-(C47-Pad1): track 0.00 -> 10.2 mm
- net Net-(C46-Pad1): track 0.00 -> 8.94 mm
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
Commit message: WIP
Parts:
- moved R23 4.66 mm to (121.2, 72.7)
- moved C45 4.23 mm to (117.7, 72.7)
- moved R13 3.37 mm to (116.2, 80.3)
- moved R14 3.37 mm to (116.2, 78.6)
- moved R22 2.38 mm to (119.4, 72.7)
- moved R21 1.40 mm to (116.9, 67.1)
- moved C28 0.51 mm to (131.9, 102.2)
- moved C26 0.51 mm to (131.9, 98.6)
- moved C27 0.51 mm to (131.9, 100.4)
- moved C22 0.41 mm to (122.4, 84.3)
- moved R11 0.38 mm to (122.3, 78.3)
- moved C23 0.38 mm to (125.5, 78.3)
- moved R12 0.38 mm to (127.1, 84.3)
- moved JP1 0.36 mm to (112.6, 83.4)
- moved C18 0.13 mm to (112.6, 91.1)
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Routing:
- net Net-(C29-Pad2): track 0.00 -> 27.6 mm
- net -5VA: track 4.51 -> 27.9 mm, vias 0 -> 4
- net OFFSET_ADJ: track 0.00 -> 19.7 mm
- net Net-(C18-Pad2): track 0.00 -> 18.7 mm
- net +5VA: track 3.61 -> 20.8 mm
- net Net-(C34-Pad2): track 0.00 -> 15.3 mm
- net Net-(R19-Pad1): track 0.00 -> 15.2 mm
- net Net-(JP1-C): track 0.00 -> 12.9 mm
- net Net-(C37-Pad2): track 5.19 -> 16.0 mm
- net Net-(L7-Pad2): track 0.00 -> 9.62 mm
- net Net-(L10-Pad1): track 0.00 -> 9.57 mm
- net Net-(U6A-+): track 0.00 -> 9.42 mm
- net Net-(R11-Pad2): track 0.00 -> 8.61 mm
- net Net-(JP1-A): track 0.00 -> 6.98 mm
- net Net-(U5--): track 0.00 -> 6.73 mm
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Other:
- board text added: "NOTE: REPLACED BY 2.7MM NPTH FOR MANUAL ASSEMBLY RIG"

Commit message: WIP
Parts:
- removed C11: 100n, Capacitor_SMD:C_0603_1608Metric
- added C7: 100n, Capacitor_SMD:C_0603_1608Metric, F.Cu at (134.5, 65.1)
- moved L22 12.3 mm to (150.3, 99.5), turned to -90 degrees
- moved C78 10.1 mm to (154.8, 105.5), turned to 90 degrees
- moved C77 6.15 mm to (158.4, 92.8), turned to 90 degrees
- moved C88 5.73 mm to (150.3, 102.9), turned to 180 degrees
- moved L21 5.10 mm to (154.8, 97.0), turned to -90 degrees
- moved C85 3.99 mm to (154.6, 101.7), turned to 180 degrees
- moved U14 2.83 mm to (159.6, 106.6), turned to 0 degrees
- moved U13 2.45 mm to (165.0, 96.8)
- moved C84 2.17 mm to (159.3, 97.2), turned to 90 degrees
- moved C87 1.47 mm to (158.3, 101.7), turned to -90 degrees
- moved L6 0.76 mm to (150.3, 94.2)
- moved R21 0.76 mm to (117.7, 67.1)
- moved L5 0.28 mm to (154.8, 92.0)
- moved U7 0.13 mm to (101.8, 77.6)
- turned L14 to 180 degrees
Routing:
- net GNDA: track 26.2 -> 271.2 mm, vias 6 -> 19
- net +5VA: track 20.8 -> 94.5 mm, vias 0 -> 4
- net -5VA: track 27.9 -> 94.2 mm
- net GND: track 90.9 -> 117.6 mm, vias 15 -> 18
- net -5V: track 0.00 -> 14.9 mm
- net +5V: track 31.3 -> 45.7 mm
- net Net-(C46-Pad1): track 8.94 -> 16.1 mm
- net Net-(C46-Pad2): track 0.00 -> 6.32 mm
- net Net-(U6B--): track 7.04 -> 12.3 mm, vias 0 -> 2
- net Net-(U4-VEE): track 31.2 -> 30.2 mm
- net Net-(U6A--): track 3.97 -> 3.21 mm
- added copper zone on B.Cu, net GNDA
- added copper zone on F.Cu, net GNDA
