File: hardware/alpha/dacattac-alpha.kicad_pcb (KiCad board)
At the start: 4 copper layers, 120 x 75 mm, 175 parts, among them J1 EXT +/- 8V, J10 HOLE, J11 HOLE, J12 HOLE, J13 HOLE, J14 HOLE, J15 HOLE, J2 VIDEO OUT1, J3 VIDEO OUT2, J4 AUDIO_OUT, J5 5V I2C, P20 P20, P22 P22, P28 P28, P30 BANK2_AUX, Q1 2N7002, Q2 2N7002, Q3 IRLML2244, U1 74LVCH16T245, U10 MCP1700x-120xxMB, U11 TPS63700DRCT, U13 L78L05_SO8, U14 L79L05_SO8, U17 MCP47FEB22A0-E/ST, U2 TPS61170DRVR, U3 74LVC1T45, U4 AD768, U5 MAX4104, U6 TLE2082, U7 MAX4104, U9 PCM5102

Commit message: WIP
Parts:
- C55, C64: footprint Capacitor_SMD:C_0603_1608Metric -> Capacitor_SMD:C_1210_3225Metric
- J1: value EXT +/- 8V -> EXT POWER
- moved C55 13.6 mm to (104.1, 113.0), turned to 0 degrees
- moved C68 11.6 mm to (179.3, 110.8), turned to 180 degrees
- moved J1 10.1 mm to (156.7, 117.2), turned to 0 degrees
- moved R41 9.64 mm to (172.4, 118.6), turned to 180 degrees
- moved D2 9.22 mm to (172.7, 115.0), turned to -90 degrees
- moved L16 8.36 mm to (175.7, 115.0), turned to 90 degrees
- moved C65 8.02 mm to (182.8, 117.9)
- moved C71 6.55 mm to (168.0, 101.3)
- moved R42 6.48 mm to (175.5, 118.6)
- moved C66 6.42 mm to (178.8, 118.6), turned to 0 degrees
- moved R40 6.42 mm to (178.0, 105.3)
- moved L17 6.20 mm to (164.5, 101.7)
- moved C73 5.92 mm to (160.3, 101.7)
- moved C72 5.72 mm to (166.7, 110.9), turned to 0 degrees
- moved C67 5.40 mm to (182.8, 114.8), turned to -90 degrees
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Routing:
- net GND: track 117.6 -> 347.6 mm, vias 18 -> 61
- net +8V: track 0.00 -> 38.9 mm, vias 0 -> 2
- net VIN: track 0.00 -> 33.0 mm
- net -8V: track 0.00 -> 28.7 mm
- net Net-(C74-Pad2): track 0.00 -> 13.5 mm
- net Net-(U13-IN): track 0.00 -> 12.3 mm
- net /power/VBUS: track 0.00 -> 8.96 mm
- net Net-(U11-FB): track 0.00 -> 7.43 mm
- net Net-(U2-COMP): track 0.00 -> 6.29 mm
- net /power/VBUSCTRL: track 0.00 -> 5.98 mm
- net Net-(D2-K): track 0.00 -> 5.85 mm
- net Net-(D1-A): track 0.00 -> 4.96 mm
- net Net-(U11-VREF): track 0.00 -> 4.84 mm
- net Net-(U11-EN): track 0.00 -> 3.88 mm
- net Net-(U2-FB): track 0.00 -> 3.53 mm
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- added copper zone on F.Cu, net +8V
- added copper zone on F.Cu, net -8V
- added copper zone on F.Cu, net GND
- added copper zone on F.Cu, net Net-(D1-A)
- added copper zone on F.Cu, net Net-(D2-K)
- added copper zone on F.Cu, net VIN
Other:
- board text added: "+8V"
- board text added: "-8V"
- board text added: "GND"

Commit message: WIP
Parts:
- removed J5: 5V I2C, Connector_Molex:Molex_KK-254_AE-6410-04A_1x04_P2.54mm_Vertical
- added D3: 1N4148, Diode_SMD:D_SOD-123, F.Cu at (52.0, 125.8)
- added D5: 1N4148, Diode_SMD:D_SOD-123, F.Cu at (52.0, 129.2)
- added D6: 1v4, Package_TO_SOT_SMD:SOT-23, F.Cu at (46.9, 125.9)
- added J6: I2C, Connector_Molex:Molex_KK-254_AE-6410-05A_1x05_P2.54mm_Vertical, F.Cu at (189.4, 75.4)
- added Q4: BC857, Package_TO_SOT_SMD:SOT-23, F.Cu at (46.0, 120.0)
- added Q5: BC857, Package_TO_SOT_SMD:SOT-23, F.Cu at (46.6, 135.3)
- added Q6: BC807, Package_TO_SOT_SMD:SOT-23, F.Cu at (46.6, 139.7)
- added R31: 220, Resistor_SMD:R_0603_1608Metric, F.Cu at (42.1, 125.4)
- added R43: 1k, Resistor_SMD:R_0603_1608Metric, F.Cu at (42.1, 127.9)
- added R44: 1k5, Resistor_SMD:R_0603_1608Metric, F.Cu at (42.1, 130.4)
- added R47: 4k3, Resistor_SMD:R_0603_1608Metric, F.Cu at (42.1, 132.9)
- added R48: 47, Resistor_SMD:R_0603_1608Metric, F.Cu at (42.1, 135.4)
- added R49: 4k3, Resistor_SMD:R_0603_1608Metric, F.Cu at (42.1, 137.9)
- added R50: 909, Resistor_SMD:R_0603_1608Metric, F.Cu at (42.1, 140.5)
- added R51: 75, Resistor_SMD:R_0603_1608Metric, F.Cu at (42.1, 143.0)
- added R52: 10k, Resistor_SMD:R_0603_1608Metric, F.Cu at (42.1, 145.5)
- J3: value VIDEO OUT2 -> SYNC OUT
- R18: value 75 -> NF
Connections:
- P28 pad 16: unconnected-(P28-Pin_16-Pad16) -> LSYNC
- R17 pad 1: Net-(R17-Pad1) -> VIDEO
- R18 pad 1: Net-(R17-Pad1) -> Net-(J3-In)
- R18 pad 2: Net-(J3-In) -> VIDEO
- R24 pad 2: Net-(R17-Pad1) -> VIDEO
- R27 pad 1: Net-(R17-Pad1) -> VIDEO
- U17 pad 6: GND -> DA_HVC
- U7 pad 1: Net-(R17-Pad1) -> VIDEO
Routing:
- net Net-(R17-Pad1): track 26.3 -> 0.00 mm
- net Net-(J3-In): track 3.87 -> 30.2 mm

Commit message: WIP
Parts:
- added C10: 100p, Capacitor_SMD:C_0603_1608Metric, F.Cu at (119.6, 109.7)
- added C11: 33u, Capacitor_SMD:C_1210_3225Metric, F.Cu at (114.3, 114.6)
- added C8: NF, Capacitor_SMD:C_0603_1608Metric, F.Cu at (136.6, 111.5)
- added C9: 82p, Capacitor_SMD:C_0603_1608Metric, F.Cu at (121.4, 109.7)
- added D4: 1N4148, Diode_SMD:D_SOD-123, F.Cu at (124.3, 115.1)
- D6: value 1v4 -> 1N4148; footprint Package_TO_SOT_SMD:SOT-23 -> Diode_SMD:D_SOD-123
- J2: renamed from J3; value SYNC OUT -> VIDEO OUT
- J3: renamed from J2; value VIDEO OUT1 -> SYNC OUT
- J4: value AUDIO_OUT -> AUDIO OUT
- moved R43 96.2 mm to (137.3, 114.0), turned to 180 degrees
- moved R31 93.9 mm to (134.7, 109.7), turned to -90 degrees
- moved R47 92.3 mm to (131.5, 109.7), turned to -90 degrees
- moved R44 90.0 mm to (129.7, 109.7), turned to 90 degrees
- moved Q4 87.9 mm to (133.6, 113.1), turned to 180 degrees
- moved Q5 85.6 mm to (129.3, 113.1)
- moved R48 85.0 mm to (123.1, 109.7), turned to -90 degrees
- moved R50 82.8 mm to (120.1, 112.6), turned to 180 degrees
- moved D6 78.6 mm to (124.3, 112.6)
- moved D3 78.4 mm to (129.7, 116.2), turned to 180 degrees
- moved R49 75.0 mm to (112.0, 110.6), turned to -90 degrees
- moved Q6 74.5 mm to (115.2, 110.8)
- moved R51 74.4 mm to (110.9, 114.6), turned to 90 degrees
- moved D5 68.7 mm to (119.2, 115.0)
- moved Q1 67.3 mm to (195.1, 80.7), turned to 180 degrees
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Connections:
- D6 pad 1: Net-(D3-A) -> Net-(D6-K)
- D6 pad 2: unconnected-(D6-NC-Pad2) -> Net-(D4-K)
- J2 pad 1: Net-(J3-In) -> Net-(J2-In)
- J3 pad 1: Net-(J2-In) -> Net-(J3-In)
Routing:
- net /audio/SCL: track 0.00 -> 96.6 mm
- net /audio/SDA: track 0.00 -> 89.6 mm
- net DA_SDA: track 0.00 -> 74.8 mm, vias 0 -> 2
- net DA_SCL: track 0.00 -> 72.3 mm
- net DA_HVC: track 0.00 -> 70.6 mm
- net +5V: track 45.7 -> 86.6 mm, vias 4 -> 5
- net GND: track 347.6 -> 383.4 mm, vias 61 -> 63
- net +3.3V_HACKRF: track 44.4 -> 75.1 mm, vias 4 -> 9
- net VIDEO: track 0.00 -> 26.5 mm
- net GNDA: track 271.2 -> 252.8 mm
- net Net-(D5-A): track 0.00 -> 10.7 mm
- net Net-(Q4-E): track 0.00 -> 9.17 mm
- net Net-(D3-A): track 0.00 -> 8.12 mm
- net Net-(D6-K): track 0.00 -> 7.60 mm
- net Net-(Q6-E): track 0.00 -> 7.51 mm
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Other:
- board text removed: "1V8"
- board text removed: "3V3"
- board text removed: "ANTENNA"
- board text removed: "CLKIN"
- board text removed: "CLKOUT"
- board text removed: "DFU"
- board text removed: "LED1"
- board text removed: "RESET"
- board text removed: "RF"
- board text removed: "RX"
- board text removed: "TX"
- board text removed: "USB"
- board text removed: "end plate templates for optional Hammond 1455J1201 enclosure"
- board text removed: "front end plate"
- board text removed: "rear end plate"

Commit message: WIP
Parts:
- added C75: 100n, Capacitor_SMD:C_0603_1608Metric, F.Cu at (135.4, 107.1)
- added C76: 100n, Capacitor_SMD:C_0603_1608Metric, F.Cu at (113.5, 117.3)
- moved R52 163.4 mm to (194.7, 86.8)
- moved C54 36.7 mm to (99.7, 124.1), turned to 90 degrees
- moved C56 36.7 mm to (95.9, 124.1), turned to 90 degrees
- moved C60 32.6 mm to (120.0, 132.8), turned to -90 degrees
- moved C57 32.2 mm to (107.6, 123.3), turned to 0 degrees
- moved C61 32.0 mm to (111.5, 133.3)
- moved U10 31.3 mm to (116.1, 132.7)
- moved JP3 30.8 mm to (97.4, 134.3)
- moved JP2 30.7 mm to (102.6, 134.3), turned to 0 degrees
- moved C52 27.9 mm to (93.3, 126.7), turned to 0 degrees
- moved R30 26.9 mm to (93.3, 130.2)
- moved R29 26.9 mm to (93.3, 128.4)
- moved C51 26.8 mm to (93.3, 131.9), turned to 0 degrees
- moved U9 26.8 mm to (100.8, 129.4)
- moved C58 26.8 mm to (97.8, 124.1), turned to 90 degrees
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Connections:
- C10 pad 2: GND -> GNDV
- C16 pad 2: GNDA -> GNDV
- C17 pad 2: GNDA -> GNDV
- C21 pad 2: GNDA -> GNDV
- C22 pad 2: GNDA -> GNDV
- C23 pad 2: GNDA -> GNDV
- C24 pad 2: GNDA -> GNDV
- C25 pad 2: GNDA -> GNDV
- C26 pad 2: GNDA -> GNDV
- C27 pad 2: GNDA -> GNDV
- C28 pad 2: GNDA -> GNDV
- C32 pad 2: GNDA -> GNDV
- C33 pad 2: GNDA -> GNDV
- C35 pad 2: GNDA -> GNDV
- C36 pad 2: GNDA -> GNDV
- C39 pad 2: GNDA -> GNDV
- C40 pad 2: GNDA -> GNDV
- C43 pad 2: GNDA -> GNDV
- C44 pad 2: GNDA -> GNDV
- C45 pad 2: GNDA -> GNDV
- C47 pad 2: GNDA -> GNDV
- C48 pad 2: GNDA -> GNDV
- C50 pad 2: GNDA -> GNDV
- C51 pad 2: GND -> GNDA
- C52 pad 2: GND -> GNDA
- C54 pad 2: GND -> GNDA
- C55 pad 2: GND -> GNDA
- C56 pad 2: GND -> GNDA
- C57 pad 2: GND -> GNDA
- C58 pad 2: GND -> GNDA
- C59 pad 2: GND -> GNDA
- C69 pad 2: GNDA -> GNDV
- C70 pad 2: GNDA -> GNDV
- C8 pad 2: GND -> GNDV
- C9 pad 2: GND -> GNDV
- D3 pad 1: GND -> GNDV
- J2 pad 2: GNDA -> GNDV
- J3 pad 2: GNDA -> GNDV
- J4 pad 3: GND -> GNDA
- JP1 pad 3: GNDA -> GNDV
- JP2 pad 1: GND -> GNDA
- JP3 pad 1: GND -> GNDA
- L10 pad 6: GNDA -> GNDV
- L11 pad 6: GNDA -> GNDV
- L12 pad 6: GNDA -> GNDV
- L13 pad 6: GNDA -> GNDV
- L14 pad 4: GNDA -> GNDV
- L14 pad 6: GNDA -> GNDV
- L7 pad 6: GNDA -> GNDV
- L8 pad 6: GNDA -> GNDV
- L9 pad 6: GNDA -> GNDV
- Q4 pad 3: GND -> GNDV
- R1 pad 2: GNDA -> GNDV
- R12 pad 2: GNDA -> GNDV
- R15 pad 2: GNDA -> GNDV
- R16 pad 2: GNDA -> GNDV
- R22 pad 2: GNDA -> GNDV
- R28 pad 2: GNDA -> GNDV
- R3 pad 2: GNDA -> GNDV
- R33 pad 2: GND -> GNDA
- R44 pad 2: GND -> GNDV
- R46 pad 2: GNDA -> GNDV
- R6 pad 1: GNDA -> GNDV
- U4 pad 28: GNDA -> GNDV
- U4 pad 5: GNDA -> GNDV
- U5 pad 3: GNDA -> GNDV
- U9 pad 16: GND -> GNDA
- U9 pad 19: GND -> GNDA
- U9 pad 3: GND -> GNDA
- U9 pad 9: GND -> GNDA
Routing:
- net GNDV: track 0.00 -> 309.7 mm, vias 0 -> 26
- net GNDA: track 252.8 -> 32.7 mm, vias 19 -> 5
- net -8V: track 33.4 -> 95.1 mm
- net +3.3VDAC: track 0.00 -> 57.3 mm
- net +5V: track 86.6 -> 139.3 mm, vias 5 -> 9
- net Net-(J4-IN2): track 0.00 -> 28.6 mm
- net LSYNC: track 0.00 -> 13.7 mm
- net Net-(J4-IN1): track 0.00 -> 10.6 mm
- net Net-(U9-VNEG): track 0.00 -> 7.49 mm
- net DA_HVC: track 70.6 -> 76.0 mm
- net Net-(U9-SCK): track 0.00 -> 5.21 mm
- net Net-(U9-XSMT): track 0.00 -> 5.00 mm
- net Net-(U9-LDOO): track 0.00 -> 4.89 mm
- net Net-(U9-OUTL): track 0.00 -> 4.67 mm
- net Net-(Q6-B): track 0.00 -> 4.46 mm
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- added copper zone on B.Cu, net GNDV
- added copper zone on F.Cu, net GNDV

Commit message: WIP
Parts:
- moved C61 6.85 mm to (115.1, 127.5)
- moved U10 6.39 mm to (118.7, 126.9)
- moved C60 6.39 mm to (122.7, 127.0)
- moved C51 1.27 mm to (94.6, 131.9)
- moved C52 1.27 mm to (94.6, 126.7)
- moved C54 1.27 mm to (101.0, 124.1)
- moved C55 1.27 mm to (104.4, 124.2)
- moved R29 1.27 mm to (94.6, 128.4)
- moved R30 1.27 mm to (94.6, 130.2)
- moved U9 1.27 mm to (102.1, 129.4)
- moved C53 1.27 mm to (97.2, 127.4)
- moved C56 1.27 mm to (97.2, 124.1)
- moved C57 1.27 mm to (108.8, 123.3)
- moved C58 1.27 mm to (99.1, 124.1)
- moved C59 1.27 mm to (108.8, 125.0)
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Routing:
- net GND: track 383.5 -> 483.6 mm, vias 63 -> 67
- net VIN: track 33.0 -> 117.1 mm
- net /audio/I2S_SDA: track 0.00 -> 66.4 mm
- net /audio/I2S_WS: track 0.00 -> 65.4 mm, vias 0 -> 2
- net /audio/I2S_SCK: track 0.00 -> 62.7 mm, vias 0 -> 2
- net +3.3VDAC: track 57.3 -> 52.8 mm
- net Net-(J3-In): track 33.5 -> 31.9 mm
- net Net-(J4-IN1): track 10.6 -> 11.8 mm
- net /audio/SDA: track 89.6 -> 90.8 mm
- net -8V: track 95.1 -> 94.1 mm
- net Net-(J4-IN2): track 28.6 -> 29.1 mm
- net GNDA: track 32.7 -> 32.8 mm, vias 5 -> 4

Commit message: WIP
Parts:
- added R53: 0, Resistor_SMD:R_1210_3225Metric, F.Cu at (113.2, 135.6)
- moved R46 0.51 mm to (136.5, 95.3)
Connections:
- J10 pad 1: GND -> unconnected-(J10-Pin_1-Pad1)
- J11 pad 1: GND -> unconnected-(J11-Pin_1-Pad1)
Routing:
- net GND: track 483.6 -> 679.2 mm, vias 67 -> 85
- net +3.3V_HACKRF: track 75.1 -> 188.8 mm, vias 9 -> 11
- net GNDV: track 309.7 -> 416.2 mm, vias 26 -> 37
- net GNDA: track 32.8 -> 115.2 mm, vias 4 -> 16
- net +8V: track 38.9 -> 97.9 mm, vias 2 -> 4
- net +5V: track 139.3 -> 192.7 mm, vias 9 -> 11
- net DAC_CLK: track 25.3 -> 28.5 mm
- net +3.3VDAC: track 52.8 -> 53.7 mm
- net Net-(U4-VEE): track 30.2 -> 31.0 mm
- net VIN: track 117.1 -> 116.3 mm
- net -5VA: track 94.4 -> 93.9 mm
- added copper zone on B.Cu, net GND

Commit message: WIP
Parts:
- removed R46, R53: 0, Resistor_SMD:R_1210_3225Metric
- U10: value MCP1700x-120xxMB -> MCP1700T-3302E/MB
- moved C20 0.38 mm to (109.4, 91.1)
- moved C29 0.38 mm to (109.4, 99.4)
- moved C19 0.25 mm to (111.1, 91.1)
- moved C30 0.25 mm to (111.1, 99.4)
- moved C18 0.13 mm to (112.7, 91.1)
- moved C31 0.13 mm to (112.7, 99.4)
- turned C37 to 90 degrees
- turned C38 to 90 degrees
Connections:
- C10 pad 2: GNDV -> GND
- C16 pad 2: GNDV -> GND
- C17 pad 2: GNDV -> GND
- C21 pad 2: GNDV -> GND
- C22 pad 2: GNDV -> GND
- C23 pad 2: GNDV -> GND
- C24 pad 2: GNDV -> GND
- C25 pad 2: GNDV -> GND
- C26 pad 2: GNDV -> GND
- C27 pad 2: GNDV -> GND
- C28 pad 2: GNDV -> GND
- C32 pad 2: GNDV -> GND
- C33 pad 2: GNDV -> GND
- C35 pad 2: GNDV -> GND
- C36 pad 2: GNDV -> GND
- C39 pad 2: GNDV -> GND
- C40 pad 2: GNDV -> GND
- C43 pad 2: GNDV -> GND
- C44 pad 2: GNDV -> GND
- C45 pad 2: GNDV -> GND
- C47 pad 2: GNDV -> GND
- C48 pad 2: GNDV -> GND
- C50 pad 2: GNDV -> GND
- C51 pad 2: GNDA -> GND
- C52 pad 2: GNDA -> GND
- C54 pad 2: GNDA -> GND
- C55 pad 2: GNDA -> GND
- C56 pad 2: GNDA -> GND
- C57 pad 2: GNDA -> GND
- C58 pad 2: GNDA -> GND
- C59 pad 2: GNDA -> GND
- C69 pad 2: GNDV -> GND
- C70 pad 2: GNDV -> GND
- C75 pad 2: GNDV -> GND
- C76 pad 1: GNDV -> GND
- C8 pad 2: GNDV -> GND
- C9 pad 2: GNDV -> GND
- D3 pad 1: GNDV -> GND
- J10 pad 1: unconnected-(J10-Pin_1-Pad1) -> GND
- J11 pad 1: unconnected-(J11-Pin_1-Pad1) -> GND
- J2 pad 2: GNDV -> GND
- J3 pad 2: GNDV -> GND
- J4 pad 3: GNDA -> GND
- JP1 pad 3: GNDV -> GND
- JP2 pad 1: GNDA -> GND
- JP3 pad 1: GNDA -> GND
- L10 pad 6: GNDV -> GND
- L11 pad 6: GNDV -> GND
- L12 pad 6: GNDV -> GND
- L13 pad 6: GNDV -> GND
- L14 pad 4: GNDV -> GND
- L14 pad 6: GNDV -> GND
- L7 pad 6: GNDV -> GND
- L8 pad 6: GNDV -> GND
- L9 pad 6: GNDV -> GND
- Q4 pad 3: GNDV -> GND
- R1 pad 2: GNDV -> GND
- R12 pad 2: GNDV -> GND
- R15 pad 2: GNDV -> GND
- R16 pad 2: GNDV -> GND
- R22 pad 2: GNDV -> GND
- R28 pad 2: GNDV -> GND
- R3 pad 2: GNDV -> GND
- R33 pad 2: GNDA -> GND
- R44 pad 2: GNDV -> GND
- R6 pad 1: GNDV -> GND
- U4 pad 28: GNDV -> GND
- U4 pad 5: GNDV -> GND
- U5 pad 3: GNDV -> GND
- U9 pad 16: GNDA -> GND
- U9 pad 19: GNDA -> GND
- U9 pad 3: GNDA -> GND
- U9 pad 9: GNDA -> GND
Routing:
- net GND: track 679.2 -> 1747.1 mm, vias 85 -> 183
- net GNDV: track 416.2 -> 0.00 mm, vias 37 -> 0
- net GNDA: track 115.2 -> 0.00 mm, vias 16 -> 0
- net Net-(C37-Pad2): track 16.0 -> 25.5 mm
- net Net-(C46-Pad2): track 6.32 -> 15.1 mm
- net Net-(C34-Pad2): track 15.3 -> 23.5 mm
- net Net-(U7--): track 14.9 -> 22.6 mm, vias 0 -> 2
- net /audio/I2S_SCK: track 62.7 -> 64.3 mm
- net +3.3V_HACKRF: track 188.8 -> 187.9 mm
- net Net-(C18-Pad2): track 18.7 -> 17.8 mm
- net +5V: track 192.7 -> 193.2 mm
- removed copper zone on B.Cu, net GNDA
- removed copper zone on F.Cu, net GNDA
- removed copper zone on B.Cu, net GNDV
- removed copper zone on F.Cu, net GNDV
