File: hardware/alpha/dacattac-alpha.kicad_pcb (KiCad board)
At the start: 4 copper layers, 120 x 75 mm, 196 parts, among them J1 EXT POWER, J10 HOLE, J11 HOLE, J12 HOLE, J13 HOLE, J14 HOLE, J15 HOLE, J2 VIDEO OUT, J3 SYNC OUT, J4 AUDIO OUT, J6 I2C, P20 P20, P22 P22, P28 P28, P30 BANK2_AUX, Q1 2N7002, Q2 2N7002, Q3 IRLML2244, Q4 BC857, Q5 BC857, Q6 BC807, U1 74LVCH16T245, U10 MCP1700T-3302E/MB, U11 TPS63700DRCT, U13 L78L05_SO8, U14 L79L05_SO8, U17 MCP47FEB22A0-E/ST, U2 TPS61170DRVR, U3 74LVC1T45, U4 AD768, U5 MAX4104, U6 TLE2082, U7 MAX4104, U9 PCM5102

Commit message: WIP
Parts:
- added C79: 22u, Capacitor_SMD:C_1210_3225Metric, F.Cu at (169.6, 115.0)
- added R46: 0, Resistor_SMD:R_0603_1608Metric, F.Cu at (112.0, 134.9)
- R49: value 4k3 -> 470
- moved R61 0.58 mm to (193.3, 73.7)
- moved J6 0.57 mm to (188.6, 75.1)
- moved Q1 0.57 mm to (194.5, 80.7)
- moved Q2 0.57 mm to (194.5, 77.0)
- moved R52 0.57 mm to (194.1, 86.8)
- moved R62 0.57 mm to (193.3, 84.1)
- moved C7 0.25 mm to (134.5, 65.3)
- moved FID2 0.10 mm to (87.9, 136.8)
Routing:
- net GND: track 1747.1 -> 1847.9 mm, vias 183 -> 198
- net Net-(U9-SCK): track 5.21 -> 9.83 mm
- net -8V: track 93.7 -> 91.6 mm
- net +5V: track 193.2 -> 194.1 mm
- net +3.3V_HACKRF: track 187.9 -> 187.2 mm
Other:
- copper layers 4 -> 2

Commit message: WIP
Parts:
- U17: footprint Package_SO:TSSOP-8_3x3mm_P0.65mm -> Package_SO:TSSOP-8_4.4x3mm_P0.65mm
- moved C33 0.23 mm to (105.0, 106.0)
Routing:
- net GND: track 1847.9 -> 1869.5 mm
- net +5V: track 194.1 -> 195.9 mm
- net OFFSET_ADJ: track 19.9 -> 19.1 mm
- net GAIN_ADJ: track 4.98 -> 4.26 mm
- net DA_SDA: track 74.9 -> 74.2 mm
- net DA_SCL: track 72.5 -> 71.8 mm
- net DA_HVC: track 76.2 -> 75.5 mm
