File: hardware/alpha/audio.kicad_sch (KiCad schematic)
At the start: 0 parts

Commit message: Updated
Parts:
- added C51, C52: 2n2, symbol Device:C
- added C53, C56, C60, C61: 2u2, symbol Device:C
- added C54, C57, C58, C59: 100n, symbol Device:C
- added C55: 10uF, symbol Device:C
- added J4: Conn_Coaxial_x2, symbol Connector:Conn_Coaxial_x2
- added JP2: FILTER MODE, symbol Jumper:Jumper_3_Open
- added JP3: DE EMPHASIS, symbol Jumper:Jumper_3_Open
- added P22: P22, symbol Connector_Generic:Conn_02x13_Odd_Even
- added R29, R30: 470, symbol Device:R
- added R32: 10K, symbol Device:R
- added R33: 18K, symbol Device:R
- added R34, R35, R37: 0, symbol Device:R
- added R36: NF, symbol Device:R
- added U10: MCP1700x-120xxMB, Package_TO_SOT_SMD:SOT-89-3, symbol Regulator_Linear:MCP1700x-120xxMB
- added U9: PCM5102, Package_SO:TSSOP-20_4.4x6.5mm_P0.65mm, symbol Audio:PCM5102
Connections:
- new net: R30.1, U9.7 (OUTR)
- new net: C51.1, J4.2 (IN2), R30.2
- new net: R34.2, U9.15 (LRCK)
- new net: C52.1, J4.1 (IN1), R29.2
- new net: JP3.2 (C), U9.10 (DEMP)
- new net: R29.1, U9.6 (OUTL)
- new net: R32.2, R33.1, U9.17 (XSMT)
- new net: R35.2, U9.14 (DIN)
- new net: JP2.2 (C), U9.11 (FLT)
- new net: R36.2, U9.12 (SCK)
- new net: R37.2, U9.13 (BCK)
- new net: C59.1, U9.18 (LDOO)
- new net: C53.1, U9.2 (CAPP)
- new net: C53.2, U9.4 (CAPM)
- new net: C56.1, U9.5 (VNEG)
- new net +3.3VDAC: C54.1, C55.1, C57.1, C58.1, C61.1, JP2.3 (B), JP3.3 (B), U10.3 (VO), U9.1 (CPVDD), U9.20 (DVDD), U9.8 (AVDD)
- new net GND: C51.2, C52.2, C54.2, C55.2, C56.2, C57.2, C58.2, C59.2, C60.2, C61.2, J4.3 (EXT), JP2.1 (A), JP3.1 (A), P22.10 (Pin_10), P22.18 (Pin_18), P22.4 (Pin_4), R33.2, U10.1 (GND), U9.16 (FMT), U9.19 (DGND), U9.3 (CPGND), U9.9 (AGND)
- new net I2S_SCK: P22.16 (Pin_16), R36.1, R37.1
- new net I2S_SDA: P22.13 (Pin_13), R35.1
- new net I2S_WS: P22.15 (Pin_15), R34.1
- new net SCL: P22.26 (Pin_26)
- new net SDA: P22.24 (Pin_24)
- new net VIN: C60.1, R32.1, U10.2 (VI)

Commit message: Updated
Parts:
- added J5: 5V I2C, symbol Connector_Generic:Conn_01x04
- added Q1, Q2: 2N7002, Package_TO_SOT_SMD:SOT-23, symbol Transistor_FET:2N7002
- J4: value Conn_Coaxial_x2 -> AUDIO_OUT
- R32: value 10K -> 10k
- R33: value 18K -> 18k
Connections:
- net GND: now also J5.1 (Pin_1)
- net SCL: now also Q2.2 (S)
- net SDA: now also Q1.2 (S)
- net VIN: no longer R32.1
- net +3.3VP: now reaches P22.11 (Pin_11)
- net +3.3VP: now also Q1.1 (G), Q2.1 (G)
- new net +5V: J5.4 (Pin_4)
- new net +8V: R32.1
- new net DA_SCL: J5.2 (Pin_2), Q2.3 (D)
- new net DA_SDA: J5.3 (Pin_3), Q1.3 (D)
Other:
- moved on the sheet: C51, C52, C53, C54, C55, C56, C57, C58, C59, C60, C61, J4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

Commit message: WIP
Parts:
- C51, C52, C53, C54, C55, C56, C57, C58, C59, C60, C61: footprint (none) -> Capacitor_SMD:C_0603_1608Metric
- J5: footprint (none) -> Connector_Molex:Molex_KK-254_AE-6410-04A_1x04_P2.54mm_Vertical
- JP2, JP3: footprint (none) -> Jumper:SolderJumper-3_P1.3mm_Open_Pad1.0x1.5mm
- R29, R30, R32, R33, R34, R35, R36, R37: footprint (none) -> Resistor_SMD:R_0603_1608Metric
Other:
- moved on the sheet: C60, C61, U10

Commit message: WIP
Changed lines of the file:
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@@
   (junction (at 79.375 50.165) (diameter 0) (color 0 0 0 0)
   )
-  (junction (at 53.975 42.545) (diameter 0) (color 0 0 0 0)
-  )
   (junction (at 170.815 140.335) (diameter 0) (color 0 0 0 0)
   )
@@
     (stroke (width 0) (type default))
   )
-  (wire (pts (xy 53.975 34.925) (xy 53.975 42.545))
+  (wire (pts (xy 48.26 35.56) (xy 48.26 42.545))
     (stroke (width 0) (type default))
   )
@@
     (stroke (width 0) (type default))
   )
-  (wire (pts (xy 45.72 42.545) (xy 53.975 42.545))
-    (stroke (width 0) (type default))
-  )
   (wire (pts (xy 197.485 130.175) (xy 197.485 133.985))
     (stroke (width 0) (type default))
@@
     (stroke (width 0) (type default))
   )
-  (wire (pts (xy 53.975 42.545) (xy 63.5 42.545))
+  (wire (pts (xy 48.26 42.545) (xy 63.5 42.545))
     (stroke (width 0) (type default))
   )
@@
     )
   )
-  (global_label "+3.3V_HACKRF" (shape input) (at 45.72 42.545 180) (fields_autoplaced)
-    (effects (font (size 1.27 1.27)) (justify right))
-    (property "Intersheetrefs" "${INTERSHEET_REFS}" (at 28.7647 42.545 0)
-      (effects (font (size 1.27 1.27)) (justify right) hide)
-    )
-  )
   (global_label "+5V" (shape input) (at 128.27 31.75 180) (fields_autoplaced)
     (effects (font (size 1.27 1.27)) (justify right))
@@
     )
   )
-  (symbol (lib_id "+3.3v_hackrf:+3.3V_HACKRF") (at 53.975 34.925 0) (unit 1)
+  (symbol (lib_id "+3.3v_hackrf:+3.3V_HACKRF") (at 48.26 35.56 0) (unit 1)
     (in_bom yes) (on_board yes) (dnp no)
-    (property "Reference" "#PWR079" (at 57.785 36.195 0)
-      (effects (font (size 1.27 1.27)) hide)
-    )
-    (property "Value" "+3.3V_HACKRF" (at 53.975 30.48 0)
-      (effects (font (size 1.27 1.27)))
-    )
-    (property "Footprint" "" (at 53.975 34.925 0)
-      (effects (font (size 1.27 1.27)) hide)
-    )
-    (property "Datasheet" "" (at 53.975 34.925 0)
-      (effects (font (size 1.27 1.27)) hide)
-    )
+    (property "Reference" "#PWR079" (at 52.07 36.83 0)
+      (effects (font (size 1.27 1.27)) hide)
+    )
+    (property "Value" "+3.3V_HACKRF" (at 48.26 31.115 0)
+      (effects (font (size 1.27 1.27)))
+    )
+    (property "Footprint" "" (at 48.26 35.56 0)
+      (effects (font (size 1.27 1.27)) hide)
+    )
+    (property "Datasheet" "" (at 48.26 35.56 0)
+      (effects (font (size 1.27 1.27)) hide)
+    )

Commit message: WIP
Parts:
- P22: footprint (none) -> hackrf:GSG-HEADER-2x13
Changed lines of the file:
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@@
       (effects (font (size 1.27 1.27)))
     )
-    (property "Footprint" "" (at 68.58 45.085 0)
+    (property "Footprint" "hackrf:GSG-HEADER-2x13" (at 68.58 45.085 0)
       (effects (font (size 1.27 1.27)) hide)
     )

Commit message: WIP
Parts:
- J4: footprint (none) -> PJRAN2X1U01X:PJRAN2X1U01X
Changed lines of the file:
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@@
       (effects (font (size 1.27 1.27)) (justify left))
     )
-    (property "Footprint" "" (at 250.825 114.935 0)
+    (property "Footprint" "PJRAN2X1U01X:PJRAN2X1U01X" (at 250.825 114.935 0)
       (effects (font (size 1.27 1.27)) hide)
     )

Commit message: WIP
Parts:
- R32: value 10k -> R
- R33: value 18k -> R
Connections:
- net +3.3VP renamed +3.3V_HACKRF
Changed lines of the file:
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@@
       (effects (font (size 1.27 1.27)))
     )
-    (property "Value" "10k" (at 125.73 132.715 90)
+    (property "Value" "R" (at 125.73 132.715 90)
       (effects (font (size 1.27 1.27)))
     )
@@
   )
   (symbol (lib_id "Device:R") (at 147.955 145.415 0) (unit 1)
-    (in_bom yes) (on_board yes) (dnp no) (fields_autoplaced)
+    (in_bom yes) (on_board yes) (dnp no)
     (property "Reference" "R33" (at 149.86 144.145 0)
       (effects (font (size 1.27 1.27)) (justify left))
     )
-    (property "Value" "18k" (at 149.86 146.685 0)
-      (effects (font (size 1.27 1.27)) (justify left))
-    )
+    (property "Value" "R" (at 147.955 146.05 90)
+      (effects (font (size 1.27 1.27)) (justify left))
+    )

Commit message: WIP
Parts:
- C55: footprint Capacitor_SMD:C_0603_1608Metric -> Capacitor_SMD:C_1210_3225Metric
Changed lines of the file:
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@@
       (effects (font (size 1.27 1.27)) (justify left))
     )
-    (property "Footprint" "Capacitor_SMD:C_0603_1608Metric" (at 177.4952 92.075 0)
+    (property "Footprint" "Capacitor_SMD:C_1210_3225Metric" (at 177.4952 92.075 0)
       (effects (font (size 1.27 1.27)) hide)
     )
