File: hardware/alpha/audio.kicad_sch (KiCad schematic)
At the start: 28 parts, among them J4 AUDIO_OUT, J5 5V I2C, P22 P22, Q1 2N7002, Q2 2N7002, U10 MCP1700x-120xxMB, U9 PCM5102

Commit message: WIP
Parts:
- removed J5: 5V I2C, Connector_Molex:Molex_KK-254_AE-6410-04A_1x04_P2.54mm_Vertical, symbol Connector_Generic:Conn_01x04
- added J6: I2C, Connector_Molex:Molex_KK-254_AE-6410-05A_1x05_P2.54mm_Vertical, symbol Connector_Generic:Conn_01x05
Connections:
- net +5V: now also J6.4 (Pin_4)
- net DA_SCL: now also J6.2 (Pin_2)
- net DA_SDA: now also J6.3 (Pin_3)
- net GND: now also J6.1 (Pin_1)
- new net DA_HVC: J6.5 (Pin_5)
Changed lines of the file:
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@@
+    (stroke (width 0) (type default))
+  )
+  (wire (pts (xy 131.445 29.21) (xy 136.525 29.21))
     (stroke (width 0) (type default))
   )
@@
     (stroke (width 0) (type default))
   )
+  (wire (pts (xy 135.255 27.305) (xy 135.255 31.75))
+    (stroke (width 0) (type default))
+  )
   (wire (pts (xy 139.7 114.935) (xy 139.7 117.475))
     (stroke (width 0) (type default))
@@
     (stroke (width 0) (type default))
   )
-  (wire (pts (xy 128.27 31.75) (xy 136.525 31.75))
-    (stroke (width 0) (type default))
-  )
   (wire (pts (xy 48.26 42.545) (xy 63.5 42.545))
     (stroke (width 0) (type default))
@@
   )
   (wire (pts (xy 250.825 130.175) (xy 250.825 132.715))
+    (stroke (width 0) (type default))
+  )
+  (wire (pts (xy 135.255 31.75) (xy 136.525 31.75))
     (stroke (width 0) (type default))
   )
@@
     )
   )
-  (global_label "+5V" (shape input) (at 128.27 31.75 180) (fields_autoplaced)
-    (effects (font (size 1.27 1.27)) (justify right))
-    (property "Intersheetrefs" "${INTERSHEET_REFS}" (at 121.4143 31.75 0)
-      (effects (font (size 1.27 1.27)) (justify right) hide)
-    )
-  )
   (global_label "DA_SCL" (shape input) (at 141.605 60.325 0) (fields_autoplaced)
     (effects (font (size 1.27 1.27)) (justify left))
@@
     )
   )
+  (global_label "DA_HVC" (shape input) (at 131.445 29.21 180) (fields_autoplaced)
+    (effects (font (size 1.27 1.27)) (justify right))
+    (property "Intersheetrefs" "${INTERSHEET_REFS}" (at 121.4445 29.21 0)
+      (effects (font (size 1.27 1.27)) (justify right) hide)
+    )
+  )
   (symbol (lib_id "+3.3v_aud:+3.3V_AUD") (at 170.815 79.375 0) (unit 1)
     (in_bom yes) (on_board yes) (dnp no) (fields_autoplaced)
@@
         (path "/487245ca-0c1f-4f9d-bc99-20c8f558090f/80e17ed4-cb43-4c12-a09c-75e0f0ffaba0"
           (reference "C51") (unit 1)
-        )
-      )
-    )
-  )
-  (symbol (lib_id "Connector_Generic:Conn_01x04") (at 141.605 36.83 0) (mirror x) (unit 1)
-    (in_bom yes) (on_board yes) (dnp no)
-    (property "Reference" "J5" (at 144.145 36.83 0)
-      (effects (font (size 1.27 1.27)) (justify left))
-    )
-    (property "Value" "5V I2C" (at 144.145 34.29 0)
-      (effects (font (size 1.27 1.27)) (justify left))
-    )
-    (property "Footprint" "Connector_Molex:Molex_KK-254_AE-6410-04A_1x04_P2.54mm_Vertical" (at 141.605 36.83 0)
-      (effects (font (size 1.27 1.27)) hide)
-    )
-    (property "Datasheet" "~" (at 141.605 36.83 0)
-      (effects (font (size 1.27 1.27)) hide)
-    )
-    (pin "3")
-    (pin "1")
-    (pin "2")
-    (pin "4")
-    (instances
-      (project "dacattac-alpha"
-        (path "/487245ca-0c1f-4f9d-bc99-20c8f558090f/80e17ed4-cb43-4c12-a09c-75e0f0ffaba0"
-          (reference "J5") (unit 1)
         )
       )
@@
     )
   )
+  (symbol (lib_id "power:+5V") (at 135.255 27.305 0) (unit 1)
+    (in_bom yes) (on_board yes) (dnp no) (fields_autoplaced)
+    (property "Reference" "#PWR0120" (at 135.255 31.115 0)
+      (effects (font (size 1.27 1.27)) hide)
+    )
+    (property "Value" "+5V" (at 135.255 22.225 0)
+      (effects (font (size 1.27 1.27)))
+    )
+    (property "Footprint" "" (at 135.255 27.305 0)
+      (effects (font (size 1.27 1.27)) hide)
+    )
+    (property "Datasheet" "" (at 135.255 27.305 0)
+      (effects (font (size 1.27 1.27)) hide)
+    )
+    (pin "1")
+    (instances
+      (project "dacattac-alpha"
+        (path "/487245ca-0c1f-4f9d-bc99-20c8f558090f/80e17ed4-cb43-4c12-a09c-75e0f0ffaba0"
+          (reference "#PWR0120") (unit 1)
+        )
+      )
+    )
+  )
   (symbol (lib_id "power:GND") (at 250.825 132.715 0) (unit 1)
     (in_bom yes) (on_board yes) (dnp no) (fields_autoplaced)
@@
         )
       )
+    )
+  )
+  (symbol (lib_id "Connector_Generic:Conn_01x05") (at 141.605 34.29 0) (mirror x) (unit 1)
+    (in_bom yes) (on_board yes) (dnp no)
+    (property "Reference" "J6" (at 144.145 35.56 0)
+      (effects (font (size 1.27 1.27)) (justify left))
+    )
+    (property "Value" "I2C" (at 144.145 33.02 0)
+      (effects (font (size 1.27 1.27)) (justify left))
+    )
+    (property "Footprint" "Connector_Molex:Molex_KK-254_AE-6410-05A_1x05_P2.54mm_Vertical" (at 141.605 34.29 0)
+      (effects (font (size 1.27 1.27)) hide)
+    )
+    (property "Datasheet" "~" (at 141.605 34.29 0)
+      (effects (font (size 1.27 1.27)) hide)
+    )
+    (pin "5")
+    (pin "3")
+    (pin "2")
+    (pin "1")
+    (pin "4")
+    (instances
+      (project "dacattac-alpha"
+        (path "/487245ca-0c1f-4f9d-bc99-20c8f558090f/80e17ed4-cb43-4c12-a09c-75e0f0ffaba0"
+          (reference "J6") (unit 1)
+        )
+      )

Commit message: WIP
Parts:
- J4: value AUDIO_OUT -> AUDIO OUT
Changed lines of the file:
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@@
   (symbol (lib_id "Connector:Conn_Coaxial_x2") (at 250.825 112.395 0) (unit 1)
     (in_bom yes) (on_board yes) (dnp no) (fields_autoplaced)
-    (property "Reference" "J4" (at 253.365 111.4182 0)
+    (property "Reference" "J4" (at 254 111.4182 0)
       (effects (font (size 1.27 1.27)) (justify left))
     )
-    (property "Value" "AUDIO_OUT" (at 253.365 113.9582 0)
+    (property "Value" "AUDIO OUT" (at 254 113.9582 0)
       (effects (font (size 1.27 1.27)) (justify left))
     )

Commit message: WIP
Parts:
- added R53: 0, symbol Device:R
Connections:
- net GND: now also R53.1; no longer C51.2, C52.2, C54.2, C55.2, C56.2, C57.2, C58.2, C59.2, J4.3 (EXT), JP2.1 (A), JP3.1 (A), R33.2, U9.16 (FMT), U9.19 (DGND), U9.3 (CPGND), U9.9 (AGND)
- new net GNDA: C51.2, C52.2, C54.2, C55.2, C56.2, C57.2, C58.2, C59.2, J4.3 (EXT), JP2.1 (A), JP3.1 (A), R33.2, R53.2, U9.16 (FMT), U9.19 (DGND), U9.3 (CPGND), U9.9 (AGND)

Commit message: WIP
Parts:
- R53: footprint (none) -> Resistor_SMD:R_1210_3225Metric
Changed lines of the file:
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@@
       (effects (font (size 1.27 1.27)))
     )
-    (property "Footprint" "" (at 79.375 172.593 90)
+    (property "Footprint" "Resistor_SMD:R_1210_3225Metric" (at 79.375 172.593 90)
       (effects (font (size 1.27 1.27)) hide)
     )

Commit message: WIP
Parts:
- removed R53: 0, Resistor_SMD:R_1210_3225Metric, symbol Device:R
- U10: value MCP1700x-120xxMB -> MCP1700T-3302E/MB
Connections:
- net GNDA is gone; now on net GND: C51.2, C52.2, C54.2, C55.2, C56.2, C57.2, C58.2, C59.2, J4.3 (EXT), JP2.1 (A), JP3.1 (A), R33.2, U9.16 (FMT), U9.19 (DGND), U9.3 (CPGND), U9.9 (AGND)

Commit message: WIP
Parts:
- added R46: 0, Resistor_SMD:R_0603_1608Metric, symbol Device:R
Connections:
- net GND: now also R46.1
- net at R36.2, U9.12 (SCK): now also R46.2
Changed lines of the file:
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@@
   (junction (at 130.175 49.53) (diameter 0) (color 0 0 0 0)
   )
+  (junction (at 153.67 117.475) (diameter 0) (color 0 0 0 0)
+  )
   (junction (at 139.7 117.475) (diameter 0) (color 0 0 0 0)
   )
@@
     (stroke (width 0) (type default))
   )
+  (wire (pts (xy 153.67 117.475) (xy 155.575 117.475))
+    (stroke (width 0) (type default))
+  )
   (wire (pts (xy 153.035 140.335) (xy 165.735 140.335))
     (stroke (width 0) (type default))
@@
     (stroke (width 0) (type default))
   )
+  (wire (pts (xy 139.7 120.015) (xy 139.7 126.365))
+    (stroke (width 0) (type default))
+  )
   (wire (pts (xy 144.145 114.935) (xy 139.7 114.935))
     (stroke (width 0) (type default))
@@
     (stroke (width 0) (type default))
   )
-  (wire (pts (xy 151.765 117.475) (xy 155.575 117.475))
+  (wire (pts (xy 151.765 117.475) (xy 153.67 117.475))
     (stroke (width 0) (type default))
   )
@@
     (stroke (width 0) (type default))
   )
+  (wire (pts (xy 151.765 120.015) (xy 153.67 120.015))
+    (stroke (width 0) (type default))
+  )
   (wire (pts (xy 97.155 57.785) (xy 97.155 49.53))
     (stroke (width 0) (type default))
@@
     (stroke (width 0) (type default))
   )
+  (wire (pts (xy 153.67 120.015) (xy 153.67 117.475))
+    (stroke (width 0) (type default))
+  )
   (wire (pts (xy 48.26 42.545) (xy 63.5 42.545))
     (stroke (width 0) (type default))
@@
   )
   (wire (pts (xy 116.84 40.005) (xy 105.41 40.005))
+    (stroke (width 0) (type default))
+  )
+  (wire (pts (xy 144.145 120.015) (xy 139.7 120.015))
     (stroke (width 0) (type default))
   )
@@
         (path "/487245ca-0c1f-4f9d-bc99-20c8f558090f/80e17ed4-cb43-4c12-a09c-75e0f0ffaba0"
           (reference "C51") (unit 1)
+        )
+      )
+    )
+  )
+  (symbol (lib_id "Device:R") (at 147.955 120.015 90) (unit 1)
+    (in_bom yes) (on_board yes) (dnp no)
+    (property "Reference" "R46" (at 142.875 118.745 90)
+      (effects (font (size 1.27 1.27)))
+    )
+    (property "Value" "0" (at 147.955 120.015 90)
+      (effects (font (size 1.27 1.27)))
+    )
+    (property "Footprint" "Resistor_SMD:R_0603_1608Metric" (at 147.955 121.793 90)
+      (effects (font (size 1.27 1.27)) hide)
+    )
+    (property "Datasheet" "~" (at 147.955 120.015 0)
+      (effects (font (size 1.27 1.27)) hide)
+    )
+    (pin "1")
+    (pin "2")
+    (instances
+      (project "dacattac-alpha"
+        (path "/487245ca-0c1f-4f9d-bc99-20c8f558090f/80e17ed4-cb43-4c12-a09c-75e0f0ffaba0"
+          (reference "R46") (unit 1)
         )
       )
@@
         )
       )
+    )
+  )
+  (symbol (lib_id "power:GND") (at 139.7 126.365 0) (unit 1)
+    (in_bom yes) (on_board yes) (dnp no)
+    (property "Reference" "#PWR012" (at 139.7 132.715 0)
+      (effects (font (size 1.27 1.27)) hide)
+    )
+    (property "Value" "GND" (at 139.7 130.175 0)
+      (effects (font (size 1.27 1.27)))
+    )
+    (property "Footprint" "" (at 139.7 126.365 0)
+      (effects (font (size 1.27 1.27)) hide)
+    )
+    (property "Datasheet" "" (at 139.7 126.365 0)
+      (effects (font (size 1.27 1.27)) hide)
+    )
+    (pin "1")
+    (instances
+      (project "dacattac-alpha"
+        (path "/487245ca-0c1f-4f9d-bc99-20c8f558090f/80e17ed4-cb43-4c12-a09c-75e0f0ffaba0"
+          (reference "#PWR012") (unit 1)
+        )
+      )

Commit message: Added / updated BOm
Parts:
- R32: value R -> 10k
- R33: value R -> 6k98
Changed lines of the file:
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@@
       (effects (font (size 1.27 1.27)))
     )
-    (property "Value" "R" (at 125.73 132.715 90)
+    (property "Value" "10k" (at 125.73 132.715 90)
       (effects (font (size 1.27 1.27)))
     )
@@
       (effects (font (size 1.27 1.27)) (justify left))
     )
-    (property "Value" "R" (at 147.955 146.05 90)
-      (effects (font (size 1.27 1.27)) (justify left))
-    )
+    (property "Value" "6k98" (at 147.955 147.955 90)
+      (effects (font (size 1.27 1.27)) (justify left))
+    )

Commit message: WIP
Connections:
- net +8V is gone; now on net VIN: R32.1
Changed lines of the file:
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@@
     )
   )
-  (global_label "+8V" (shape input) (at 107.315 132.715 180) (fields_autoplaced)
+  (global_label "VIN" (shape input) (at 107.315 132.715 180) (fields_autoplaced)
     (effects (font (size 1.27 1.27)) (justify right))
-    (property "Intersheetrefs" "${INTERSHEET_REFS}" (at 100.4593 132.715 0)
+    (property "Intersheetrefs" "${INTERSHEET_REFS}" (at 101.3059 132.715 0)
       (effects (font (size 1.27 1.27)) (justify right) hide)
     )
