File: hardware/alpha/audio.kicad_sch (KiCad schematic)
At the start: 29 parts, among them J4 AUDIO OUT, J6 I2C, P22 P22, Q1 2N7002, Q2 2N7002, U10 MCP1700T-3302E/MB, U9 PCM5102

Commit message: WIP
Parts:
- added L1: L, symbol Device:L
Connections:
- net VIN: now also L1.1; no longer C60.1, U10.2 (VI)
- new net: C60.1, L1.2, U10.2 (VI)
Other:
- moved on the sheet: C60, C61, U10

Commit message: WIP
Parts:
- L11: renamed from L1; footprint (none) -> Inductor_SMD:L_1210_3225Metric
- renumbered C60 to C55, C61 to C56, C55 to C59, C53 to C60, C56 to C61, C54 to C62, C59 to C63, C51 to C64, C52 to C65, J6 to J3, JP3 to JP2, JP2 to JP3, P22 to P2, Q1 to Q4, Q2 to Q5, R32 to R44, R34 to R45, R35 to R46, R37 to R47, R36 to R48, R46 to R49, R33 to R50, R29 to R51, R30 to R52, U10 to U8
