File: hardware/alpha/power.kicad_sch (KiCad schematic)
At the start: 1 part, among them U2 TPS61170DRVR

Commit message: Updated
Parts:
- added C62: 10n, symbol Device:C
- added C63, C68: 10u, symbol Device:C
- added C64: 4.7u, symbol Device:C
- added C65: 4n7, symbol Device:C
- added C66: 220n, symbol Device:C
- added C67: C, symbol Device:C
- added D1, D2: MBR0540T1, symbol Device:D_Schottky
- added J1: EXT +/- 8V, symbol Connector_Generic:Conn_01x03
- added L15: 10uH, symbol Device:L
- added L16: 4u7, symbol Device:L
- added P20: P20, symbol Connector_Generic:Conn_02x11_Odd_Even
- added Q3: IRF7324, Package_SO:SOIC-8_3.9x4.9mm_P1.27mm, symbol Transistor_FET:IRF7324
- added R38, R39, R41, R42, R45: R, symbol Device:R
- added R40: 4k99, symbol Device:R
- added U11: TPS63700DRCT, TPS63700DRCT:VREG_V62_16624-01YE, symbol TPS63700:TPS63700DRCT
Connections:
- net at U2.1 (FB): now also R38.2, R39.1
- net at U2.2 (COMP): now also R40.2
- net GND: now reaches U2.3 (GND)
- net GND: now also U2.7 (THERMALPAD), C62.2, C63.2, C64.2, C65.2, C66.2, C67.2, C68.2, J1.2 (Pin_2), L16.1, R39.2, U11.11 (EP), U11.2 (GND), U11.7 (PS_GND)
- net at U2.4 (SW): now also D1.2 (A), L15.2
- net VIN: now reaches U2.5 (CTRL)
- net VIN: now also U2.6 (VIN), C64.1, C68.1, L15.1, Q3.7 (D1), Q3.8 (D1), R45.2, U11.5 (IN)
- new net: C67.1, R45.1, U11.3 (VIN), U11.4 (EN)
- new net: C65.1, U11.1 (COMP)
- new net: R41.1, R42.2, U11.9 (FB)
- new net: D2.1 (K), L16.2, U11.6 (SW)
- new net: C62.1, R40.1
- new net: C66.1, R42.1, U11.10 (VREF)
- new net +8V: C63.1, D1.1 (K), J1.1 (Pin_1), R38.1
- new net -8V: D2.2 (A), J1.3 (Pin_3), R41.2, U11.8 (OUT)
- new net VBUS: P20.21 (Pin_21), Q3.1 (S1)
- new net VBUSCTRL: P20.17 (Pin_17), Q3.2 (G1)

Commit message: WIP
Parts:
- C62, C63, C64, C65, C66, C67, C68: footprint (none) -> Capacitor_SMD:C_0603_1608Metric
- D1, D2: footprint (none) -> Diode_SMD:D_SOD-123
- J1: footprint (none) -> Connector_Molex:Molex_KK-254_AE-6410-03A_1x03_P2.54mm_Vertical
- L15: value 10uH -> 10u
- R38, R39, R40, R41, R42, R45: footprint (none) -> Resistor_SMD:R_0603_1608Metric
Changed lines of the file:
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@@
       (effects (font (size 1.27 1.27)))
     )
-    (property "Footprint" "" (at 175.895 43.18 0)
+    (property "Footprint" "Diode_SMD:D_SOD-123" (at 175.895 43.18 0)
       (effects (font (size 1.27 1.27)) hide)
     )
@@
       (effects (font (size 1.27 1.27)) (justify left))
     )
-    (property "Footprint" "" (at 117.8052 106.68 0)
+    (property "Footprint" "Capacitor_SMD:C_0603_1608Metric" (at 117.8052 106.68 0)
       (effects (font (size 1.27 1.27)) hide)
     )
@@
       (effects (font (size 1.27 1.27)) (justify left))
     )
-    (property "Footprint" "" (at 225.425 79.375 0)
+    (property "Footprint" "Connector_Molex:Molex_KK-254_AE-6410-03A_1x03_P2.54mm_Vertical" (at 225.425 79.375 0)
       (effects (font (size 1.27 1.27)) hide)
     )
@@
       (effects (font (size 1.27 1.27)) (justify left))
     )
-    (property "Footprint" "" (at 128.6002 133.985 0)
+    (property "Footprint" "Capacitor_SMD:C_0603_1608Metric" (at 128.6002 133.985 0)
       (effects (font (size 1.27 1.27)) hide)
     )
@@
       (effects (font (size 1.27 1.27)) (justify left))
     )
-    (property "Footprint" "" (at 188.722 113.665 90)
+    (property "Footprint" "Resistor_SMD:R_0603_1608Metric" (at 188.722 113.665 90)
       (effects (font (size 1.27 1.27)) hide)
     )
@@
       (effects (font (size 1.27 1.27)) (justify left))
     )
-    (property "Footprint" "" (at 121.6152 55.245 0)
+    (property "Footprint" "Capacitor_SMD:C_0603_1608Metric" (at 121.6152 55.245 0)
       (effects (font (size 1.27 1.27)) hide)
     )
@@
       (effects (font (size 1.27 1.27)) (justify left))
     )
-    (property "Footprint" "" (at 126.492 105.41 90)
+    (property "Footprint" "Resistor_SMD:R_0603_1608Metric" (at 126.492 105.41 90)
       (effects (font (size 1.27 1.27)) hide)
     )
@@
       (effects (font (size 1.27 1.27)))
     )
-    (property "Footprint" "" (at 180.975 119.38 0)
+    (property "Footprint" "Diode_SMD:D_SOD-123" (at 180.975 119.38 0)
       (effects (font (size 1.27 1.27)) hide)
     )
@@
       (effects (font (size 1.27 1.27)) (justify left))
     )
-    (property "Footprint" "" (at 121.6152 74.93 0)
+    (property "Footprint" "Capacitor_SMD:C_0603_1608Metric" (at 121.6152 74.93 0)
       (effects (font (size 1.27 1.27)) hide)
     )
@@
       (effects (font (size 1.27 1.27)) (justify left))
     )
-    (property "Footprint" "" (at 201.6252 106.68 0)
+    (property "Footprint" "Capacitor_SMD:C_0603_1608Metric" (at 201.6252 106.68 0)
       (effects (font (size 1.27 1.27)) hide)
     )
@@
       (effects (font (size 1.27 1.27)) (justify left))
     )
-    (property "Footprint" "" (at 180.467 59.69 90)
+    (property "Footprint" "Resistor_SMD:R_0603_1608Metric" (at 180.467 59.69 90)
       (effects (font (size 1.27 1.27)) hide)
     )
@@
       (effects (font (size 1.27 1.27)) (justify left))
     )
-    (property "Footprint" "" (at 117.8052 133.985 0)
+    (property "Footprint" "Capacitor_SMD:C_0603_1608Metric" (at 117.8052 133.985 0)
       (effects (font (size 1.27 1.27)) hide)
     )
@@
       (effects (font (size 1.27 1.27)))
     )
-    (property "Footprint" "" (at 127 67.183 90)
+    (property "Footprint" "Resistor_SMD:R_0603_1608Metric" (at 127 67.183 90)
       (effects (font (size 1.27 1.27)) hide)
     )
@@
       (effects (font (size 1.27 1.27)) (justify left))
     )
-    (property "Footprint" "" (at 180.467 70.485 90)
+    (property "Footprint" "Resistor_SMD:R_0603_1608Metric" (at 180.467 70.485 90)
       (effects (font (size 1.27 1.27)) hide)
     )
@@
       (effects (font (size 1.27 1.27)) (justify left))
     )
-    (property "Footprint" "" (at 188.722 102.87 90)
+    (property "Footprint" "Resistor_SMD:R_0603_1608Metric" (at 188.722 102.87 90)
       (effects (font (size 1.27 1.27)) hide)
     )
@@
       (effects (font (size 1.27 1.27)) (justify left))
     )
-    (property "Footprint" "" (at 194.6402 53.34 0)
+    (property "Footprint" "Capacitor_SMD:C_0603_1608Metric" (at 194.6402 53.34 0)
       (effects (font (size 1.27 1.27)) hide)
     )
@@
       (effects (font (size 1.27 1.27)))
     )
-    (property "Value" "10uH" (at 151.13 40.005 90)
-      (effects (font (size 1.27 1.27)))
-    )
+    (property "Value" "10u" (at 151.13 40.005 90)
+      (effects (font (size 1.27 1.27)))
+    )

Commit message: WIP
Changed lines of the file:
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@@
   (junction (at 170.18 125.73) (diameter 0) (color 0 0 0 0)
   )
+  (junction (at 100.965 64.77) (diameter 0) (color 0 0 0 0)
+  )
+  (junction (at 170.18 128.27) (diameter 0) (color 0 0 0 0)
+  )
   (junction (at 218.44 119.38) (diameter 0) (color 0 0 0 0)
   )
-  (junction (at 100.965 64.77) (diameter 0) (color 0 0 0 0)
-  )
-  (junction (at 170.18 128.27) (diameter 0) (color 0 0 0 0)
-  )
   (junction (at 218.44 43.18) (diameter 0) (color 0 0 0 0)
   )
@@
   (junction (at 130.81 53.975) (diameter 0) (color 0 0 0 0)
   )
-  (wire (pts (xy 218.44 119.38) (xy 222.25 119.38))
-    (stroke (width 0) (type default))
-  )
   (wire (pts (xy 100.965 115.57) (xy 100.965 64.77))
     (stroke (width 0) (type default))
@@
     (stroke (width 0) (type default))
   )
+  (wire (pts (xy 218.44 41.275) (xy 218.44 43.18))
+    (stroke (width 0) (type default))
+  )
   (wire (pts (xy 128.27 100.33) (xy 132.715 100.33))
     (stroke (width 0) (type default))
@@
     (stroke (width 0) (type default))
   )
+  (wire (pts (xy 218.44 119.38) (xy 218.44 121.285))
+    (stroke (width 0) (type default))
+  )
   (wire (pts (xy 193.675 43.18) (xy 193.675 45.72))
     (stroke (width 0) (type default))
@@
   )
   (wire (pts (xy 128.27 115.57) (xy 128.27 109.22))
-    (stroke (width 0) (type default))
-  )
-  (wire (pts (xy 218.44 43.18) (xy 222.25 43.18))
     (stroke (width 0) (type default))
   )
@@
     (property "Intersheetrefs" "${INTERSHEET_REFS}" (at 91.7809 43.18 0)
       (effects (font (size 1.27 1.27)) (justify right) hide)
-    )
-  )
-  (global_label "-8V" (shape input) (at 222.25 119.38 0) (fields_autoplaced)
-    (effects (font (size 1.27 1.27)) (justify left))
-    (property "Intersheetrefs" "${INTERSHEET_REFS}" (at 229.1057 119.38 0)
-      (effects (font (size 1.27 1.27)) (justify left) hide)
-    )
-  )
-  (global_label "+8V" (shape input) (at 222.25 43.18 0) (fields_autoplaced)
-    (effects (font (size 1.27 1.27)) (justify left))
-    (property "Intersheetrefs" "${INTERSHEET_REFS}" (at 229.1057 43.18 0)
-      (effects (font (size 1.27 1.27)) (justify left) hide)
     )
   )
@@
     )
   )
+  (symbol (lib_id "power:+8V") (at 218.44 41.275 0) (unit 1)
+    (in_bom yes) (on_board yes) (dnp no)
+    (property "Reference" "#PWR049" (at 218.44 45.085 0)
+      (effects (font (size 1.27 1.27)) hide)
+    )
+    (property "Value" "+8V" (at 218.44 36.83 0)
+      (effects (font (size 1.27 1.27)))
+    )
+    (property "Footprint" "" (at 218.44 41.275 0)
+      (effects (font (size 1.27 1.27)) hide)
+    )
+    (property "Datasheet" "" (at 218.44 41.275 0)
+      (effects (font (size 1.27 1.27)) hide)
+    )
+    (pin "1")
+    (instances
+      (project "dacattac-alpha"
+        (path "/487245ca-0c1f-4f9d-bc99-20c8f558090f/b8114b5f-896b-4ea4-b003-c1721b486c01"
+          (reference "#PWR049") (unit 1)
+        )
+      )
+    )
+  )
   (symbol (lib_id "Device:R") (at 182.245 70.485 0) (unit 1)
     (in_bom yes) (on_board yes) (dnp no) (fields_autoplaced)
@@
         )
       )
+    )
+  )
+  (symbol (lib_id "power:-8V") (at 218.44 121.285 180) (unit 1)
+    (in_bom yes) (on_board yes) (dnp no) (fields_autoplaced)
+    (property "Reference" "#PWR050" (at 218.44 123.825 0)
+      (effects (font (size 1.27 1.27)) hide)
+    )
+    (property "Value" "-8V" (at 218.44 125.73 0)
+      (effects (font (size 1.27 1.27)))
+    )
+    (property "Footprint" "" (at 218.44 121.285 0)
+      (effects (font (size 1.27 1.27)) hide)
+    )
+    (property "Datasheet" "" (at 218.44 121.285 0)
+      (effects (font (size 1.27 1.27)) hide)
+    )
+    (pin "1")
+    (instances
+      (project "dacattac-alpha"
+        (path "/487245ca-0c1f-4f9d-bc99-20c8f558090f/b8114b5f-896b-4ea4-b003-c1721b486c01"
+          (reference "#PWR050") (unit 1)
+        )
+      )

Commit message: WIP
Parts:
- L15, L16: footprint (none) -> Inductor_SMD:L_1210_3225Metric
- P20: footprint (none) -> hackrf:GSG-HEADER-2x11
Changed lines of the file:
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@@
       (effects (font (size 1.27 1.27)))
     )
-    (property "Footprint" "" (at 55.245 72.39 0)
+    (property "Footprint" "hackrf:GSG-HEADER-2x11" (at 55.245 72.39 0)
       (effects (font (size 1.27 1.27)) hide)
     )
@@
       (effects (font (size 1.27 1.27)) (justify right))
     )
-    (property "Footprint" "" (at 174.625 125.095 0)
+    (property "Footprint" "Inductor_SMD:L_1210_3225Metric" (at 174.625 125.095 0)
       (effects (font (size 1.27 1.27)) hide)
     )
@@
       (effects (font (size 1.27 1.27)))
     )
-    (property "Footprint" "" (at 151.13 43.18 0)
-      (effects (font (size 1.27 1.27)) hide)
-    )
+    (property "Footprint" "Inductor_SMD:L_1210_3225Metric" (at 151.13 43.18 0)
+      (effects (font (size 1.27 1.27)) hide)
+    )

Commit message: WIP
Parts:
- added J10, J11, J12, J13, J14, J15: HOLE, hackrf:GSG-HOLE126MIL-COPPER, symbol Connector_Generic:Conn_01x01
Connections:
- net GND: now also J10.1 (Pin_1), J11.1 (Pin_1), J12.1 (Pin_1), J13.1 (Pin_1), J14.1 (Pin_1), J15.1 (Pin_1)

Commit message: WIP
Parts:
- removed Q3: IRF7324, Package_SO:SOIC-8_3.9x4.9mm_P1.27mm, symbol Transistor_FET:IRF7324
- added P28: P28, hackrf:GSG-HEADER-2x11, symbol Connector_Generic:Conn_02x11_Odd_Even
- added Q3: IRLML2244, Package_TO_SOT_SMD:SOT-23, symbol Transistor_FET:IRLML5203
- C63, C68: footprint Capacitor_SMD:C_0603_1608Metric -> Capacitor_SMD:C_1210_3225Metric
Connections:
- net GND: now also P28.12 (Pin_12), P28.2 (Pin_2)
- net VBUS: now also Q3.2 (S)
- net VBUSCTRL: now also Q3.1 (G)
- net VIN: now also Q3.3 (D)
- new net +3.3V_HACKRF: P28.1 (Pin_1)
Changed lines of the file:
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@@
   (junction (at 67.945 169.545) (diameter 0) (color 0 0 0 0)
   )
+  (junction (at 64.135 118.745) (diameter 0) (color 0 0 0 0)
+  )
   (junction (at 120.65 43.18) (diameter 0) (color 0 0 0 0)
   )
@@
     (stroke (width 0) (type default))
   )
+  (wire (pts (xy 60.325 106.045) (xy 64.135 106.045))
+    (stroke (width 0) (type default))
+  )
   (wire (pts (xy 100.965 43.18) (xy 97.79 43.18))
     (stroke (width 0) (type default))
   )
+  (wire (pts (xy 43.815 100.965) (xy 43.815 106.045))
+    (stroke (width 0) (type default))
+  )
   (wire (pts (xy 186.69 119.38) (xy 190.5 119.38))
     (stroke (width 0) (type default))
@@
     (stroke (width 0) (type default))
   )
+  (wire (pts (xy 64.135 118.745) (xy 64.135 136.525))
+    (stroke (width 0) (type default))
+  )
   (wire (pts (xy 220.345 76.835) (xy 218.44 76.835))
     (stroke (width 0) (type default))
@@
     (stroke (width 0) (type default))
   )
+  (wire (pts (xy 43.815 106.045) (xy 47.625 106.045))
+    (stroke (width 0) (type default))
+  )
   (wire (pts (xy 190.5 97.79) (xy 200.66 97.79))
     (stroke (width 0) (type default))
   )
+  (wire (pts (xy 64.135 106.045) (xy 64.135 118.745))
+    (stroke (width 0) (type default))
+  )
   (wire (pts (xy 83.185 64.77) (xy 83.185 74.93))
     (stroke (width 0) (type default))
@@
   )
   (wire (pts (xy 170.18 43.18) (xy 170.18 53.975))
+    (stroke (width 0) (type default))
+  )
+  (wire (pts (xy 60.325 118.745) (xy 64.135 118.745))
     (stroke (width 0) (type default))
   )
@@
     )
   )
+  (symbol (lib_id "Transistor_FET:IRLML5203") (at 80.645 80.01 0) (unit 1)
+    (in_bom yes) (on_board yes) (dnp no) (fields_autoplaced)
+    (property "Reference" "Q3" (at 86.36 78.74 0)
+      (effects (font (size 1.27 1.27)) (justify left))
+    )
+    (property "Value" "IRLML2244" (at 86.36 81.28 0)
+      (effects (font (size 1.27 1.27)) (justify left))
+    )
+    (property "Footprint" "Package_TO_SOT_SMD:SOT-23" (at 85.725 81.915 0)
+      (effects (font (size 1.27 1.27) italic) (justify left) hide)
+    )
+    (property "Datasheet" "https://www.infineon.com/dgdl/irlml5203pbf.pdf?fileId=5546d462533600a40153566868da261d" (at 80.645 80.01 0)
+      (effects (font (size 1.27 1.27)) (justify left) hide)
+    )
+    (pin "2")
+    (pin "3")
+    (pin "1")
+    (instances
+      (project "dacattac-alpha"
+        (path "/487245ca-0c1f-4f9d-bc99-20c8f558090f/b8114b5f-896b-4ea4-b003-c1721b486c01"
+          (reference "Q3") (unit 1)
+        )
+      )
+    )
+  )
   (symbol (lib_id "Device:C") (at 116.84 102.87 0) (unit 1)
     (in_bom yes) (on_board yes) (dnp no) (fields_autoplaced)
@@
         (path "/487245ca-0c1f-4f9d-bc99-20c8f558090f/b8114b5f-896b-4ea4-b003-c1721b486c01"
           (reference "#PWR081") (unit 1)
-        )
-      )
-    )
-  )
-  (symbol (lib_id "Transistor_FET:IRF7324") (at 80.645 80.01 0) (unit 1)
-    (in_bom yes) (on_board yes) (dnp no)
-    (property "Reference" "Q3" (at 86.36 78.74 0)
-      (effects (font (size 1.27 1.27)) (justify left))
-    )
-    (property "Value" "IRF7324" (at 86.36 81.28 0)
-      (effects (font (size 1.27 1.27)) (justify left))
-    )
-    (property "Footprint" "Package_SO:SOIC-8_3.9x4.9mm_P1.27mm" (at 85.725 81.915 0)
-      (effects (font (size 1.27 1.27)) (justify left) hide)
-    )
-    (property "Datasheet" "http://www.infineon.com/dgdl/irf7324pbf.pdf?fileId=5546d462533600a4015355f5f0861b4b" (at 83.185 80.01 0)
-      (effects (font (size 1.27 1.27)) (justify left) hide)
-    )
-    (pin "7")
-    (pin "5")
-    (pin "2")
-    (pin "6")
-    (pin "4")
-    (pin "1")
-    (pin "8")
-    (pin "3")
-    (instances
-      (project "dacattac-alpha"
-        (path "/487245ca-0c1f-4f9d-bc99-20c8f558090f/b8114b5f-896b-4ea4-b003-c1721b486c01"
-          (reference "Q3") (unit 1)
         )
       )
@@
     )
   )
+  (symbol (lib_id "Connector_Generic:Conn_02x11_Odd_Even") (at 52.705 118.745 0) (unit 1)
+    (in_bom yes) (on_board yes) (dnp no)
+    (property "Reference" "P28" (at 53.975 100.33 0)
+      (effects (font (size 1.27 1.27)))
+    )
+    (property "Value" "P28" (at 53.975 102.87 0)
+      (effects (font (size 1.27 1.27)))
+    )
+    (property "Footprint" "hackrf:GSG-HEADER-2x11" (at 52.705 118.745 0)
+      (effects (font (size 1.27 1.27)) hide)
+    )
+    (property "Datasheet" "~" (at 52.705 118.745 0)
+      (effects (font (size 1.27 1.27)) hide)
+    )
+    (pin "7")
+    (pin "19")
+    (pin "18")
+    (pin "17")
+    (pin "10")
+    (pin "6")
+    (pin "9")
+    (pin "14")
+    (pin "20")
+    (pin "13")
+    (pin "11")
+    (pin "8")
+    (pin "15")
+    (pin "16")
+    (pin "4")
+    (pin "2")
+    (pin "21")
+    (pin "3")
+    (pin "1")
+    (pin "12")
+    (pin "5")
+    (pin "22")
+    (instances
+      (project "dacattac-alpha"
+        (path "/487245ca-0c1f-4f9d-bc99-20c8f558090f/b8114b5f-896b-4ea4-b003-c1721b486c01"
+          (reference "P28") (unit 1)
+        )
+      )
+    )
+  )
   (symbol (lib_id "Connector_Generic:Conn_01x01") (at 62.865 163.195 90) (unit 1)
     (in_bom yes) (on_board yes) (dnp no)
@@
       (effects (font (size 1.27 1.27)) (justify left))
     )
-    (property "Footprint" "Capacitor_SMD:C_0603_1608Metric" (at 117.8052 133.985 0)
+    (property "Footprint" "Capacitor_SMD:C_1210_3225Metric" (at 117.8052 133.985 0)
       (effects (font (size 1.27 1.27)) hide)
     )
@@
     )
   )
+  (symbol (lib_id "+3.3v_hackrf:+3.3V_HACKRF") (at 43.815 100.965 0) (unit 1)
+    (in_bom yes) (on_board yes) (dnp no) (fields_autoplaced)
+    (property "Reference" "#PWR0103" (at 47.625 102.235 0)
+      (effects (font (size 1.27 1.27)) hide)
+    )
+    (property "Value" "+3.3V_HACKRF" (at 43.815 96.52 0)
+      (effects (font (size 1.27 1.27)))
+    )
+    (property "Footprint" "" (at 43.815 100.965 0)
+      (effects (font (size 1.27 1.27)) hide)
+    )
+    (property "Datasheet" "" (at 43.815 100.965 0)
+      (effects (font (size 1.27 1.27)) hide)
+    )
+    (pin "1")
+    (instances
+      (project "dacattac-alpha"
+        (path "/487245ca-0c1f-4f9d-bc99-20c8f558090f/b8114b5f-896b-4ea4-b003-c1721b486c01"
+          (reference "#PWR0103") (unit 1)
+        )
+      )
+    )
+  )
   (symbol (lib_id "power:+8V") (at 218.44 41.275 0) (unit 1)
     (in_bom yes) (on_board yes) (dnp no)
@@
     )
   )
+  (symbol (lib_id "power:GND") (at 64.135 136.525 0) (unit 1)
+    (in_bom yes) (on_board yes) (dnp no) (fields_autoplaced)
+    (property "Reference" "#PWR0102" (at 64.135 142.875 0)
+      (effects (font (size 1.27 1.27)) hide)
+    )
+    (property "Value" "GND" (at 64.135 141.605 0)
+      (effects (font (size 1.27 1.27)))
+    )
+    (property "Footprint" "" (at 64.135 136.525 0)
+      (effects (font (size 1.27 1.27)) hide)
+    )
+    (property "Datasheet" "" (at 64.135 136.525 0)
+      (effects (font (size 1.27 1.27)) hide)
+    )
+    (pin "1")
+    (instances
+      (project "dacattac-alpha"
+        (path "/487245ca-0c1f-4f9d-bc99-20c8f558090f/b8114b5f-896b-4ea4-b003-c1721b486c01"
+          (reference "#PWR0102") (unit 1)
+        )
+      )
+    )
+  )
   (symbol (lib_id "Device:R") (at 190.5 102.87 0) (unit 1)
     (in_bom yes) (on_board yes) (dnp no) (fields_autoplaced)
@@
       (effects (font (size 1.27 1.27)) (justify left))
     )
-    (property "Footprint" "Capacitor_SMD:C_0603_1608Metric" (at 194.6402 53.34 0)
-      (effects (font (size 1.27 1.27)) hide)
-    )
+    (property "Footprint" "Capacitor_SMD:C_1210_3225Metric" (at 194.6402 53.34 0)
+      (effects (font (size 1.27 1.27)) hide)
+    )

Commit message: WIP
Parts:
- C64: footprint Capacitor_SMD:C_0603_1608Metric -> Capacitor_SMD:C_1210_3225Metric
- J1: value EXT +/- 8V -> EXT POWER
Changed lines of the file:
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@@
       (effects (font (size 1.27 1.27)) (justify left))
     )
-    (property "Value" "EXT +/- 8V" (at 228.6 80.645 0)
+    (property "Value" "EXT POWER" (at 228.6 80.645 0)
       (effects (font (size 1.27 1.27)) (justify left))
     )
@@
       (effects (font (size 1.27 1.27)) (justify left))
     )
-    (property "Footprint" "Capacitor_SMD:C_0603_1608Metric" (at 121.6152 55.245 0)
+    (property "Footprint" "Capacitor_SMD:C_1210_3225Metric" (at 121.6152 55.245 0)
       (effects (font (size 1.27 1.27)) hide)
     )

Commit message: WIP
Connections:
- net LSYNC: now reaches P28.16 (Pin_16)
Changed lines of the file:
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@@
+    (stroke (width 0) (type default))
+  )
+  (wire (pts (xy 60.325 123.825) (xy 68.58 123.825))
     (stroke (width 0) (type default))
   )
@@
     )
   )
+  (global_label "LSYNC" (shape input) (at 68.58 123.825 0) (fields_autoplaced)
+    (effects (font (size 1.27 1.27)) (justify left))
+    (property "Intersheetrefs" "${INTERSHEET_REFS}" (at 77.4919 123.825 0)
+      (effects (font (size 1.27 1.27)) (justify left) hide)
+    )
+  )
