File: hardware/alpha/power.kicad_sch (KiCad schematic)
At the start: 29 parts, among them J1 EXT POWER, J10 HOLE, J11 HOLE, J12 HOLE, J13 HOLE, J14 HOLE, J15 HOLE, P20 P20, P28 P28, Q3 IRLML2244, U11 TPS63700DRCT, U2 TPS61170DRVR

Commit message: WIP
Connections:
- net GND: no longer J10.1 (Pin_1), J11.1 (Pin_1)
Changed lines of the file:
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@@
   (junction (at 190.5 119.38) (diameter 0) (color 0 0 0 0)
   )
-  (junction (at 47.625 169.545) (diameter 0) (color 0 0 0 0)
-  )
   (junction (at 186.69 119.38) (diameter 0) (color 0 0 0 0)
   )
@@
   (junction (at 182.245 43.18) (diameter 0) (color 0 0 0 0)
   )
-  (junction (at 52.705 169.545) (diameter 0) (color 0 0 0 0)
-  )
   (junction (at 130.81 53.975) (diameter 0) (color 0 0 0 0)
   )
@@
     (stroke (width 0) (type default))
   )
-  (wire (pts (xy 42.545 169.545) (xy 47.625 169.545))
-    (stroke (width 0) (type default))
-  )
   (wire (pts (xy 170.18 123.19) (xy 170.18 125.73))
     (stroke (width 0) (type default))
@@
     (stroke (width 0) (type default))
   )
-  (wire (pts (xy 47.625 169.545) (xy 52.705 169.545))
-    (stroke (width 0) (type default))
-  )
   (wire (pts (xy 170.18 43.18) (xy 170.18 53.975))
     (stroke (width 0) (type default))
@@
     (stroke (width 0) (type default))
   )
-  (wire (pts (xy 42.545 168.275) (xy 42.545 169.545))
-    (stroke (width 0) (type default))
-  )
   (wire (pts (xy 130.81 65.405) (xy 132.715 65.405))
     (stroke (width 0) (type default))
@@
     (stroke (width 0) (type default))
   )
-  (wire (pts (xy 47.625 168.275) (xy 47.625 169.545))
-    (stroke (width 0) (type default))
-  )

Commit message: WIP
Connections:
- net GND: now also J10.1 (Pin_1), J11.1 (Pin_1)
Changed lines of the file:
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@@
   (junction (at 120.65 43.18) (diameter 0) (color 0 0 0 0)
   )
+  (junction (at 52.705 169.545) (diameter 0) (color 0 0 0 0)
+  )
   (junction (at 170.18 43.18) (diameter 0) (color 0 0 0 0)
   )
@@
   (junction (at 128.27 97.79) (diameter 0) (color 0 0 0 0)
   )
+  (junction (at 47.625 169.545) (diameter 0) (color 0 0 0 0)
+  )
   (junction (at 190.5 107.95) (diameter 0) (color 0 0 0 0)
   )
@@
     (stroke (width 0) (type default))
   )
+  (wire (pts (xy 42.545 169.545) (xy 42.545 168.275))
+    (stroke (width 0) (type default))
+  )
   (wire (pts (xy 218.44 119.38) (xy 218.44 121.285))
     (stroke (width 0) (type default))
@@
     (stroke (width 0) (type default))
   )
+  (wire (pts (xy 47.625 169.545) (xy 42.545 169.545))
+    (stroke (width 0) (type default))
+  )
   (wire (pts (xy 130.81 56.515) (xy 130.81 53.975))
     (stroke (width 0) (type default))
@@
     (stroke (width 0) (type default))
   )
+  (wire (pts (xy 47.625 168.275) (xy 47.625 169.545))
+    (stroke (width 0) (type default))
+  )
+  (wire (pts (xy 52.705 169.545) (xy 47.625 169.545))
+    (stroke (width 0) (type default))
+  )

Commit message: WIP
Parts:
- added C79: 22u, Capacitor_SMD:C_1210_3225Metric, symbol Device:C
Connections:
- net -8V: now also C79.1
- net GND: now also C79.2
Changed lines of the file:
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@@
   (junction (at 182.245 43.18) (diameter 0) (color 0 0 0 0)
   )
+  (junction (at 200.66 119.38) (diameter 0) (color 0 0 0 0)
+  )
   (junction (at 130.81 53.975) (diameter 0) (color 0 0 0 0)
   )
@@
     (stroke (width 0) (type default))
   )
+  (wire (pts (xy 200.66 119.38) (xy 218.44 119.38))
+    (stroke (width 0) (type default))
+  )
   (wire (pts (xy 220.345 81.915) (xy 218.44 81.915))
     (stroke (width 0) (type default))
@@
     (stroke (width 0) (type default))
   )
+  (wire (pts (xy 200.66 129.54) (xy 200.66 131.445))
+    (stroke (width 0) (type default))
+  )
   (wire (pts (xy 47.625 169.545) (xy 42.545 169.545))
     (stroke (width 0) (type default))
@@
     (stroke (width 0) (type default))
   )
-  (wire (pts (xy 190.5 119.38) (xy 218.44 119.38))
+  (wire (pts (xy 190.5 119.38) (xy 200.66 119.38))
     (stroke (width 0) (type default))
   )
@@
   )
   (wire (pts (xy 182.245 43.18) (xy 193.675 43.18))
+    (stroke (width 0) (type default))
+  )
+  (wire (pts (xy 200.66 119.38) (xy 200.66 121.92))
     (stroke (width 0) (type default))
   )
@@
       (effects (font (size 1.27 1.27)) hide)
     )
-    (property "Value" "GND" (at 116.84 112.395 0)
+    (property "Value" "GND" (at 116.84 111.76 0)
       (effects (font (size 1.27 1.27)))
     )
@@
       (effects (font (size 1.27 1.27)) hide)
     )
-    (property "Value" "GND" (at 170.18 135.89 0)
+    (property "Value" "GND" (at 170.18 135.255 0)
       (effects (font (size 1.27 1.27)))
     )
@@
         (path "/487245ca-0c1f-4f9d-bc99-20c8f558090f/b8114b5f-896b-4ea4-b003-c1721b486c01"
           (reference "#PWR076") (unit 1)
+        )
+      )
+    )
+  )
+  (symbol (lib_id "power:GND") (at 200.66 131.445 0) (unit 1)
+    (in_bom yes) (on_board yes) (dnp no)
+    (property "Reference" "#PWR01" (at 200.66 137.795 0)
+      (effects (font (size 1.27 1.27)) hide)
+    )
+    (property "Value" "GND" (at 200.66 135.255 0)
+      (effects (font (size 1.27 1.27)))
+    )
+    (property "Footprint" "" (at 200.66 131.445 0)
+      (effects (font (size 1.27 1.27)) hide)
+    )
+    (property "Datasheet" "" (at 200.66 131.445 0)
+      (effects (font (size 1.27 1.27)) hide)
+    )
+    (pin "1")
+    (instances
+      (project "dacattac-alpha"
+        (path "/487245ca-0c1f-4f9d-bc99-20c8f558090f/b8114b5f-896b-4ea4-b003-c1721b486c01"
+          (reference "#PWR01") (unit 1)
         )
       )
@@
     )
   )
+  (symbol (lib_id "Device:C") (at 200.66 125.73 0) (unit 1)
+    (in_bom yes) (on_board yes) (dnp no) (fields_autoplaced)
+    (property "Reference" "C79" (at 204.47 124.46 0)
+      (effects (font (size 1.27 1.27)) (justify left))
+    )
+    (property "Value" "22u" (at 204.47 127 0)
+      (effects (font (size 1.27 1.27)) (justify left))
+    )
+    (property "Footprint" "Capacitor_SMD:C_1210_3225Metric" (at 201.6252 129.54 0)
+      (effects (font (size 1.27 1.27)) hide)
+    )
+    (property "Datasheet" "~" (at 200.66 125.73 0)
+      (effects (font (size 1.27 1.27)) hide)
+    )
+    (pin "2")
+    (pin "1")
+    (instances
+      (project "dacattac-alpha"
+        (path "/487245ca-0c1f-4f9d-bc99-20c8f558090f/b8114b5f-896b-4ea4-b003-c1721b486c01"
+          (reference "C79") (unit 1)
+        )
+      )
+    )
+  )
   (symbol (lib_id "power:GND") (at 174.625 131.445 0) (unit 1)
     (in_bom yes) (on_board yes) (dnp no)
@@
       (effects (font (size 1.27 1.27)) hide)
     )
-    (property "Value" "GND" (at 174.625 135.89 0)
-      (effects (font (size 1.27 1.27)))
-    )
+    (property "Value" "GND" (at 174.625 135.255 0)
+      (effects (font (size 1.27 1.27)))
+    )

Commit message: Added / updated BOm
Parts:
- added C5, C6: 33u, Capacitor_SMD:C_1210_3225Metric, symbol Device:C
- added C7, C71, C72, C73, C74, C77, C78, C8: 100n, Capacitor_SMD:C_0603_1608Metric, symbol Device:C
- added L1, L2, L3, L4: 5u6, Inductor_SMD:L_1210_3225Metric, symbol Device:L
- added U12: L79L05_SO8, Package_SO:SOIC-8_3.9x4.9mm_P1.27mm, symbol Regulator_Linear:L79L05_SO8
- added U6: TLE2082, Package_SO:SOIC-8_3.9x4.9mm_P1.27mm, symbol Amplifier_Operational:AD8620
- added U8: L78L05_SO8, Package_SO:SOIC-8_3.9x4.9mm_P1.27mm, symbol Regulator_Linear:L78L05_SO8
- R38: value R -> 55k6
- R39: value R -> 10k
- R41: value R -> 988k
- R42: value R -> 150k
- R45: value R -> 10
Connections:
- net +8V: now also C71.1, L1.1
- net -8V: now also C72.2, L2.1
- net GND: now also C5.2, C6.1, C7.2, C71.2, C72.1, C73.2, C74.1, C77.2, C78.1, C8.1, U12.5 (GND), U8.2 (GND), U8.3 (GND), U8.6 (GND), U8.7 (GND)
- new net: C74.2, L2.2, U12.2 (IN), U12.3 (IN), U12.6 (IN), U12.7 (IN)
- new net: C73.1, L1.2, U8.8 (IN)
- new net +5V: C77.1, L3.1, U8.1 (OUT)
- new net +5VA: C5.1, C7.1, L3.2, U6.8 (V+)
- new net -5V: C78.2, L4.1, U12.1 (OUT)
- new net -5VA: C6.2, C8.2, L4.2, U6.4 (V-)
Other:
- note added: "DAC POWER FILTERING / REGULATION"
- moved on the sheet: C62, C63, C64, C65, C66, C67, C68, C79, D1, D2, J1, J10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

Commit message: BOM WIP
Parts:
- C64: value 4.7u -> 4u7
- C67: value C -> 100n
- renumbered L1 to L17, L2 to L18, L3 to L21, L4 to L22, U8 to U13, U12 to U14
Other:
- moved on the sheet: C5, C6, C62, C63, C64, C65, C66, C67, C68, C7, C71, C72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

Commit message: WIP
Connections:
- net TCXO_CLK: now reaches P28.15 (Pin_15)
Other:
- note added: "-5V: 619K"
- note added: "5V: 30k9"
- moved on the sheet: C5, C6, C7, C71, C72, C73, C74, C77, C78, C8, L17, L18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

Commit message: WIP
Parts:
- added D7: VIDEO OUT, symbol Device:LED
- added D8: POWER ON, symbol Device:LED
- added J5: EXT 5V, symbol Connector:Barrel_Jack_Switch
- added R57, R58: 0, symbol Device:R
- added R59: NF, symbol Device:R
- added R60, R63: R, symbol Device:R
- added U12: KF33BDT, Package_TO_SOT_SMD:TO-252-2, symbol Regulator_Linear:KF33BDT
- added U8: LM66200, symbol LM66200:LM66200
- renumbered C5 to C84, C6 to C85, C7 to C87, C8 to C88
Connections:
- net +3.3V_HACKRF: now also R63.1
- net +5V: now also R57.2
- net -5V: now also R58.2
- net GND: now also D7.1 (K), D8.1 (K), J5.2, J5.3, U12.2 (GND), U8.1 (GND), U8.4 (~{ON})
- net VIN: now also R59.2, U8.2 (VOUT), U8.7 (VOUT); no longer Q3.3 (D)
- net at C74.2, L18.2, U14.2 (IN)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: now also R58.1
- net at C73.1, L17.2, U13.8 (IN): now also R57.1
- net VIDEO_OUT_LED: now reaches P28.9 (Pin_9)
- net VIDEO_OUT_LED: now also R60.1
- new net: D7.2 (A), R60.2
- new net: Q3.3 (D), R59.1, U8.2 (VOUT)
- new net: D8.2 (A), R63.2
- new net: J5.1, U12.1 (VI)
- new net: U12.3 (VO), U8.6 (VIN2)
Other:
- moved on the sheet: C62, C63, C64, C65, C66, C67, C68, C71, C72, C73, C74, C77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

Commit message: WIP
Parts:
- added L2: NF, symbol Device:L
- added R64: 0, symbol Device:R
- U12: value KF33BDT -> KF50BDT
Connections:
- net +5V: now also L2.1
- net +8V renamed +VDAC
- net +VDAC: now also R64.1
- net -8V renamed -VDAC
- new net VCC: L2.2, R64.2
