File: hardware/alpha/power.kicad_sch (KiCad schematic)
At the start: 59 parts, among them J1 EXT POWER, J10 HOLE, J11 HOLE, J12 HOLE, J13 HOLE, J14 HOLE, J15 HOLE, J5 EXT 5V, P20 P20, P28 P28, Q3 IRLML2244, U11 TPS63700DRCT, U12 KF50BDT, U13 L78L05_SO8, U14 L79L05_SO8, U2 TPS61170DRVR, U6 TLE2082, U8 LM66200

Commit message: WIP
Parts:
- added C68, C71: 1u, Capacitor_SMD:C_0603_1608Metric, symbol Device:C
- D5: renamed from D8; footprint (none) -> LED_SMD:LED_0805_2012Metric
- D6: renamed from D7; footprint (none) -> LED_SMD:LED_0805_2012Metric
- J5: footprint (none) -> Connector_BarrelJack:BarrelJack_Horizontal
- L16: renamed from L2; footprint (none) -> Inductor_SMD:L_1210_3225Metric
- R53: renamed from R63; footprint (none) -> Resistor_SMD:R_0603_1608Metric
- R54: renamed from R60; footprint (none) -> Resistor_SMD:R_0603_1608Metric
- R55: renamed from R57; footprint (none) -> Resistor_SMD:R_0603_1608Metric
- R56: renamed from R58; footprint (none) -> Resistor_SMD:R_0603_1608Metric
- R57: renamed from R59; footprint (none) -> Resistor_SMD:R_0603_1608Metric
- R58: renamed from R64; footprint (none) -> Resistor_SMD:R_0603_1608Metric
- U13: renamed from U8; footprint (none) -> Package_TO_SOT_SMD:SOT-583-8
- renumbered C71 to C66, C72 to C67, C73 to C69, C74 to C70, C77 to C72, C78 to C73, C84 to C74, C85 to C75, C87 to C76, C88 to C77, C67 to C78, C68 to C79, C64 to C80, C62 to C81, C65 to C82, C63 to C83, C79 to C84, C66 to C85, D1 to D7, D2 to D8, J14 to J10, J15 to J11, J1 to J12, J10 to J6, J11 to J7, J12 to J8, J13 to J9, L17 to L12, L18 to L13, L21 to L14, L22 to L15, L15 to L17, L16 to L18, P20 to P3, P28 to P4, Q3 to Q6, R40 to R59, R45 to R60, R38 to R61, R39 to R62, R42 to R63, R41 to R64, U12 to U10, U13 to U11, U14 to U12, U2 to U14, U11 to U15, U6 to U3
Connections:
- net GND: now also U13.5 (GND), C68.2, C71.2
- net at Q6.3 (D), R57.1: now also U13.3 (VIN1); no longer U13.2 (VOUT)
- net at J5.1, U10.1 (VI): now also C68.1
- net at U10.3 (VO), U13.6 (VIN2): now also C71.1
Other:
- moved on the sheet: J5, U10
