File: hardware/alpha/video-misc.kicad_sch (KiCad schematic)
At the start: 21 parts, among them U1 L78L05_SO8, U3 L79L05_SO8, U6 TLE2082, U8 MCP47FEB22A0-E/ST

Commit message: WIP
Parts:
- added C1, C2, C3, C4, C5, C6: 100n, symbol Device:C
- added P30: BANK2_AUX, symbol Connector_Generic:Conn_02x10_Odd_Even
- added U1: 74LVCH16T245, symbol 74lvc16t245:74LVC16T245
- added U3: 74LVC1T45, symbol 74lvc1t45:74LVC1T45
Connections:
- net +5V: now also C3.1, C4.1, C6.1, U1.18 (VCCB), U1.7 (VCCB), U3.6 (VCCB)
- net GND: now also C1.2, C2.2, C3.2, C4.2, C5.2, C6.2, P30.2 (Pin_2), P30.20 (Pin_20), U1.10 (GND), U1.15 (GND), U1.21 (GND), U1.24 (2DIR), U1.25 (2OE), U1.28 (GND), U1.34 (GND), U1.39 (GND), U1.4 (GND), U1.45 (GND), U1.48 (1OE), U3.2 (GND), U3.5 (DIR)
- new net +3.3VP: C1.1, C2.1, C5.1, P30.1 (Pin_1), U1.1 (1DIR), U1.31 (VCCA), U1.42 (VCCA), U3.1 (VCCA)
- new net AD0: U1.2 (1B1)
- new net AD1: U1.3 (1B2)
- new net AD10: U1.16 (2B3)
- new net AD11: U1.17 (2B4)
- new net AD12: U1.19 (2B5)
- new net AD13: U1.20 (2B6)
- new net AD14: U1.22 (2B7)
- new net AD15: U1.23 (2B8)
- new net AD2: U1.5 (1B3)
- new net AD3: U1.6 (1B4)
- new net AD4: U1.8 (1B5)
- new net AD5: U1.9 (1B6)
- new net AD6: U1.11 (1B7)
- new net AD7: U1.12 (1B8)
- new net AD8: U1.13 (2B1)
- new net AD9: U1.14 (2B2)
- new net DAC_CLK: U3.4 (B)
- new net LAD0: P30.3 (Pin_3), U1.47 (1A1)
- new net LAD1: P30.4 (Pin_4), U1.46 (1A2)
- new net LAD10: P30.13 (Pin_13), U1.33 (2A3)
- new net LAD11: P30.14 (Pin_14), U1.32 (2A4)
- new net LAD12: P30.15 (Pin_15), U1.30 (2A5)
- new net LAD13: P30.16 (Pin_16), U1.29 (2A6)
- new net LAD14: P30.17 (Pin_17), U1.27 (2A7)
- new net LAD15: P30.18 (Pin_18), U1.26 (2A8)
- new net LAD2: P30.5 (Pin_5), U1.44 (1A3)
- new net LAD3: P30.6 (Pin_6), U1.43 (1A4)
- new net LAD4: P30.7 (Pin_7), U1.41 (1A5)
- new net LAD5: P30.8 (Pin_8), U1.40 (1A6)
- new net LAD6: P30.9 (Pin_9), U1.38 (1A7)
- new net LAD7: P30.10 (Pin_10), U1.37 (1A8)
- new net LAD8: P30.11 (Pin_11), U1.36 (2A1)
- new net LAD9: P30.12 (Pin_12), U1.35 (2A2)
- new net LCLK: P30.19 (Pin_19), U3.3 (A)
Other:
- moved on the sheet: C1, C2, C3, C4, C5, C6, C7, C8, L1, L2, R31, U1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

Commit message: WIP
Parts:
- C1, C2, C3, C4, C5, C6: footprint (none) -> Capacitor_SMD:C_0603_1608Metric
- P30: footprint (none) -> hackrf:GSG-HEADER-2x10
- U1: footprint (none) -> Package_TO_SOT_SMD:SOT-23-6
- U3: footprint (none) -> Package_SO:TSSOP-48_6.1x12.5mm_P0.5mm
Changed lines of the file:
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@@
       (effects (font (size 1.27 1.27)) (justify left))
     )
-    (property "Footprint" "" (at 144.4752 41.275 0)
+    (property "Footprint" "Capacitor_SMD:C_0603_1608Metric" (at 144.4752 41.275 0)
       (effects (font (size 1.27 1.27)) hide)
     )
@@
       (effects (font (size 1.27 1.27)) (justify left))
     )
-    (property "Footprint" "" (at 181.9402 76.2 0)
+    (property "Footprint" "Capacitor_SMD:C_0603_1608Metric" (at 181.9402 76.2 0)
       (effects (font (size 1.27 1.27)) hide)
     )
@@
       (effects (font (size 1.27 1.27)) (justify left))
     )
-    (property "Footprint" "" (at 156.5402 41.275 0)
+    (property "Footprint" "Capacitor_SMD:C_0603_1608Metric" (at 156.5402 41.275 0)
       (effects (font (size 1.27 1.27)) hide)
     )
@@
       (effects (font (size 1.27 1.27)) (justify left))
     )
-    (property "Footprint" "" (at 54.3052 41.91 0)
+    (property "Footprint" "Capacitor_SMD:C_0603_1608Metric" (at 54.3052 41.91 0)
       (effects (font (size 1.27 1.27)) hide)
     )
@@
       (effects (font (size 1.524 1.524)))
     )
-    (property "Footprint" "" (at 118.745 68.58 0)
+    (property "Footprint" "Package_TO_SOT_SMD:SOT-23-6" (at 118.745 68.58 0)
       (effects (font (size 1.27 1.27)) hide)
     )
@@
       (effects (font (size 1.524 1.524)))
     )
-    (property "Footprint" "" (at 222.25 69.85 0)
+    (property "Footprint" "Package_SO:TSSOP-48_6.1x12.5mm_P0.5mm" (at 222.25 69.85 0)
       (effects (font (size 1.27 1.27)) hide)
     )
@@
   (symbol (lib_id "Connector_Generic:Conn_02x10_Odd_Even") (at 50.8 78.74 0) (unit 1)
     (in_bom yes) (on_board yes) (dnp no) (fields_autoplaced)
-    (property "Reference" "P30" (at 52.07 62.865 0)
-      (effects (font (size 1.27 1.27)))
-    )
-    (property "Value" "BANK2_AUX" (at 52.07 65.405 0)
-      (effects (font (size 1.27 1.27)))
-    )
-    (property "Footprint" "" (at 50.8 78.74 0)
+    (property "Reference" "P30" (at 52.07 62.23 0)
+      (effects (font (size 1.27 1.27)))
+    )
+    (property "Value" "BANK2_AUX" (at 52.07 64.77 0)
+      (effects (font (size 1.27 1.27)))
+    )
+    (property "Footprint" "hackrf:GSG-HEADER-2x10" (at 50.8 78.74 0)
       (effects (font (size 1.27 1.27)) hide)
     )
@@
         )
         (path "/487245ca-0c1f-4f9d-bc99-20c8f558090f/e1e307fe-d49b-45b6-b177-774a7a482979"
-          (reference "P1") (unit 1)
+          (reference "P30") (unit 1)
         )
       )
@@
       (effects (font (size 1.27 1.27)) (justify left))
     )
-    (property "Footprint" "" (at 265.7602 74.295 0)
+    (property "Footprint" "Capacitor_SMD:C_0603_1608Metric" (at 265.7602 74.295 0)
       (effects (font (size 1.27 1.27)) hide)
     )
@@
       (effects (font (size 1.27 1.27)) (justify left))
     )
-    (property "Footprint" "" (at 66.3702 41.91 0)
-      (effects (font (size 1.27 1.27)) hide)
-    )
+    (property "Footprint" "Capacitor_SMD:C_0603_1608Metric" (at 66.3702 41.91 0)
+      (effects (font (size 1.27 1.27)) hide)
+    )

Commit message: WIP
Parts:
- U1: footprint Package_TO_SOT_SMD:SOT-23-6 -> Package_SO:TSSOP-48_6.1x12.5mm_P0.5mm
- U3: footprint Package_SO:TSSOP-48_6.1x12.5mm_P0.5mm -> Package_TO_SOT_SMD:SOT-23-6
- U8: footprint Package_SO:SOIC-8_3.9x4.9mm_P1.27mm -> Package_SO:TSSOP-8_3x3mm_P0.65mm
Connections:
- net LAD0: now also P30.17 (Pin_17); no longer P30.3 (Pin_3)
- net LAD1: now also P30.18 (Pin_18); no longer P30.4 (Pin_4)
- net LAD10: now also P30.7 (Pin_7); no longer P30.13 (Pin_13)
- net LAD11: now also P30.8 (Pin_8); no longer P30.14 (Pin_14)
- net LAD12: now also P30.5 (Pin_5); no longer P30.15 (Pin_15)
- net LAD13: now also P30.6 (Pin_6); no longer P30.16 (Pin_16)
- net LAD14: now also P30.3 (Pin_3); no longer P30.17 (Pin_17)
- net LAD15: now also P30.4 (Pin_4); no longer P30.18 (Pin_18)
- net LAD2: now also P30.15 (Pin_15); no longer P30.5 (Pin_5)
- net LAD3: now also P30.16 (Pin_16); no longer P30.6 (Pin_6)
- net LAD4: now also P30.13 (Pin_13); no longer P30.7 (Pin_7)
- net LAD5: now also P30.14 (Pin_14); no longer P30.8 (Pin_8)
- net LAD6: now also P30.11 (Pin_11); no longer P30.9 (Pin_9)
- net LAD7: now also P30.12 (Pin_12); no longer P30.10 (Pin_10)
- net LAD8: now also P30.9 (Pin_9); no longer P30.11 (Pin_11)
- net LAD9: now also P30.10 (Pin_10); no longer P30.12 (Pin_12)
Changed lines of the file:
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@@
     (effects (font (size 1.27 1.27)) (justify left bottom))
   )
-  (label "LAD7" (at 61.595 78.74 0) (fields_autoplaced)
+  (label "LAD7" (at 62.23 81.28 0) (fields_autoplaced)
     (effects (font (size 1.27 1.27)) (justify left bottom))
   )
@@
     (effects (font (size 1.27 1.27)) (justify right bottom))
   )
-  (label "LAD14" (at 38.735 88.9 0) (fields_autoplaced)
+  (label "LAD14" (at 38.735 71.12 0) (fields_autoplaced)
     (effects (font (size 1.27 1.27)) (justify left bottom))
   )
@@
     (effects (font (size 1.27 1.27)) (justify left bottom))
   )
-  (label "LAD3" (at 61.595 73.66 0) (fields_autoplaced)
+  (label "LAD3" (at 62.23 86.36 0) (fields_autoplaced)
     (effects (font (size 1.27 1.27)) (justify left bottom))
   )
@@
     (effects (font (size 1.27 1.27)) (justify left bottom))
   )
-  (label "LAD0" (at 38.735 71.12 0) (fields_autoplaced)
+  (label "LAD0" (at 38.735 88.9 0) (fields_autoplaced)
     (effects (font (size 1.27 1.27)) (justify left bottom))
   )
@@
     (effects (font (size 1.27 1.27)) (justify left bottom))
   )
+  (label "LAD[0..15]" (at 73.025 101.6 0) (fields_autoplaced)
+    (effects (font (size 1.27 1.27)) (justify left bottom))
+  )
   (label "AD4" (at 147.955 64.77 180) (fields_autoplaced)
     (effects (font (size 1.27 1.27)) (justify right bottom))
@@
     (effects (font (size 1.27 1.27)) (justify left bottom))
   )
-  (label "LAD1" (at 61.595 71.12 0) (fields_autoplaced)
+  (label "LAD1" (at 62.23 88.9 0) (fields_autoplaced)
     (effects (font (size 1.27 1.27)) (justify left bottom))
   )
@@
     (effects (font (size 1.27 1.27)) (justify right bottom))
   )
-  (label "LAD10" (at 38.735 83.82 0) (fields_autoplaced)
-    (effects (font (size 1.27 1.27)) (justify left bottom))
-  )
-  (label "LAD5" (at 61.595 76.2 0) (fields_autoplaced)
-    (effects (font (size 1.27 1.27)) (justify left bottom))
-  )
-  (label "LAD4" (at 38.735 76.2 0) (fields_autoplaced)
-    (effects (font (size 1.27 1.27)) (justify left bottom))
-  )
-  (label "LAD8" (at 38.735 81.28 0) (fields_autoplaced)
-    (effects (font (size 1.27 1.27)) (justify left bottom))
-  )
-  (label "LAD12" (at 38.735 86.36 0) (fields_autoplaced)
+  (label "LAD10" (at 38.735 76.2 0) (fields_autoplaced)
+    (effects (font (size 1.27 1.27)) (justify left bottom))
+  )
+  (label "LAD5" (at 62.23 83.82 0) (fields_autoplaced)
+    (effects (font (size 1.27 1.27)) (justify left bottom))
+  )
+  (label "LAD4" (at 38.735 83.82 0) (fields_autoplaced)
+    (effects (font (size 1.27 1.27)) (justify left bottom))
+  )
+  (label "LAD8" (at 38.735 78.74 0) (fields_autoplaced)
+    (effects (font (size 1.27 1.27)) (justify left bottom))
+  )
+  (label "LAD12" (at 38.735 73.66 0) (fields_autoplaced)
     (effects (font (size 1.27 1.27)) (justify left bottom))
   )
@@
     (effects (font (size 1.27 1.27)) (justify left bottom))
   )
-  (label "LAD15" (at 61.595 88.9 0) (fields_autoplaced)
+  (label "LAD15" (at 62.23 71.12 0) (fields_autoplaced)
     (effects (font (size 1.27 1.27)) (justify left bottom))
   )
@@
     (effects (font (size 1.27 1.27)) (justify left bottom))
   )
-  (label "LAD11" (at 61.595 83.82 0) (fields_autoplaced)
+  (label "LAD11" (at 62.23 76.2 0) (fields_autoplaced)
     (effects (font (size 1.27 1.27)) (justify left bottom))
   )
@@
     (effects (font (size 1.27 1.27)) (justify left bottom))
   )
-  (label "LAD2" (at 38.735 73.66 0) (fields_autoplaced)
+  (label "LAD2" (at 38.735 86.36 0) (fields_autoplaced)
     (effects (font (size 1.27 1.27)) (justify left bottom))
   )
@@
     (effects (font (size 1.27 1.27)) (justify right bottom))
   )
-  (label "LAD13" (at 61.595 86.36 0) (fields_autoplaced)
-    (effects (font (size 1.27 1.27)) (justify left bottom))
-  )
-  (label "LAD9" (at 61.595 81.28 0) (fields_autoplaced)
-    (effects (font (size 1.27 1.27)) (justify left bottom))
-  )
-  (label "LAD6" (at 38.735 78.74 0) (fields_autoplaced)
+  (label "LAD13" (at 62.23 73.66 0) (fields_autoplaced)
+    (effects (font (size 1.27 1.27)) (justify left bottom))
+  )
+  (label "LAD9" (at 62.23 78.74 0) (fields_autoplaced)
+    (effects (font (size 1.27 1.27)) (justify left bottom))
+  )
+  (label "LAD6" (at 38.735 81.28 0) (fields_autoplaced)
     (effects (font (size 1.27 1.27)) (justify left bottom))
   )
@@
     (effects (font (size 1.27 1.27)) (justify right bottom))
   )
-  (global_label "DAC_AD[0..15]" (shape input) (at 167.005 101.6 0) (fields_autoplaced)
+  (global_label "AD[0..15]" (shape input) (at 167.005 101.6 0) (fields_autoplaced)
     (effects (font (size 1.27 1.27)) (justify left))
-    (property "Intersheetrefs" "${INTERSHEET_REFS}" (at 183.4765 101.6 0)
+    (property "Intersheetrefs" "${INTERSHEET_REFS}" (at 178.8803 101.6 0)
       (effects (font (size 1.27 1.27)) (justify left) hide)
     )
@@
       (effects (font (size 1.524 1.524)))
     )
-    (property "Footprint" "Package_TO_SOT_SMD:SOT-23-6" (at 118.745 68.58 0)
+    (property "Footprint" "Package_SO:TSSOP-48_6.1x12.5mm_P0.5mm" (at 118.745 68.58 0)
       (effects (font (size 1.27 1.27)) hide)
     )
@@
       (effects (font (size 1.524 1.524)))
     )
-    (property "Footprint" "Package_SO:TSSOP-48_6.1x12.5mm_P0.5mm" (at 222.25 69.85 0)
+    (property "Footprint" "Package_TO_SOT_SMD:SOT-23-6" (at 222.25 69.85 0)
       (effects (font (size 1.27 1.27)) hide)
     )
@@
       (effects (font (size 1.27 1.27)) (justify left))
     )
-    (property "Footprint" "Package_SO:SOIC-8_3.9x4.9mm_P1.27mm" (at 254.635 147.955 0)
-      (effects (font (size 1.27 1.27)) hide)
-    )
+    (property "Footprint" "Package_SO:TSSOP-8_3x3mm_P0.65mm" (at 254.635 147.955 0)
+      (effects (font (size 1.27 1.27)) hide)
+    )

Commit message: WIP
Connections:
- net +3.3VP renamed +3.3V_HACKRF
Changed lines of the file:
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@@
   (symbol (lib_id "Amplifier_Operational:AD8620") (at 147.32 154.305 0) (unit 3)
     (in_bom yes) (on_board yes) (dnp no) (fields_autoplaced)
-    (property "Reference" "U6" (at 145.415 153.035 0)
+    (property "Reference" "U6" (at 146.05 153.035 0)
       (effects (font (size 1.27 1.27)) (justify left))
     )
-    (property "Value" "TLE2082" (at 145.415 155.575 0)
+    (property "Value" "TLE2082" (at 146.05 155.575 0)
       (effects (font (size 1.27 1.27)) (justify left))
     )
@@
         )
         (path "/487245ca-0c1f-4f9d-bc99-20c8f558090f/e1e307fe-d49b-45b6-b177-774a7a482979"
-          (reference "U16") (unit 3)
+          (reference "U6") (unit 3)
         )
       )

Commit message: WIP
Changed lines of the file:
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@@
     (stroke (width 0) (type default))
   )
-  (wire (pts (xy 249.555 141.605) (xy 266.7 141.605))
+  (wire (pts (xy 249.555 141.605) (xy 257.175 141.605))
     (stroke (width 0) (type default))
   )
@@
     (stroke (width 0) (type default))
   )
-  (wire (pts (xy 249.555 144.145) (xy 266.7 144.145))
+  (wire (pts (xy 249.555 144.145) (xy 257.175 144.145))
     (stroke (width 0) (type default))
   )
@@
     (effects (font (size 1.27 1.27)) (justify left bottom))
   )
-  (label "GAIN_ADJ" (at 254.635 144.145 0) (fields_autoplaced)
-    (effects (font (size 1.27 1.27)) (justify left bottom))
-  )
   (label "LAD4" (at 89.535 64.77 0) (fields_autoplaced)
     (effects (font (size 1.27 1.27)) (justify left bottom))
@@
   )
   (label "LAD11" (at 62.23 76.2 0) (fields_autoplaced)
-    (effects (font (size 1.27 1.27)) (justify left bottom))
-  )
-  (label "OFFSET_ADJ" (at 254.635 141.605 0) (fields_autoplaced)
     (effects (font (size 1.27 1.27)) (justify left bottom))
   )
@@
     )
   )
+  (global_label "GAIN_ADJ" (shape input) (at 257.175 144.145 0) (fields_autoplaced)
+    (effects (font (size 1.27 1.27)) (justify left))
+    (property "Intersheetrefs" "${INTERSHEET_REFS}" (at 268.7479 144.145 0)
+      (effects (font (size 1.27 1.27)) (justify left) hide)
+    )
+  )
+  (global_label "OFFSET_ADJ" (shape input) (at 257.175 141.605 0) (fields_autoplaced)
+    (effects (font (size 1.27 1.27)) (justify left))
+    (property "Intersheetrefs" "${INTERSHEET_REFS}" (at 271.2878 141.605 0)
+      (effects (font (size 1.27 1.27)) (justify left) hide)
+    )
+  )

Commit message: WIP
Parts:
- added C7: 100n, Capacitor_SMD:C_0603_1608Metric, symbol Device:C
Connections:
- net +5V: now also C7.1
- net GND: now also C7.2
Other:
- moved on the sheet: R43, R44, U8

Commit message: WIP
Parts:
- added C10: 100p, symbol Device:C
- added C11: 33u, symbol Device:C
- added C8: NF, symbol Device:C
- added C9: 82p, symbol Device:C
- added D3, D5: 1N4148, Diode_SMD:D_SOD-123, symbol Device:D
- added D6: 1v4, Package_TO_SOT_SMD:SOT-23, symbol Diode:BZX84Cxx
- added J3: SYNC OUT, MOLEX_73101:731010120, symbol Connector:Conn_Coaxial
- added Q4, Q5: BC857, Package_TO_SOT_SMD:SOT-23, symbol Transistor_BJT:BC857
- added Q6: BC807, Package_TO_SOT_SMD:SOT-23, symbol Transistor_BJT:BC807
- added R18: NF, Resistor_SMD:R_0603_1608Metric, symbol Device:R
- added R31: 220, Resistor_SMD:R_0603_1608Metric, symbol Device:R
- added R43: 1k, Resistor_SMD:R_0603_1608Metric, symbol Device:R
- added R44: 1k5, Resistor_SMD:R_0603_1608Metric, symbol Device:R
- added R47, R49: 4k3, Resistor_SMD:R_0603_1608Metric, symbol Device:R
- added R48: 47, Resistor_SMD:R_0603_1608Metric, symbol Device:R
- added R50: 909, Resistor_SMD:R_0603_1608Metric, symbol Device:R
- added R51: 75, Resistor_SMD:R_0603_1608Metric, symbol Device:R
- added R52: 10k, Resistor_SMD:R_0603_1608Metric, symbol Device:R
Connections:
- net +5V: now also R31.1, R47.1, R49.1
- net -8V: now also D5.1 (K), Q6.3 (C)
- net GND: now also C10.2, C8.2, C9.2, D3.1 (K), Q4.3 (C), R44.2, R52.2; no longer U8.6 (LAT/HVC)
- net GNDA: now also J3.2 (Ext)
- new net: C11.2, D5.2 (A), R50.2
- new net: C8.1, Q4.1 (B), R43.2
- new net: Q6.1 (B), R48.1
- new net: C10.1, C9.1, D6.3 (K), R48.2, R50.1
- new net: C11.1, Q6.2 (E), R49.2, R51.1
- new net: J3.1 (In), R18.1, R51.2
- new net: D3.2 (A), D6.1 (A), Q5.3 (C)
- new net: Q4.2 (E), Q5.2 (E), R31.2
- new net: Q5.1 (B), R44.1, R47.2
- new net DA_HVC: R52.1, U8.6 (LAT/HVC)
- new net LSYNC: R43.1
- new net VIDEO: R18.2
Other:
- note added: "CALIBRATION DAC"
- note added: "DAC CLOCK BUFFER"
- note added: "DAC DATA BUFFER"
- note added: "DAC POWER FILTERING / REGULATION"
- note added: "SYNC OUTPUT"
- moved on the sheet: C5, C6, C7, R43, R44, U3, U8

Commit message: WIP
Parts:
- removed D6: 1v4, Package_TO_SOT_SMD:SOT-23, symbol Diode:BZX84Cxx
- added D4, D6: 1N4148, Diode_SMD:D_SOD-123, symbol Device:D
- C10, C8, C9: footprint (none) -> Capacitor_SMD:C_0603_1608Metric
- C11: footprint (none) -> Capacitor_SMD:C_1210_3225Metric
Connections:
- net at C10.1, C9.1, R48.2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: now also D6.1 (K)
- net at D3.2 (A), Q5.3 (C): now also D4.2 (A)
- new net: D4.1 (K), D6.2 (A)
Other:
- moved on the sheet: C1, C10, C11, C2, C3, C4, C7, C8, C9, D3, D5, J3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
