File: hardware/alpha/video-misc.kicad_sch (KiCad schematic)
At the start: 53 parts, among them J3 SYNC OUT, P30 BANK2_AUX, Q4 BC857, Q5 BC857, Q6 BC807, U1 74LVCH16T245, U1 L78L05_SO8, U3 74LVC1T45, U3 L79L05_SO8, U6 TLE2082, U8 MCP47FEB22A0-E/ST

Commit message: WIP
Parts:
- added C75, C76: 100n, Capacitor_SMD:C_0603_1608Metric, symbol Device:C
Connections:
- net +5V: now also C75.1
- net -8V: now also C76.2
- net GND: no longer C10.2, C8.2, C9.2, D3.1 (K), Q4.3 (C), R44.2
- net GNDA renamed GNDV
- net GNDV: now also C10.2, C8.2, C9.2, D3.1 (K), Q4.3 (C), R44.2, C75.2, C76.1

Commit message: WIP
Parts:
- removed R31: 0, Resistor_SMD:R_1210_3225Metric, symbol Device:R
Connections:
- net GNDV is gone; now on net GND: C10.2, C75.2, C76.1, C8.2, C9.2, D3.1 (K), J3.2 (Ext), Q4.3 (C), R44.2
Changed lines of the file:
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@@
   (junction (at 133.985 154.94) (diameter 0) (color 0 0 0 0)
   )
-  (junction (at 43.18 154.94) (diameter 0) (color 0 0 0 0)
-  )
   (junction (at 133.35 31.75) (diameter 0) (color 0 0 0 0)
   )
@@
     (stroke (width 0) (type default))
   )
-  (wire (pts (xy 43.18 154.94) (xy 39.37 154.94))
-    (stroke (width 0) (type default))
-  )
   (wire (pts (xy 175.895 84.455) (xy 175.895 86.995))
     (stroke (width 0) (type default))
@@
     (stroke (width 0) (type default))
   )
-  (wire (pts (xy 31.75 154.94) (xy 29.845 154.94))
-    (stroke (width 0) (type default))
-  )
   (wire (pts (xy 83.82 105.41) (xy 85.725 105.41))
     (stroke (width 0) (type default))
@@
     (stroke (width 0) (type default))
   )
-  (wire (pts (xy 29.845 154.94) (xy 29.845 158.115))
-    (stroke (width 0) (type default))
-  )
   (wire (pts (xy 133.35 41.275) (xy 133.35 43.18))
     (stroke (width 0) (type default))
@@
     )
   )
-  (symbol (lib_id "gndv:GNDV") (at 208.915 102.87 0) (unit 1)
+  (symbol (lib_id "power:GND") (at 208.915 102.87 0) (unit 1)
     (in_bom yes) (on_board yes) (dnp no)
     (property "Reference" "#PWR042" (at 208.915 109.22 0)
       (effects (font (size 1.27 1.27)) hide)
     )
-    (property "Value" "GNDV" (at 208.915 106.68 0)
+    (property "Value" "GND" (at 208.915 106.68 0)
       (effects (font (size 1.27 1.27)))
     )
@@
         )
         (path "/487245ca-0c1f-4f9d-bc99-20c8f558090f/e1e307fe-d49b-45b6-b177-774a7a482979"
-          (reference "#PWR0149") (unit 1)
+          (reference "#PWR0155") (unit 1)
         )
       )
@@
     )
   )
-  (symbol (lib_id "gndv:GNDV") (at 259.715 110.49 0) (unit 1)
+  (symbol (lib_id "power:GND") (at 259.715 110.49 0) (unit 1)
     (in_bom yes) (on_board yes) (dnp no)
     (property "Reference" "#PWR042" (at 259.715 116.84 0)
       (effects (font (size 1.27 1.27)) hide)
     )
-    (property "Value" "GNDV" (at 259.715 114.3 0)
+    (property "Value" "GND" (at 259.715 114.3 0)
       (effects (font (size 1.27 1.27)))
     )
@@
         )
         (path "/487245ca-0c1f-4f9d-bc99-20c8f558090f/e1e307fe-d49b-45b6-b177-774a7a482979"
-          (reference "#PWR0155") (unit 1)
+          (reference "#PWR0151") (unit 1)
         )
       )
@@
     )
   )
-  (symbol (lib_id "gndv:GNDV") (at 198.755 102.87 0) (unit 1)
+  (symbol (lib_id "power:GND") (at 198.755 102.87 0) (unit 1)
     (in_bom yes) (on_board yes) (dnp no)
     (property "Reference" "#PWR042" (at 198.755 109.22 0)
       (effects (font (size 1.27 1.27)) hide)
     )
-    (property "Value" "GNDV" (at 198.755 106.68 0)
+    (property "Value" "GND" (at 198.755 106.68 0)
       (effects (font (size 1.27 1.27)))
     )
@@
         )
         (path "/487245ca-0c1f-4f9d-bc99-20c8f558090f/e1e307fe-d49b-45b6-b177-774a7a482979"
-          (reference "#PWR0150") (unit 1)
+          (reference "#PWR0156") (unit 1)
         )
       )
     )
   )
-  (symbol (lib_id "gndv:GNDV") (at 238.125 102.87 0) (unit 1)
+  (symbol (lib_id "power:GND") (at 238.125 102.87 0) (unit 1)
     (in_bom yes) (on_board yes) (dnp no)
     (property "Reference" "#PWR042" (at 238.125 109.22 0)
       (effects (font (size 1.27 1.27)) hide)
     )
-    (property "Value" "GNDV" (at 238.125 106.68 0)
+    (property "Value" "GND" (at 238.125 106.68 0)
       (effects (font (size 1.27 1.27)))
     )
@@
         )
         (path "/487245ca-0c1f-4f9d-bc99-20c8f558090f/e1e307fe-d49b-45b6-b177-774a7a482979"
-          (reference "#PWR0152") (unit 1)
+          (reference "#PWR0153") (unit 1)
         )
       )
@@
     )
   )
-  (symbol (lib_id "Device:R") (at 35.56 154.94 270) (mirror x) (unit 1)
-    (in_bom yes) (on_board yes) (dnp no)
-    (property "Reference" "R31" (at 35.56 152.4 90)
-      (effects (font (size 1.27 1.27)))
-    )
-    (property "Value" "0" (at 35.56 154.94 90)
-      (effects (font (size 1.27 1.27)))
-    )
-    (property "Footprint" "Resistor_SMD:R_1210_3225Metric" (at 35.56 156.718 90)
-      (effects (font (size 1.27 1.27)) hide)
-    )
-    (property "Datasheet" "~" (at 35.56 154.94 0)
-      (effects (font (size 1.27 1.27)) hide)
-    )
-    (pin "1")
-    (pin "2")
-    (instances
-      (project "dacattac-alpha"
-        (path "/487245ca-0c1f-4f9d-bc99-20c8f558090f/b4bbface-dd1a-4873-ab51-f35caad404be"
-          (reference "R31") (unit 1)
-        )
-        (path "/487245ca-0c1f-4f9d-bc99-20c8f558090f/e1e307fe-d49b-45b6-b177-774a7a482979"
-          (reference "R46") (unit 1)
-        )
-      )
-    )
-  )
   (symbol (lib_id "power:GND") (at 50.165 93.345 0) (unit 1)
     (in_bom yes) (on_board yes) (dnp no) (fields_autoplaced)
@@
     )
   )
-  (symbol (lib_id "gndv:GNDV") (at 271.145 81.915 0) (unit 1)
+  (symbol (lib_id "power:GND") (at 271.145 81.915 0) (unit 1)
     (in_bom yes) (on_board yes) (dnp no)
     (property "Reference" "#PWR042" (at 271.145 88.265 0)
       (effects (font (size 1.27 1.27)) hide)
     )
-    (property "Value" "GNDV" (at 271.145 85.725 0)
+    (property "Value" "GND" (at 271.145 85.725 0)
       (effects (font (size 1.27 1.27)))
     )
@@
         )
         (path "/487245ca-0c1f-4f9d-bc99-20c8f558090f/e1e307fe-d49b-45b6-b177-774a7a482979"
-          (reference "#PWR0154") (unit 1)
+          (reference "#PWR0152") (unit 1)
         )
       )
@@
     )
   )
-  (symbol (lib_id "gndv:GNDV") (at 175.895 95.885 0) (unit 1)
+  (symbol (lib_id "power:GND") (at 175.895 95.885 0) (unit 1)
     (in_bom yes) (on_board yes) (dnp no)
     (property "Reference" "#PWR042" (at 175.895 102.235 0)
       (effects (font (size 1.27 1.27)) hide)
     )
-    (property "Value" "GNDV" (at 175.895 99.695 0)
+    (property "Value" "GND" (at 175.895 99.695 0)
       (effects (font (size 1.27 1.27)))
     )
@@
         )
         (path "/487245ca-0c1f-4f9d-bc99-20c8f558090f/e1e307fe-d49b-45b6-b177-774a7a482979"
-          (reference "#PWR0148") (unit 1)
+          (reference "#PWR0147") (unit 1)
         )
       )
@@
     )
   )
-  (symbol (lib_id "gndv:GNDV") (at 227.965 102.87 0) (unit 1)
+  (symbol (lib_id "power:GND") (at 227.965 102.87 0) (unit 1)
     (in_bom yes) (on_board yes) (dnp no)
     (property "Reference" "#PWR042" (at 227.965 109.22 0)
       (effects (font (size 1.27 1.27)) hide)
     )
-    (property "Value" "GNDV" (at 227.965 106.68 0)
+    (property "Value" "GND" (at 227.965 106.68 0)
       (effects (font (size 1.27 1.27)))
     )
@@
         )
         (path "/487245ca-0c1f-4f9d-bc99-20c8f558090f/e1e307fe-d49b-45b6-b177-774a7a482979"
-          (reference "#PWR0153") (unit 1)
-        )
-      )
-    )
-  )
-  (symbol (lib_id "gndv:GNDV") (at 29.845 158.115 0) (mirror y) (unit 1)
-    (in_bom yes) (on_board yes) (dnp no)
-    (property "Reference" "#PWR054" (at 29.845 164.465 0)
-      (effects (font (size 1.27 1.27)) hide)
-    )
-    (property "Value" "GNDV" (at 29.845 161.925 0)
-      (effects (font (size 1.27 1.27)))
-    )
-    (property "Footprint" "" (at 29.845 158.115 0)
-      (effects (font (size 1.27 1.27)) hide)
-    )
-    (property "Datasheet" "" (at 29.845 158.115 0)
-      (effects (font (size 1.27 1.27)) hide)
-    )
-    (pin "1")
-    (instances
-      (project "dacattac-alpha"
-        (path "/487245ca-0c1f-4f9d-bc99-20c8f558090f/b4bbface-dd1a-4873-ab51-f35caad404be"
-          (reference "#PWR054") (unit 1)
-        )
-        (path "/487245ca-0c1f-4f9d-bc99-20c8f558090f/e1e307fe-d49b-45b6-b177-774a7a482979"
-          (reference "#PWR0156") (unit 1)
+          (reference "#PWR0154") (unit 1)
         )
       )
@@
     )
   )
-  (symbol (lib_id "gndv:GNDV") (at 185.42 95.885 0) (unit 1)
+  (symbol (lib_id "power:GND") (at 185.42 95.885 0) (unit 1)
     (in_bom yes) (on_board yes) (dnp no)
     (property "Reference" "#PWR042" (at 185.42 102.235 0)
       (effects (font (size 1.27 1.27)) hide)
     )
-    (property "Value" "GNDV" (at 185.42 99.695 0)
+    (property "Value" "GND" (at 185.42 99.695 0)
       (effects (font (size 1.27 1.27)))
     )
@@
         )
         (path "/487245ca-0c1f-4f9d-bc99-20c8f558090f/e1e307fe-d49b-45b6-b177-774a7a482979"
-          (reference "#PWR0147") (unit 1)
+          (reference "#PWR0148") (unit 1)
         )
       )
@@
     )
   )
-  (symbol (lib_id "gndv:GNDV") (at 227.965 71.12 0) (unit 1)
+  (symbol (lib_id "power:GND") (at 227.965 71.12 0) (unit 1)
     (in_bom yes) (on_board yes) (dnp no)
     (property "Reference" "#PWR042" (at 227.965 77.47 0)
       (effects (font (size 1.27 1.27)) hide)
     )
-    (property "Value" "GNDV" (at 227.965 75.565 0)
+    (property "Value" "GND" (at 227.965 74.93 0)
       (effects (font (size 1.27 1.27)))
     )
@@
         )
         (path "/487245ca-0c1f-4f9d-bc99-20c8f558090f/e1e307fe-d49b-45b6-b177-774a7a482979"
-          (reference "#PWR0151") (unit 1)
+          (reference "#PWR0150") (unit 1)
         )
       )

Commit message: WIP
Parts:
- R49: value 4k3 -> 470
Changed lines of the file:
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@@
   (junction (at 133.35 31.75) (diameter 0) (color 0 0 0 0)
   )
-  (junction (at 238.125 62.23) (diameter 0) (color 0 0 0 0)
-  )
   (junction (at 83.82 39.37) (diameter 0) (color 0 0 0 0)
   )
@@
   (junction (at 27.94 29.21) (diameter 0) (color 0 0 0 0)
   )
+  (junction (at 238.125 61.595) (diameter 0) (color 0 0 0 0)
+  )
   (junction (at 73.025 143.51) (diameter 0) (color 0 0 0 0)
   )
@@
     (stroke (width 0) (type default))
   )
+  (wire (pts (xy 238.125 61.595) (xy 238.125 62.865))
+    (stroke (width 0) (type default))
+  )
   (wire (pts (xy 139.7 57.15) (xy 131.445 57.15))
     (stroke (width 0) (type default))
@@
     (stroke (width 0) (type default))
   )
-  (wire (pts (xy 238.125 61.595) (xy 238.125 62.23))
+  (wire (pts (xy 238.125 60.325) (xy 238.125 61.595))
     (stroke (width 0) (type default))
   )
@@
     (stroke (width 0) (type default))
   )
-  (wire (pts (xy 238.125 62.23) (xy 238.125 62.865))
-    (stroke (width 0) (type default))
-  )
   (wire (pts (xy 77.47 90.17) (xy 85.725 90.17))
     (stroke (width 0) (type default))
@@
     (stroke (width 0) (type default))
   )
-  (wire (pts (xy 238.125 62.23) (xy 227.965 62.23))
+  (wire (pts (xy 238.125 61.595) (xy 227.965 61.595))
     (stroke (width 0) (type default))
   )
@@
     (stroke (width 0) (type default))
   )
-  (wire (pts (xy 227.965 62.23) (xy 227.965 62.865))
+  (wire (pts (xy 227.965 61.595) (xy 227.965 62.865))
     (stroke (width 0) (type default))
   )
@@
     )
   )
-  (symbol (lib_id "power:+5V") (at 238.125 61.595 0) (unit 1)
+  (symbol (lib_id "power:+5V") (at 238.125 60.325 0) (unit 1)
     (in_bom yes) (on_board yes) (dnp no)
-    (property "Reference" "#PWR0116" (at 238.125 65.405 0)
+    (property "Reference" "#PWR0116" (at 238.125 64.135 0)
       (effects (font (size 1.27 1.27)) hide)
     )
-    (property "Value" "+5V" (at 238.125 57.785 0)
+    (property "Value" "+5V" (at 238.125 56.515 0)
       (effects (font (size 1.27 1.27)))
     )
-    (property "Footprint" "" (at 238.125 61.595 0)
+    (property "Footprint" "" (at 238.125 60.325 0)
       (effects (font (size 1.27 1.27)) hide)
     )
-    (property "Datasheet" "" (at 238.125 61.595 0)
+    (property "Datasheet" "" (at 238.125 60.325 0)
       (effects (font (size 1.27 1.27)) hide)
     )
@@
       (effects (font (size 1.27 1.27)) hide)
     )
-    (property "Value" "-8V" (at 250.825 107.315 0)
+    (property "Value" "-8V" (at 250.825 106.68 0)
       (effects (font (size 1.27 1.27)))
     )
@@
       (effects (font (size 1.27 1.27)) hide)
     )
-    (property "Value" "-8V" (at 238.125 88.9 0)
+    (property "Value" "-8V" (at 238.125 88.265 0)
       (effects (font (size 1.27 1.27)))
     )
@@
       (effects (font (size 1.27 1.27)) (justify left))
     )
-    (property "Value" "4k3" (at 238.125 68.58 90)
+    (property "Value" "470" (at 238.125 68.58 90)
       (effects (font (size 1.27 1.27)) (justify left))
     )

Commit message: WIP
Parts:
- U8: footprint Package_SO:TSSOP-8_3x3mm_P0.65mm -> Package_SO:TSSOP-8_4.4x3mm_P0.65mm
Changed lines of the file:
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@@
       (effects (font (size 1.27 1.27)) (justify left))
     )
-    (property "Footprint" "Package_SO:TSSOP-8_3x3mm_P0.65mm" (at 241.3 148.59 0)
+    (property "Footprint" "Package_SO:TSSOP-8_4.4x3mm_P0.65mm" (at 241.3 148.59 0)
       (effects (font (size 1.27 1.27)) hide)
     )

Commit message: Added / updated BOm
Parts:
- removed C1 (x2), C2 (x2), C3, C4, C7, C8: 100n, Capacitor_SMD:C_0603_1608Metric, symbol Device:C
- removed C5, C6: 33u, Capacitor_SMD:C_1210_3225Metric, symbol Device:C
- removed L1 (x2), L2 (x2): 5.6u, Inductor_SMD:L_1210_3225Metric, symbol Device:L
- removed U1: L78L05_SO8, Package_SO:SOIC-8_3.9x4.9mm_P1.27mm, symbol Regulator_Linear:L78L05_SO8
- removed U3: L79L05_SO8, Package_SO:SOIC-8_3.9x4.9mm_P1.27mm, symbol Regulator_Linear:L79L05_SO8
- removed U6: TLE2082, Package_SO:SOIC-8_3.9x4.9mm_P1.27mm, symbol Amplifier_Operational:AD8620
Other:
- note removed: "DAC POWER FILTERING / REGULATION"
- moved on the sheet: C10, C11, C5, C6, C7, C75, C76, C8, C9, D3, D4, D5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

Commit message: WIP
Parts:
- removed C8: NF, Capacitor_SMD:C_0603_1608Metric, symbol Device:C
- removed Q4: BC857, Package_TO_SOT_SMD:SOT-23, symbol Transistor_BJT:BC857
- added C80: 100n, symbol Device:C
- added Q1: 2N7002, Package_TO_SOT_SMD:SOT-23, symbol Transistor_FET:2N7002
- added R53, R55: 100, symbol Device:R
- added R54: 39, symbol Device:R
- added R56: NF, symbol Device:R
- added X1: ECS-TXO-3225-270-TR, Oscillator:Oscillator_SMD_Abracon_ASV-4Pin_7.0x5.1mm, symbol Oscillator:ASV-xxxMHz
- R43: value 1k -> 10
- U8: value MCP47FEB22A0-E/ST -> MCP47FEB22A1-E/ST
Connections:
- net +3.3V_HACKRF: now also U1.24 (2DIR), U3.5 (DIR), C80.1, R56.1, X1.4 (Vdd)
- net DAC_CLK: now also R53.2; no longer U3.4 (B)
- net GND: now also C80.2, Q1.2 (S), X1.2 (GND); no longer U1.24 (2DIR), U3.5 (DIR)
- net LCLK: now also R54.1; no longer U3.3 (A)
- net at R43.2: now also Q1.1 (G)
- net at Q5.2 (E), R31.2: now also Q1.3 (D)
- new net: R56.2, X1.1 (EN)
- new net: R53.1, U3.4 (B)
- new net: R54.2, U3.3 (A)
- new net: R55.1, X1.3 (OUT)
- new net TCXO_CLK: R55.2
Other:
- note added: "27 MHz REFERENCE"
- note added: "NOTE: 100R after output to allow TCXO safely clash with P56 (output) on standard HackRF CPLD code"
- note added: "NOTE: Input using FET to allow CPLD to pull P55 high when running HackRF CPLD code."
- moved on the sheet: C10, C11, C5, C6, C7, C75, C76, C9, D3, D4, D5, D6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

Commit message: WIP
Parts:
- U17: renamed from U8; value MCP47FEB22A1-E/ST -> MCP47FEB22A1-E/ST
- X1: value ECS-TXO-3225-270-TR -> ECS-TXO-3225-270-TR
- renumbered Q1 to Q4, R43 to R61, R44 to R62

Commit message: WIP
Connections:
- net +5V: no longer C3.1, C4.1, C6.1, C75.1, R31.1, R47.1, R49.1, U1.18 (VCCB), U1.7 (VCCB), U3.6 (VCCB)
- net -8V: no longer C76.2, D5.1 (K)
- new net +5VA: C75.1, R31.1, R47.1, R49.1
- new net -VDAC: C76.2, D5.1 (K)
- new net VCC: C3.1, C4.1, C6.1, U1.18 (VCCB), U1.7 (VCCB), U3.6 (VCCB)
