File: hardware/alpha/video-misc.kicad_sch (KiCad schematic)
At the start: 42 parts, among them J3 SYNC OUT, P30 BANK2_AUX, Q4 2N7002, Q5 BC857, Q6 BC807, U1 74LVCH16T245, U17 MCP47FEB22A1-E/ST, U3 74LVC1T45, X1 ECS-TXO-3225-270-TR

Commit message: WIP
Parts:
- C45: renamed from C80; footprint (none) -> Capacitor_SMD:C_0603_1608Metric
- R31: renamed from R56; footprint (none) -> Resistor_SMD:R_0603_1608Metric
- R32: renamed from R55; footprint (none) -> Resistor_SMD:R_0603_1608Metric
- R35: renamed from R54; footprint (none) -> Resistor_SMD:R_0603_1608Metric
- R39: renamed from R53; footprint (none) -> Resistor_SMD:R_0603_1608Metric
- X1: footprint Oscillator:Oscillator_SMD_Abracon_ASV-4Pin_7.0x5.1mm -> Oscillator:Oscillator_SMD_EuroQuartz_XO32-4Pin_3.2x2.5mm
- renumbered C2 to C42, C1 to C43, C7 to C44, C3 to C46, C4 to C47, C5 to C48, C75 to C49, C9 to C50, C10 to C51, C11 to C52, C76 to C53, C6 to C54, D3 to D1, D4 to D2, D6 to D3, D5 to D4, J3 to J2, P30 to P1, Q4 to Q1, Q5 to Q2, Q6 to Q3, R61 to R28, R62 to R29, R52 to R30, R43 to R33, R31 to R34, R47 to R36, R44 to R37, R48 to R38, R49 to R40, R50 to R41, R51 to R42, R18 to R43, U17 to U5, U1 to U6, U3 to U7
Other:
- note added: "OR WURTH 830207670409 (54 MHz)"

Commit message: WIP
Connections:
- net -8V is gone; now on net -VDAC: Q3.3 (C)
Changed lines of the file:
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@@
-	)
-	(symbol
-		(lib_id "power:-8V")
-		(at 238.125 106.045 180)
-		(unit 1)
-		(exclude_from_sim no)
-		(in_bom yes)
-		(on_board yes)
-		(dnp no)
-		(property "Reference" "#PWR069"
-			(at 238.125 108.585 0)
-			(effects
-				(font
-					(size 1.27 1.27)
-				)
-				(hide yes)
-			)
-		)
-		(property "Value" "-8V"
-			(at 238.125 109.855 0)
-			(effects
-				(font
-					(size 1.27 1.27)
-				)
-			)
-		)
-		(property "Footprint" ""
-			(at 238.125 106.045 0)
-			(effects
-				(font
-					(size 1.27 1.27)
-				)
-				(hide yes)
-			)
-		)
-		(property "Datasheet" ""
-			(at 238.125 106.045 0)
-			(effects
-				(font
-					(size 1.27 1.27)
-				)
-				(hide yes)
-			)
-		)
-		(property "Description" ""
-			(at 238.125 106.045 0)
-			(effects
-				(font
-					(size 1.27 1.27)
-				)
-				(hide yes)
-			)
-		)
-		(pin "1"
-		)
-		(instances
-			(project "dacattac-alpha"
-				(path "/487245ca-0c1f-4f9d-bc99-20c8f558090f/e1e307fe-d49b-45b6-b177-774a7a482979"
-					(reference "#PWR069")
-					(unit 1)
-				)
-			)
-		)
 	)
 	(symbol
@@
 					(unit 1)
 				)
+			)
+		)
+	)
+	(symbol
+		(lib_id "-VDAC:-VDAC")
+		(at 238.125 106.045 180)
+		(unit 1)
+		(exclude_from_sim no)
+		(in_bom yes)
+		(on_board yes)
+		(dnp no)
+		(property "Reference" "#PWR069"
+			(at 238.125 102.235 0)
+			(effects
+				(font
+					(size 1.27 1.27)
+				)
+				(hide yes)
+			)
+		)
+		(property "Value" "-VDAC"
+			(at 238.125 110.49 0)
+			(effects
+				(font
+					(size 1.27 1.27)
+				)
+			)
+		)
+		(property "Footprint" ""
+			(at 238.125 106.045 0)
+			(effects
+				(font
+					(size 1.27 1.27)
+				)
+				(hide yes)
+			)
+		)
+		(property "Datasheet" ""
+			(at 238.125 106.045 0)
+			(effects
+				(font
+					(size 1.27 1.27)
+				)
+				(hide yes)
+			)
+		)
+		(property "Description" "Power symbol creates a global label with name \"-VDAC\""
+			(at 238.125 106.045 0)
+			(effects
+				(font
+					(size 1.27 1.27)
+				)
+				(hide yes)
+			)
+		)
+		(pin "1"
+		)
+		(instances
+			(project "dacattac-alpha"
+				(path "/487245ca-0c1f-4f9d-bc99-20c8f558090f/e1e307fe-d49b-45b6-b177-774a7a482979"
+					(reference "#PWR069")
+					(unit 1)
+				)
